File: _saved_ortho40.sch (KiCad schematic (older format))
At the start: 115 parts, among them J1 USB_mini_micro_B, K11 KEYSW, K110 KEYSW, K111 KEYSW, K112 KEYSW, K12 KEYSW, K13 KEYSW, K14 KEYSW, K15 KEYSW, K16 KEYSW, K17 KEYSW, K18 KEYSW, K19 KEYSW, K21 KEYSW, K210 KEYSW, K211 KEYSW, K212 KEYSW, K22 KEYSW, K23 KEYSW, K24 KEYSW, K25 KEYSW, K26 KEYSW, K27 KEYSW, K28 KEYSW, K29 KEYSW, K31 KEYSW, K310 KEYSW, K311 KEYSW, K312 KEYSW, K32 KEYSW, K33 KEYSW, K34 KEYSW, K35 KEYSW, K36 KEYSW, K37 KEYSW, K38 KEYSW, K39 KEYSW, K41 KEYSW, K410 KEYSW, K411 KEYSW, K412 KEYSW, K42 KEYSW, K43 KEYSW, K44 KEYSW, K45 KEYSW, K46 KEYSW, K48 KEYSW, K49 KEYSW, SW1 SW_PUSH, U1 ATMEGA32U4, X1 XTAL

Commit message: Added Planck-compatible mounting holes
Parts:
- H1, H2, H3, H4, H5, H6: footprint MountingHole:MountingHole_5mm_Pad_Via -> MountingHole:MountingHole_2.5mm_Pad
Changed lines of the file:
@@
 F 0 "H3" H 14800 2021 50  0000 L CNN
 F 1 "MountingHole" H 14800 1930 50  0000 L CNN
-F 2 "MountingHole:MountingHole_5mm_Pad_Via" H 14700 1975 50  0001 C CNN
+F 2 "MountingHole:MountingHole_2.5mm_Pad" H 14700 1975 50  0001 C CNN
 F 3 "~" H 14700 1975 50  0001 C CNN
 	1    14700 1975
@@
 F 0 "H4" H 14800 2221 50  0000 L CNN
 F 1 "MountingHole" H 14800 2130 50  0000 L CNN
-F 2 "MountingHole:MountingHole_5mm_Pad_Via" H 14700 2175 50  0001 C CNN
+F 2 "MountingHole:MountingHole_2.5mm_Pad" H 14700 2175 50  0001 C CNN
 F 3 "~" H 14700 2175 50  0001 C CNN
 	1    14700 2175
@@
 F 0 "H1" H 14800 1621 50  0000 L CNN
 F 1 "MountingHole" H 14800 1530 50  0000 L CNN
-F 2 "MountingHole:MountingHole_5mm_Pad_Via" H 14700 1575 50  0001 C CNN
+F 2 "MountingHole:MountingHole_2.5mm_Pad" H 14700 1575 50  0001 C CNN
 F 3 "~" H 14700 1575 50  0001 C CNN
 	1    14700 1575
@@
 F 0 "H2" H 14800 1821 50  0000 L CNN
 F 1 "MountingHole" H 14800 1730 50  0000 L CNN
-F 2 "MountingHole:MountingHole_5mm_Pad_Via" H 14700 1775 50  0001 C CNN
+F 2 "MountingHole:MountingHole_2.5mm_Pad" H 14700 1775 50  0001 C CNN
 F 3 "~" H 14700 1775 50  0001 C CNN
 	1    14700 1775
@@
 F 0 "H5" H 14800 2421 50  0000 L CNN
 F 1 "MountingHole" H 14800 2330 50  0000 L CNN
-F 2 "MountingHole:MountingHole_5mm_Pad_Via" H 14700 2375 50  0001 C CNN
+F 2 "MountingHole:MountingHole_2.5mm_Pad" H 14700 2375 50  0001 C CNN
 F 3 "~" H 14700 2375 50  0001 C CNN
 	1    14700 2375
@@
 F 0 "H6" H 14800 2621 50  0000 L CNN
 F 1 "MountingHole" H 14800 2530 50  0000 L CNN
-F 2 "MountingHole:MountingHole_5mm_Pad_Via" H 14700 2575 50  0001 C CNN
+F 2 "MountingHole:MountingHole_2.5mm_Pad" H 14700 2575 50  0001 C CNN
 F 3 "~" H 14700 2575 50  0001 C CNN
 	1    14700 2575
