File: ortho40.sch (KiCad schematic (older format))
At the start: 115 parts, among them J1 USB_mini_micro_B, K11 KEYSW, K110 KEYSW, K111 KEYSW, K112 KEYSW, K12 KEYSW, K13 KEYSW, K14 KEYSW, K15 KEYSW, K16 KEYSW, K17 KEYSW, K18 KEYSW, K19 KEYSW, K21 KEYSW, K210 KEYSW, K211 KEYSW, K212 KEYSW, K22 KEYSW, K23 KEYSW, K24 KEYSW, K25 KEYSW, K26 KEYSW, K27 KEYSW, K28 KEYSW, K29 KEYSW, K31 KEYSW, K310 KEYSW, K311 KEYSW, K312 KEYSW, K32 KEYSW, K33 KEYSW, K34 KEYSW, K35 KEYSW, K36 KEYSW, K37 KEYSW, K38 KEYSW, K39 KEYSW, K41 KEYSW, K410 KEYSW, K411 KEYSW, K412 KEYSW, K42 KEYSW, K43 KEYSW, K44 KEYSW, K45 KEYSW, K46 KEYSW, K48 KEYSW, K49 KEYSW, SW1 SW_PUSH, U1 ATMEGA32U4, X1 XTAL

Commit message: Added support for full grid and 2x2U
Parts:
- added D47: 1N4148, Diode_THT:D_DO-34_SOD68_P2.54mm_Vertical_AnodeUp, symbol Device:D
- added K2U1, K2U2, K2U3: KEYSW, keebs:Mx_Alps_200, symbol keyboard_parts:KEYSW
- added K47: KEYSW, keebs:Mx_Alps_100, symbol keyboard_parts:KEYSW
- H1, H2, H3, H4, H5, H6: footprint MountingHole:MountingHole_5mm_Pad_Via -> MountingHole:MountingHole_2.5mm_Pad
- K46: footprint keebs:Mx_Alps_200 -> keebs:Mx_Alps_100
Connections:
- wire segments 370 -> 388
Other:
- moved on the sheet: D41, D410, D411, D412, D42, D43, D44, D45, D46, D48, D49
