File: ortho40.kicad_pcb (KiCad board)
At the start: 2 copper layers, 229 x 79.3 mm, 109 parts, among them J1 USB_mini_micro_B, K11 KEYSW, K110 KEYSW, K111 KEYSW, K112 KEYSW, K12 KEYSW, K13 KEYSW, K14 KEYSW, K15 KEYSW, K16 KEYSW, K17 KEYSW, K18 KEYSW, K19 KEYSW, K21 KEYSW, K210 KEYSW, K211 KEYSW, K212 KEYSW, K22 KEYSW, K23 KEYSW, K24 KEYSW, K25 KEYSW, K26 KEYSW, K27 KEYSW, K28 KEYSW, K29 KEYSW, K31 KEYSW, K310 KEYSW, K311 KEYSW, K312 KEYSW, K32 KEYSW, K33 KEYSW, K34 KEYSW, K35 KEYSW, K36 KEYSW, K37 KEYSW, K38 KEYSW, K39 KEYSW, K41 KEYSW, K410 KEYSW, K411 KEYSW, K412 KEYSW, K42 KEYSW, K43 KEYSW, K44 KEYSW, K45 KEYSW, K46 KEYSW, K48 KEYSW, K49 KEYSW, SW1 SW_PUSH, U1 ATMEGA32U4, X1 XTAL

Commit message: Added Planck-compatible mounting holes
Parts:
- added G***: LOGO, SharkPCB:mountHoles, F.Cu at (104.5, -42.8)
- added G***: LOGO, SharkPCB:mountHoles, F.Cu at (109.7, 0.95)
- added G***: LOGO, SharkPCB:mountHoles, F.Cu at (140.1, 31.4)
- added H1: MountingHole, MountingHole:MountingHole_2.5mm_Pad, F.Cu at (91.2, 121.6)
- added H2: MountingHole, MountingHole:MountingHole_2.5mm_Pad, F.Cu at (53.2, 102.6)
- added H3: MountingHole, MountingHole:MountingHole_2.5mm_Pad, F.Cu at (91.2, 83.6)
- added H4: MountingHole, MountingHole:MountingHole_2.5mm_Pad, F.Cu at (243.2, 102.6)
- added H5: MountingHole, MountingHole:MountingHole_2.5mm_Pad, F.Cu at (205.2, 83.6)
- added H6: MountingHole, MountingHole:MountingHole_2.5mm_Pad, F.Cu at (205.2, 121.6)
- moved C1 19.0 mm to (189.1, 83.6)
- moved C2 19.0 mm to (183.1, 83.6)
- moved X1 19.0 mm to (186.2, 83.6)
- moved D212 3.16 mm to (243.2, 97.5)
- moved D312 2.85 mm to (243.2, 107.3)
- moved D39 2.21 mm to (205.2, 116.1)
- turned C8 to 270 degrees
Routing:
- net /XTAL2: track 13.5 -> 32.4 mm
- net /Row3: track 236.2 -> 247.5 mm
- net /XTAL1: track 20.5 -> 30.8 mm
- net /Row2: track 368.4 -> 372.1 mm
- net Net-(D212-Pad2): track 21.0 -> 17.5 mm
- net /Row4: track 246.3 -> 249.0 mm
- net Net-(D39-Pad2): track 11.8 -> 9.55 mm
- net /Col1: track 216.5 -> 218.2 mm
- net Net-(D28-Pad2): track 10.3 -> 8.70 mm
- net Net-(D312-Pad2): track 12.8 -> 14.0 mm

Commit message: Added support for full grid and 2x2U
Parts:
- removed G*** (x3): LOGO, SharkPCB:mountHoles
- added D47: 1N4148, Diode_THT:D_DO-34_SOD68_P2.54mm_Vertical_AnodeUp, F.Cu at (146.8, 121.6)
- added K2U1: KEYSW, keebs:Mx_Alps_200, F.Cu at (129.2, 131.1)
- added K2U2: KEYSW, keebs:Mx_Alps_200, F.Cu at (167.2, 131.1)
- added K2U3: KEYSW, keebs:Mx_Alps_200, F.Cu at (148.2, 131.1)
- added K47: KEYSW, keebs:Mx_Alps_100, F.Cu at (157.7, 131.1)
- K46: footprint keebs:Mx_Alps_200 -> keebs:Mx_Alps_100
- moved D45 14.1 mm to (121.0, 121.6), turned to 0 degrees
- moved D46 12.1 mm to (171.2, 121.6), turned to 180 degrees
- moved K46 9.50 mm to (138.7, 131.1)
Routing:
- net /Col6: track 138.0 -> 178.6 mm
- net /Row4: track 249.0 -> 270.6 mm
- net Net-(D47-Pad2): track 0.00 -> 20.1 mm
- net Net-(D46-Pad2): track 18.2 -> 36.7 mm
- net /Col5: track 148.6 -> 158.7 mm
- net Net-(D45-Pad2): track 9.72 -> 15.7 mm
Other:
- outline, holes or cut-outs redrawn

Commit message: Added gerber files
Routing:
- net /Col7: track 92.2 -> 112.4 mm
- net Net-(D46-Pad2): track 36.7 -> 49.4 mm
- net /Col5: track 158.7 -> 161.9 mm
- net Net-(D47-Pad2): track 20.1 -> 20.6 mm
Other:
- outline, holes or cut-outs redrawn
Changed lines of the file:
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@@
   (general
     (thickness 1.6)
-    (drawings 23)
-    (tracks 711)
+    (drawings 22)
+    (tracks 723)
     (zones 0)
     (modules 120)
@@
     (38 B.Mask user)
     (39 F.Mask user)
-    (40 Dwgs.User user)
+    (40 Dwgs.User user hide)
     (41 Cmts.User user)
     (42 Eco1.User user)
-    (43 Eco2.User user)
+    (43 Eco2.User user hide)
     (44 Edge.Cuts user)
     (45 Margin user hide)
@@
     (visible_elements FFFFFF7F)
     (pcbplotparams
-      (layerselection 0x010fc_ffffffff)
-      (usegerberextensions false)
+      (layerselection 0x030f0_ffffffff)
+      (usegerberextensions true)
       (usegerberattributes false)
       (usegerberadvancedattributes false)
@@
       (outputformat 1)
       (mirror false)
-      (drillshape 1)
+      (drillshape 0)
       (scaleselection 1)
-      (outputdirectory ""))
+      (outputdirectory "gerbers/"))
   )
   (net 0 "")
@@
   (gr_arc (start 218.975 63.65) (end 218.975 64.125) (angle -90) (layer Edge.Cuts) (width 0.15))
   (gr_arc (start 219.925 63.65) (end 219.925 63.175) (angle -90) (layer Edge.Cuts) (width 0.15))
-  (gr_line (start 229.9 64.125) (end 261.25 64.125) (layer Edge.Cuts) (width 0.15))
+  (gr_line (start 229.9 64.125) (end 261.725 64.125) (layer Edge.Cuts) (width 0.15))
   (gr_line (start 34.675 64.125) (end 218.025 64.125) (layer Edge.Cuts) (width 0.15))
   (gr_arc (start 34.675 65.075) (end 34.675 64.125) (angle -90) (layer Edge.Cuts) (width 0.15))
@@
   (gr_line (start 262.675 65.075) (end 262.675 140.125) (layer Edge.Cuts) (width 0.15))
   (gr_arc (start 261.725 65.075) (end 262.675 65.075) (angle -90) (layer Edge.Cuts) (width 0.15))
-  (gr_line (start 261.725 64.125) (end 261.25 64.125) (layer Edge.Cuts) (width 0.15))
   (segment (start 189.05 82.575001) (end 189.05 81.900001) (width 0.25) (layer F.Cu) (net 1) (status 10))
   (segment (start 188.149998 80.999999) (end 188.1 80.999999) (width 0.25) (layer F.Cu) (net 1))
@@
   (segment (start 189.05 81.900001) (end 189.05 80.999999) (width 0.25) (layer F.Cu) (net 1))
   (segment (start 188.1 80.999999) (end 189.05 80.999999) (width 0.25) (layer F.Cu) (net 1))
+  (segment (start 197.224999 80.999999) (end 206.475 90.25) (width 0.25) (layer F.Cu) (net 1))
+  (segment (start 189.05 80.999999) (end 197.224999 80.999999) (width 0.25) (layer F.Cu) (net 1))
+  (segment (start 206.475 95.325) (end 206.475 90.25) (width 0.25) (layer F.Cu) (net 1) (status 10))
   (segment (start 216.6 102.2) (end 222.225 102.2) (width 0.25) (layer F.Cu) (net 2) (status 30))
   (segment (start 222.225 102.2) (end 222.3 102.2) (width 0.25) (layer F.Cu) (net 2) (status 30))
@@
   (segment (start 184.050001 86.200001) (end 186.2 86.200001) (width 0.25) (layer F.Cu) (net 3) (status 20))
   (segment (start 183.5875 85.7375) (end 184.050001 86.200001) (width 0.25) (layer F.Cu) (net 3))
-  (segment (start 197.224999 80.999999) (end 206.475 90.25) (width 0.25) (layer F.Cu) (net 1))
-  (segment (start 189.05 80.999999) (end 197.224999 80.999999) (width 0.25) (layer F.Cu) (net 1))
-  (segment (start 206.475 95.325) (end 206.475 90.25) (width 0.25) (layer F.Cu) (net 1) (status 10))
   (segment (start 186.2 86.200001) (end 189.537499 86.200001) (width 0.25) (layer F.Cu) (net 3) (status 10))
   (segment (start 189.537499 86.200001) (end 192.85 82.8875) (width 0.25) (layer F.Cu) (net 3))
@@
   (segment (start 225.675 68.875) (end 225.675 69.875) (width 0.25) (layer F.Cu) (net 4))
   (segment (start 225.675 67.25) (end 225.675 68.875) (width 0.25) (layer F.Cu) (net 4) (status 10))
-  (via (at 227.525 68.875) (size 1) (drill 0.2) (layers F.Cu B.Cu) (net 4))
+  (via (at 227.525 68.875) (size 1) (drill 0.5) (layers F.Cu B.Cu) (net 4))
   (segment (start 211.525 101.175) (end 214.35 101.175) (width 0.25) (layer F.Cu) (net 5) (status 10))
   (segment (start 214.7 100.825) (end 214.7 100.15) (width 0.25) (layer F.Cu) (net 5) (status 20))
@@
   (segment (start 169.72 126.31) (end 169.72 122.6225) (width 0.25) (layer F.Cu) (net 41))
   (segment (start 149.645468 125.235468) (end 150.72 126.31) (width 0.25) (layer F.Cu) (net 41))
-  (segment (start 151.81861 125.21139) (end 151.81861 123.20639) (width 0.25) (layer F.Cu) (net 41))
-  (segment (start 150.72 126.31) (end 151.81861 125.21139) (width 0.25) (layer F.Cu) (net 41))
-  (segment (start 167.63684 121.6) (end 168.6975 121.6) (width 0.25) (layer F.Cu) (net 41))
-  (segment (start 153.425 121.6) (end 167.63684 121.6) (width 0.25) (layer F.Cu) (net 41))
-  (segment (start 151.81861 123.20639) (end 153.425 121.6) (width 0.25) (layer F.Cu) (net 41))
+  (segment (start 150.72 126.31) (end 150.72 129.345) (width 0.25) (layer F.Cu) (net 41))
+  (segment (start 150.72 129.345) (end 151.05 129.675) (width 0.25) (layer F.Cu) (net 41))
+  (segment (start 151.05 129.675) (end 151.05 132.7625) (width 0.25) (layer F.Cu) (net 41))
+  (segment (start 151.05 132.7625) (end 153.1875 134.9) (width 0.25) (layer F.Cu) (net 41))
+  (segment (start 153.1875 134.9) (end 168.15 134.9) (width 0.25) (layer F.Cu) (net 41))
+  (segment (start 169.72 133.33) (end 169.72 126.31) (width 0.25) (layer F.Cu) (net 41))
+  (segment (start 168.15 134.9) (end 169.72 133.33) (width 0.25) (layer F.Cu) (net 41))
   (segment (start 179.22 126.31) (end 184.735 126.31) (width 0.25) (layer F.Cu) (net 42) (status 10))
   (segment (start 186.2 127.775) (end 186.2 130.46) (width 0.25) (layer F.Cu) (net 42) (status 20))
@@
   (segment (start 199.825 101.975) (end 103.6375 101.975) (width 0.25) (layer F.Cu) (net 61) (status 10))
   (segment (start 103.6375 101.975) (end 97.295 95.6325) (width 0.25) (layer F.Cu) (net 61))
-  (segment (start 116.295 108.83) (end 116.295 127.83) (width 0.25) (layer F.Cu) (net 62) (status 30))
   (segment (start 116.295 70.83) (end 116.295 89.83) (width 0.25) (layer F.Cu) (net 62) (status 30))
   (segment (start 116.295 93.034666) (end 116.295 89.83) (width 0.25) (layer B.Cu) (net 62) (status 20))
@@
   (segment (start 124.265115 127.83) (end 125.795 127.83) (width 0.25) (layer F.Cu) (net 62))
   (segment (start 123.5 128.4875) (end 124.1575 127.83) (width 0.25) (layer F.Cu) (net 62))
+  (segment (start 114.765115 127.83) (end 113.525 126.589885) (width 0.25) (layer F.Cu) (net 62))
+  (segment (start 116.295 127.83) (end 114.765115 127.83) (width 0.25) (layer F.Cu) (net 62))
+  (segment (start 113.525 126.589885) (end 113.525 118.275) (width 0.25) (layer F.Cu) (net 62))
+  (segment (start 116.295 115.505) (end 116.295 108.83) (width 0.25) (layer F.Cu) (net 62))
+  (segment (start 113.525 118.275) (end 116.295 115.505) (width 0.25) (layer F.Cu) (net 62))
   (segment (start 135.295 70.83) (end 135.295 72.839178) (width 0.25) (layer F.Cu) (net 63) (status 30))
   (segment (start 135.295 108.83) (end 135.295 112.02) (width 0.25) (layer F.Cu) (net 63) (status 10))
@@
   (segment (start 154.295 97.77) (end 154.295 89.83) (width 0.25) (layer F.Cu) (net 64) (status 20))
   (segment (start 156.1 99.575) (end 154.295 97.77) (width 0.25) (layer F.Cu) (net 64))
+  (segment (start 153.305016 126.840016) (end 153.202516 126.840016) (width 0.25) (layer F.Cu) (net 64))
+  (segment (start 154.295 127.83) (end 153.305016 126.840016) (width 0.25) (layer F.Cu) (net 64))
+  (segment (start 153.202516 126.840016) (end 152.95 126.5875) (width 0.25) (layer F.Cu) (net 64))
+  (segment (start 152.95 126.5875) (end 152.95 118.75) (width 0.25) (layer F.Cu) (net 64))
+  (segment (start 154.295 117.405) (end 154.295 108.83) (width 0.25) (layer F.Cu) (net 64))
+  (segment (start 152.95 118.75) (end 154.295 117.405) (width 0.25) (layer F.Cu) (net 64))
   (segment (start 173.295 127.83) (end 173.295 108.83) (width 0.25) (layer F.Cu) (net 65) (status 30))
   (segment (start 173.295 72.839178) (end 173.295 89.83) (width 0.25) (layer F.Cu) (net 65) (status 30))
@@
   (segment (start 85.7375 95) (end 84.3125 93.575) (width 0.25) (layer B.Cu) (net 81))
   (segment (start 161.572901 126.31) (end 160.22 126.31) (width 0.25) (layer B.Cu) (net 90))
-  (segment (start 162.015 126.31) (end 161.572901 126.31) (width 0.25) (layer B.Cu) (net 90))
-  (segment (start 162.925 122.3125) (end 162.925 125.4) (width 0.25) (layer B.Cu) (net 90))
-  (segment (start 149.315 121.6) (end 162.2125 121.6) (width 0.25) (layer B.Cu) (net 90))
-  (segment (start 162.925 125.4) (end 162.015 126.31) (width 0.25) (layer B.Cu) (net 90))
-  (segment (start 162.2125 121.6) (end 162.925 122.3125) (width 0.25) (layer B.Cu) (net 90))
+  (segment (start 149.315 121.6) (end 161.5 121.6) (width 0.25) (layer B.Cu) (net 90))
+  (segment (start 161.5 121.6) (end 162.45 122.55) (width 0.25) (layer B.Cu) (net 90))
+  (segment (start 162.45 122.55) (end 162.45 125.875) (width 0.25) (layer B.Cu) (net 90))
+  (segment (start 162.015 126.31) (end 160.22 126.31) (width 0.25) (layer B.Cu) (net 90))
+  (segment (start 162.45 125.875) (end 162.015 126.31) (width 0.25) (layer B.Cu) (net 90))
   (zone (net 2) (net_name GND) (layer F.Cu) (hatch edge 0.508)
     (connect_pads (clearance 0.13))
