File: ortho40.kicad_pcb (KiCad board)
At the start: 2 copper layers, 227.1 x 76 mm, 120 parts, among them J1 USB_mini_micro_B, K11 KEYSW, K110 KEYSW, K111 KEYSW, K112 KEYSW, K12 KEYSW, K13 KEYSW, K14 KEYSW, K15 KEYSW, K16 KEYSW, K17 KEYSW, K18 KEYSW, K19 KEYSW, K21 KEYSW, K210 KEYSW, K211 KEYSW, K212 KEYSW, K22 KEYSW, K23 KEYSW, K24 KEYSW, K25 KEYSW, K26 KEYSW, K27 KEYSW, K28 KEYSW, K29 KEYSW, K2U1 KEYSW, K2U2 KEYSW, K2U3 KEYSW, K31 KEYSW, K310 KEYSW, K311 KEYSW, K312 KEYSW, K32 KEYSW, K33 KEYSW, K34 KEYSW, K35 KEYSW, K36 KEYSW, K37 KEYSW, K38 KEYSW, K39 KEYSW, K41 KEYSW, K410 KEYSW, K411 KEYSW, K412 KEYSW, K42 KEYSW, K43 KEYSW, K44 KEYSW, K45 KEYSW, K46 KEYSW, K47 KEYSW, K48 KEYSW, K49 KEYSW, SW1 SW_PUSH, U1 ATMEGA32U4, X1 XTAL

Commit message: Added Shark illustration
Parts:
- added G***: LOGO, sharkLogo:sharkLogo, B.Cu at (158.9, 105.9)
- added G***: LOGO, sharkLogo:sharkLogo, F.Cu at (138.2, 105.9)
Other:
- board text added: "GondolinElectronics UndecidedSharkPCB v1.0 "I like the nick 'Shark', but I'm so undecided" Shark illustration by Yohan Plantec at vectorportal.com"
- board text removed: "GondolinElectronics UndecidedSharkPCB v1.0 "I like the nick 'Shark', but I'm so undecided""
