File: plate.kicad_pcb (KiCad board)
At the start: 2 copper layers, 229 x 79.3 mm, 0 parts

Commit message: Updated plate files
Routing:
- net (no net): track 39.9 -> 0.00 mm
Other:
- board text removed: "GondolinElectronics UndecidedSharkPCB v1.0 "I like the nick 'Shark', but I'm so undecided""
- board text removed: "SharkPCB Plate V1.0"
Changed lines of the file:
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@@
   (general
     (thickness 1.6)
-    (drawings 228)
-    (tracks 8)
+    (drawings 224)
+    (tracks 0)
     (zones 0)
     (modules 0)
@@
     (0 F.Cu signal)
     (31 B.Cu signal)
-    (32 B.Adhes user hide)
-    (33 F.Adhes user hide)
-    (34 B.Paste user hide)
-    (35 F.Paste user hide)
-    (36 B.SilkS user hide)
-    (37 F.SilkS user hide)
-    (38 B.Mask user hide)
-    (39 F.Mask user hide)
-    (40 Dwgs.User user hide)
-    (41 Cmts.User user hide)
-    (42 Eco1.User user hide)
-    (43 Eco2.User user hide)
+    (32 B.Adhes user)
+    (33 F.Adhes user)
+    (34 B.Paste user)
+    (35 F.Paste user)
+    (36 B.SilkS user)
+    (37 F.SilkS user)
+    (38 B.Mask user)
+    (39 F.Mask user)
+    (40 Dwgs.User user)
+    (41 Cmts.User user)
+    (42 Eco1.User user)
+    (43 Eco2.User user)
     (44 Edge.Cuts user)
-    (45 Margin user hide)
-    (46 B.CrtYd user hide)
-    (47 F.CrtYd user hide)
-    (48 B.Fab user hide)
-    (49 F.Fab user hide)
+    (45 Margin user)
+    (46 B.CrtYd user)
+    (47 F.CrtYd user)
+    (48 B.Fab user)
+    (49 F.Fab user)
   )
   (setup
@@
       (usegerberadvancedattributes false)
       (creategerberjobfile false)
-      (excludeedgelayer true)
+      (excludeedgelayer false)
       (linewidth 0.100000)
       (plotframeref false)
@@
     (uvia_drill 0.2)
   )
-  (gr_text "SharkPCB Plate V1.0" (at 148.707192 102.661104) (layer F.Cu)
-    (effects (font (size 1 1) (thickness 0.25)))
-  )
+  (gr_circle (center 91.260912 83.690472) (end 92.582028 85.27878) (layer Edge.Cuts) (width 0.15))
   (gr_line (start 112.695648 138.078888) (end 112.695648 124.09584) (layer Edge.Cuts) (width 0.15))
   (gr_line (start 114.981624 138.078888) (end 112.695648 138.078888) (layer Edge.Cuts) (width 0.15))
@@
   (gr_line (start 245.712732 119.04888) (end 245.712732 105.09552) (layer Edge.Cuts) (width 0.15))
   (gr_circle (center 91.14216 121.42392) (end 92.463276 123.012228) (layer Edge.Cuts) (width 0.15))
-  (gr_circle (center 91.260912 83.690472) (end 92.582028 85.27878) (layer Edge.Cuts) (width 0.15))
   (gr_circle (center 53.200896 102.601728) (end 54.522012 104.190036) (layer Edge.Cuts) (width 0.15))
   (gr_circle (center 205.084704 121.57236) (end 206.40582 123.160668) (layer Edge.Cuts) (width 0.15))
@@
   (gr_line (start 50.677416 67.124568) (end 50.677416 81.077928) (layer Edge.Cuts) (width 0.15))
   (gr_line (start 36.724056 67.124568) (end 50.677416 67.124568) (layer Edge.Cuts) (width 0.15))
-  (dimension 76.95 (width 0.3) (layer F.SilkS)
-    (gr_text "76.950 mm" (at 27.1125 102.6 90) (layer F.SilkS)
-      (effects (font (size 1.5 1.5) (thickness 0.3)))
-    )
-    (feature1 (pts (xy 33.725 64.125) (xy 28.626079 64.125)))
-    (feature2 (pts (xy 33.725 141.075) (xy 28.626079 141.075)))
-    (crossbar (pts (xy 29.2125 141.075) (xy 29.2125 64.125)))
-    (arrow1a (pts (xy 29.2125 64.125) (xy 29.798921 65.251504)))
-    (arrow1b (pts (xy 29.2125 64.125) (xy 28.626079 65.251504)))
-    (arrow2a (pts (xy 29.2125 141.075) (xy 29.798921 139.948496)))
-    (arrow2b (pts (xy 29.2125 141.075) (xy 28.626079 139.948496)))
-  )
-  (dimension 228.95 (width 0.3) (layer F.SilkS)
-    (gr_text "228.950 mm" (at 148.2 151.725) (layer F.SilkS)
-      (effects (font (size 1.5 1.5) (thickness 0.3)))
-    )
-    (feature1 (pts (xy 262.675 142.975) (xy 262.675 150.211421)))
-    (feature2 (pts (xy 33.725 142.975) (xy 33.725 150.211421)))
-    (crossbar (pts (xy 33.725 149.625) (xy 262.675 149.625)))
-    (arrow1a (pts (xy 262.675 149.625) (xy 261.548496 150.211421)))
-    (arrow1b (pts (xy 262.675 149.625) (xy 261.548496 149.038579)))
-    (arrow2a (pts (xy 33.725 149.625) (xy 34.851504 150.211421)))
-    (arrow2b (pts (xy 33.725 149.625) (xy 34.851504 149.038579)))
-  )
   (gr_line (start 181.925 141.075) (end 261.725 141.075) (layer Edge.Cuts) (width 0.15))
   (gr_line (start 180.5 142.5) (end 181.925 141.075) (layer Edge.Cuts) (width 0.15))
@@
   (gr_line (start 114.475 141.075) (end 115.9 142.5) (layer Edge.Cuts) (width 0.15))
   (gr_line (start 34.675 141.075) (end 114.475 141.075) (layer Edge.Cuts) (width 0.15))
-  (gr_text "GondolinElectronics UndecidedSharkPCB v1.0\n\"I like the nick 'Shark', but I'm so undecided\"" (at 63.65 121.6) (layer F.SilkS)
-    (effects (font (size 1 1) (thickness 0.25)))
-  )
   (gr_line (start 218.975 64.125) (end 218.025 64.125) (layer Edge.Cuts) (width 0.15))
   (gr_line (start 228.95 63.175) (end 219.925 63.175) (layer Edge.Cuts) (width 0.15))
@@
   (gr_line (start 262.675 65.075) (end 262.675 140.125) (layer Edge.Cuts) (width 0.15))
   (gr_arc (start 261.725 65.075) (end 262.675 65.075) (angle -90) (layer Edge.Cuts) (width 0.15))
-  (segment (start 140.097672 103.61112) (end 140.097672 101.800152) (width 0.25) (layer F.Cu) (net 0))
-  (segment (start 156.812016 100.879824) (end 157.762032 101.82984) (width 0.25) (layer F.Cu) (net 0))
-  (segment (start 141.018 100.879824) (end 156.812016 100.879824) (width 0.25) (layer F.Cu) (net 0))
-  (segment (start 140.097672 101.800152) (end 141.018 100.879824) (width 0.25) (layer F.Cu) (net 0))
-  (segment (start 157.762032 101.82984) (end 157.762032 103.136112) (width 0.25) (layer F.Cu) (net 0))
-  (segment (start 157.762032 103.136112) (end 156.693264 104.20488) (width 0.25) (layer F.Cu) (net 0))
-  (segment (start 156.693264 104.20488) (end 140.691432 104.20488) (width 0.25) (layer F.Cu) (net 0))
-  (segment (start 140.691432 104.20488) (end 140.097672 103.61112) (width 0.25) (layer F.Cu) (net 0))
 )

Commit message: Changed board size for Planck case compatibility
Parts:
- added H1: MountingHole, MountingHole:MountingHole_2.5mm_Pad, F.Cu at (91.2, 121.6)
- added H2: MountingHole, MountingHole:MountingHole_2.5mm_Pad, F.Cu at (53.2, 102.6)
- added H3: MountingHole, MountingHole:MountingHole_2.5mm_Pad, F.Cu at (91.2, 83.6)
- added H4: MountingHole, MountingHole:MountingHole_2.5mm_Pad, F.Cu at (243.2, 102.6)
- added H5: MountingHole, MountingHole:MountingHole_2.5mm_Pad, F.Cu at (205.2, 83.6)
- added H6: MountingHole, MountingHole:MountingHole_2.5mm_Pad, F.Cu at (205.2, 121.6)
Other:
- board size 229 x 79.3 mm -> 227.1 x 76 mm
