File: shark.sch (KiCad schematic (older format))
At the start: 132 parts, among them J101 USB_B_Mini, SW1 MXSwitch, SW10 MXSwitch, SW11 MXSwitch, SW12 MXSwitch, SW13 MXSwitch, SW14 MXSwitch, SW15 MXSwitch, SW16 MXSwitch, SW17 MXSwitch, SW18 MXSwitch, SW19 MXSwitch, SW2 MXSwitch, SW20 MXSwitch, SW21 MXSwitch, SW22 MXSwitch, SW23 MXSwitch, SW24 MXSwitch, SW25 MXSwitch, SW26 MXSwitch, SW27 MXSwitch, SW28 MXSwitch, SW29 MXSwitch, SW3 MXSwitch, SW30 MXSwitch, SW31 MXSwitch, SW32 MXSwitch, SW33 MXSwitch, SW34 MXSwitch, SW35 MXSwitch, SW36 MXSwitch, SW37 MXSwitch, SW38 MXSwitch, SW39 MXSwitch, SW4 MXSwitch, SW40 MXSwitch, SW41 MXSwitch, SW42 MXSwitch, SW43 MXSwitch, SW44 MXSwitch, SW45 MXSwitch, SW46 MXSwitch, SW47 MXSwitch, SW48 MXSwitch, SW49 MXSwitch, SW5 MXSwitch, SW50 MXSwitch, SW51 MXSwitch, SW6 MXSwitch, SW7 MXSwitch, SW8 MXSwitch, SW9 MXSwitch, U1 ATmega32U4-AU, Y1 Crystal

Commit message: Started adding LEDs
Parts:
- added LED1, LED10, LED11, LED12, LED13, LED14, LED15, LED16, LED17, LED18, LED19, LED2, LED20, LED21, LED22, LED23, LED24, LED25, LED26, LED27, LED28, LED29, LED3, LED30, LED31, LED32, LED33, LED34, LED35, LED36, LED37, LED38, LED39, LED4, LED40, LED41, LED42, LED43, LED44, LED45, LED46, LED47, LED48, LED49, LED5, LED50, LED51, LED6, LED7, LED8, LED9: LED, Keyboard_switches:thtLED, symbol Keyboard_switches:LED
- added Q1: AO4406AL, Keyboard_switches:AO4406AL, symbol Keyboard_switches:AO4406AL
- added RL1, RL10, RL11, RL12, RL13, RL14, RL15, RL16, RL17, RL18, RL19, RL2, RL20, RL21, RL22, RL23, RL24, RL25, RL26, RL27, RL28, RL29, RL3, RL30, RL31, RL32, RL33, RL34, RL35, RL36, RL37, RL38, RL39, RL4, RL40, RL41, RL42, RL43, RL44, RL45, RL46, RL47, RL48, RL5, RL6, RL7, RL8, RL9: R_LED, Keyboard_switches:Resistor_THT_5.08mm_Horizontal, symbol Device:R_Small
- added RPGate101: 10k, Resistor_SMD:R_1206_3216Metric_Pad1.42x1.75mm_HandSolder, symbol Device:R_Small
- added RSGate101: 1k, Resistor_SMD:R_1206_3216Metric_Pad1.42x1.75mm_HandSolder, symbol Device:R_Small
Connections:
- net GND: now also Q1.S, RPGate101.1
- net Row2: now also U1.38 (PF5); no longer U1.10 (PB2)
- net VCC: now also RL1.1, RL10.1, RL11.1, RL12.1, RL13.1, RL14.1, RL15.1, RL16.1, RL17.1, RL18.1, RL19.1, RL2.1, RL20.1, RL21.1, RL22.1, RL23.1, RL24.1, RL25.1, RL26.1, RL27.1, RL28.1, RL29.1, RL3.1, RL30.1, RL31.1, RL32.1, RL33.1, RL34.1, RL35.1, RL36.1, RL37.1, RL38.1, RL39.1, RL4.1, RL40.1, RL41.1, RL42.1, RL43.1, RL44.1, RL45.1, RL46.1, RL47.1, RL48.1, RL5.1, RL6.1, RL7.1, RL8.1, RL9.1
- net LED_PWM: now reaches U1.12 (PB7)
- net LED_PWM: now also RSGate101.2
- new net: LED1.A, RL1.2
- new net: LED2.A, RL2.2
- new net: LED3.A, RL3.2
- new net: LED4.A, RL4.2
- new net: LED5.A, RL5.2
- new net: LED6.A, RL6.2
- new net: LED7.A, RL7.2
- new net: LED8.A, RL8.2
- new net: LED9.A, RL9.2
- new net: LED10.A, RL10.2
- new net: LED11.A, RL11.2
- new net: LED12.A, RL12.2
- new net: LED13.A, RL13.2
- new net: LED14.A, RL14.2
- new net: LED15.A, RL15.2
- new net: LED16.A, RL16.2
- new net: LED17.A, RL17.2
- new net: LED18.A, RL18.2
- new net: LED19.A, RL19.2
- new net: LED20.A, RL20.2
- new net: LED21.A, RL21.2
- new net: LED22.A, RL22.2
- new net: LED23.A, RL23.2
- new net: LED24.A, RL24.2
- new net: LED25.A, RL25.2
- new net: LED26.A, RL26.2
- new net: LED27.A, RL27.2
- new net: LED28.A, RL28.2
- new net: LED29.A, RL29.2
- new net: LED30.A, RL30.2
- new net: LED31.A, RL31.2
- new net: LED32.A, RL32.2
- new net: LED33.A, RL33.2
- new net: LED34.A, RL34.2
- new net: LED35.A, RL35.2
- new net: LED36.A, RL36.2
- new net: LED37.A, RL37.2
- new net: LED38.A, RL38.2
- new net: LED39.A, RL39.2
- new net: LED40.A, RL40.2
- new net: LED41.A, LED49.A, RL41.2
- new net: LED42.A, LED50.A, RL42.2
- new net: LED43.A, LED51.A, RL43.2
- new net: LED44.A, RL44.2
- new net: LED45.A, RL45.2
- new net: LED46.A, RL46.2
- new net: LED47.A, RL47.2
- new net: LED48.A, RL48.2
- new net: Q1.G, RPGate101.2, RSGate101.1
- new net: LED1.K, LED10.K, LED11.K, LED12.K, LED13.K, LED14.K, LED15.K, LED16.K, LED17.K, LED18.K, LED19.K, LED2.K, LED20.K, LED21.K, LED22.K, LED23.K, LED24.K, LED25.K, LED26.K, LED27.K, LED28.K, LED29.K, LED3.K, LED30.K, LED31.K, LED32.K, LED33.K, LED34.K, LED35.K, LED36.K, LED37.K, LED38.K, LED39.K, LED4.K, LED40.K, LED41.K, LED42.K, LED43.K, LED44.K, LED45.K, LED46.K, LED47.K, LED48.K, LED49.K, LED5.K, LED50.K, LED51.K, LED6.K, LED7.K, LED8.K, LED9.K, Q1.D
- no-connect marks 13 -> 12

Commit message: Finished routing
Connections:
- net Row1: now also U1.10 (PB2); no longer U1.9 (PB1)
- net Row2: now also U1.30 (PB6); no longer U1.38 (PF5)
Changed lines of the file:
@@
 Connection ~ 2225 1950
 NoConn ~ 15100 6050
-NoConn ~ 15100 6350
 NoConn ~ 15100 7450
 NoConn ~ 13900 6650
@@
 	14550 4575 14550 4625
 NoConn ~ 15100 8450
-NoConn ~ 15100 6650
 $Comp
 L Device:C_Small C7
@@
 Wire Wire Line
 	15150 6250 15100 6250
-Text GLabel 15150 6150 2    50   Input ~ 0
+Text GLabel 15150 6250 2    50   Input ~ 0
 Row1
-Wire Wire Line
-	15150 6150 15100 6150
 Text GLabel 13500 7050 0    50   Input ~ 0
 D+
@@
 	1    0    0    -1
 $EndComp
-Text GLabel 15125 8750 2    50   Input ~ 0
+Text GLabel 15150 6650 2    50   Input ~ 0
 Row2
-Wire Wire Line
-	15125 8750 15100 8750
-NoConn ~ 15150 6250
 $Comp
 L Keyboard_switches:LED LED49
@@
 $EndComp
 Connection ~ 4200 10150
+NoConn ~ 15100 6150
+NoConn ~ 15100 8750
+Wire Wire Line
+	15150 6650 15100 6650
+NoConn ~ 15100 6350
 $EndSCHEMATC
