File: shark.sch (KiCad schematic (older format))
At the start: 234 parts, among them J101 USB_B_Mini, Q1 AO4406AL, SW1 MXSwitch, SW10 MXSwitch, SW11 MXSwitch, SW12 MXSwitch, SW13 MXSwitch, SW14 MXSwitch, SW15 MXSwitch, SW16 MXSwitch, SW17 MXSwitch, SW18 MXSwitch, SW19 MXSwitch, SW2 MXSwitch, SW20 MXSwitch, SW21 MXSwitch, SW22 MXSwitch, SW23 MXSwitch, SW24 MXSwitch, SW25 MXSwitch, SW26 MXSwitch, SW27 MXSwitch, SW28 MXSwitch, SW29 MXSwitch, SW3 MXSwitch, SW30 MXSwitch, SW31 MXSwitch, SW32 MXSwitch, SW33 MXSwitch, SW34 MXSwitch, SW35 MXSwitch, SW36 MXSwitch, SW37 MXSwitch, SW38 MXSwitch, SW39 MXSwitch, SW4 MXSwitch, SW40 MXSwitch, SW41 MXSwitch, SW42 MXSwitch, SW43 MXSwitch, SW44 MXSwitch, SW45 MXSwitch, SW46 MXSwitch, SW47 MXSwitch, SW48 MXSwitch, SW49 MXSwitch, SW5 MXSwitch, SW50 MXSwitch, SW51 MXSwitch, SW6 MXSwitch, SW7 MXSwitch, SW8 MXSwitch, SW9 MXSwitch, U1 ATmega32U4-AU, Y1 Crystal

Commit message: Added logo
Parts:
- added L1: Logo, sharkLogo:sharkLogo, symbol Mechanical:MountingHole
Other:
- note added: "ESD Protection"
Changed lines of the file:
@@
 	15150 6650 15100 6650
 NoConn ~ 15100 6350
+Text Notes 13200 4400 0    50   ~ 0
+ESD Protection
+$Comp
+L Mechanical:MountingHole L1
+U 1 1 5C54F135
+P 15300 3450
+F 0 "L1" H 15400 3496 50  0000 L CNN
+F 1 "Logo" H 15400 3405 50  0000 L CNN
+F 2 "sharkLogo:sharkLogo" H 15300 3450 50  0001 C CNN
+F 3 "~" H 15300 3450 50  0001 C CNN
+	1    15300 3450
+	1    0    0    -1
+$EndComp
 $EndSCHEMATC

Commit message: Started switch to STM32F303 processor
Parts:
- removed C3, C4, C5: 0.1u, Capacitor_SMD:C_0805_2012Metric_Pad1.15x1.40mm_HandSolder, symbol Device:C_Small
- removed C6: 4.7u, Capacitor_SMD:C_0805_2012Metric_Pad1.15x1.40mm_HandSolder, symbol Device:C_Small
- removed C8: 1u, Capacitor_SMD:C_0805_2012Metric_Pad1.15x1.40mm_HandSolder, symbol Device:C_Small
- removed J101: USB_B_Mini, Keyboard_switches:miniB_connector, symbol Connector:USB_B_Mini
- removed PSH1: SW_Push, Button_Switch_SMD:SW_SPST_SKQG_WithStem, symbol Switch:SW_Push
- removed R1, R2: 10k, Resistor_SMD:R_1206_3216Metric_Pad1.42x1.75mm_HandSolder, symbol Device:R
- removed R3, R4: 22, Resistor_SMD:R_1206_3216Metric_Pad1.42x1.75mm_HandSolder, symbol Device:R
- removed U1: ATmega32U4-AU, Package_QFP:TQFP-44_10x10mm_P0.8mm, symbol MCU_Microchip_ATmega:ATmega32U4-AU
- removed Y1: Crystal, Crystal:Crystal_SMD_5032-2Pin_5.0x3.2mm_HandSoldering, symbol Device:Crystal
- added CRST1, CSRT2: 4.7n, Capacitor_SMD:C_0805_2012Metric_Pad1.15x1.40mm_HandSolder, symbol Device:C_Small
- added CSin, CSout: 100n, Capacitor_SMD:C_0805_2012Metric_Pad1.15x1.40mm_HandSolder, symbol Device:C_Small
- added CVBus1, CVBus2, CVBus3: 100n, symbol Device:C_Small
- added CVBus4: 1u, symbol Device:C_Small
- added CVBus?: 4.7u, symbol Device:C_Small
- added DRST, DS1: 1N4148, Keyboard_switches:thtDiode, symbol Device:D
- added J1: USB_C_Receptacle, symbol Connector:USB_C_Receptacle
- added QRST: Q_NPN_BCE, symbol Device:Q_NPN_BCE
- added RCC: 5.1k, symbol Device:R_Small
- added RD+, RD-: 22R, symbol Device:R_Small
- added RD+Up: 1.5k, symbol Device:R_Small
- added RRST: 100k, symbol Device:R_Small
- added SW1: SW_Push, symbol Switch:SW_Push
- added U1: STM32F303CCT7, symbol stm32f303cct7:STM32F303CCT7
- added U2: MCP1700-3302E_SOT23, Package_TO_SOT_SMD:SOT-23, symbol Regulator_Linear:MCP1700-3302E_SOT23
- added Y1: 8MHz, symbol Device:Crystal_GND24
Connections:
- net D+: now also RD+.1, U1.33 (PA12/USB_DP)
- net D-: now also RD-.1, U1.32 (PA11/USB_DM)
- net GND: now also CRST1.1, CSRT2.2, CSin.1, CSout.1, CVBus1.2, CVBus2.2, CVBus3.2, CVBus4.2, CVBus?.2, J1.A1 (GND), J1.A12 (GND), J1.B1 (GND), J1.B12 (GND), QRST.3 (E), RCC.1, RRST.2, U1.23 (GND), U1.35 (GND), U1.47 (GND), U1.8 (GND/VSSA/VREF-), U2.1 (GND), Y1.2, Y1.4
- net VCC: now also SW1.1; no longer DS1.1 (K), F1.1, RL1.1, RL10.1, RL11.1, RL12.1, RL13.1, RL14.1, RL15.1, RL16.1, RL17.1, RL18.1, RL19.1, RL2.1, RL20.1, RL21.1, RL22.1, RL23.1, RL24.1, RL25.1, RL26.1, RL27.1, RL28.1, RL29.1, RL3.1, RL30.1, RL31.1, RL32.1, RL33.1, RL34.1, RL35.1, RL36.1, RL37.1, RL38.1, RL39.1, RL4.1, RL40.1, RL41.1, RL42.1, RL43.1, RL44.1, RL45.1, RL46.1, RL47.1, RL48.1, RL5.1, RL6.1, RL7.1, RL8.1, RL9.1
- net XTAL1: now also U1.5 (PF0/OSC_IN/I2C2_SDA), Y1.3
- net XTAL2: now also U1.6 (PF1/OSC_OUT/I2C2_SCL), Y1.1
- net at C7.2, R5.1: now also J1.S1 (SHIELD)
- net VBUS: now reaches F1.2
- net VBUS: now also J1.A4 (VBUS), J1.A9 (VBUS), J1.B4 (VBUS), J1.B9 (VBUS)
- new net: J1.A5 (CC1), J1.B5 (CC2), RCC.2
- new net: J1.A6 (D+), J1.B6 (D+), RD+.2, RD+Up.2
- new net: J1.A7 (D-), J1.B7 (D-), RD-.2
- new net: DRST.2 (A), QRST.1 (B), SW1.2
- new net 3.3V: CSout.2, CVBus1.1, CVBus2.1, CVBus3.1, CVBus4.1, CVBus?.1, DS1.2 (A), U1.1 (VBAT), U1.24 (VCC), U1.36 (VCC), U1.48 (VCC), U1.9 (VCC/VDDA/VREF+), U2.2 (VO)
- new net 5V: CSin.2, DS1.1 (K), DS1.1 (K), F1.1, RD+Up.1, RL1.1, RL10.1, RL11.1, RL12.1, RL13.1, RL14.1, RL15.1, RL16.1, RL17.1, RL18.1, RL19.1, RL2.1, RL20.1, RL21.1, RL22.1, RL23.1, RL24.1, RL25.1, RL26.1, RL27.1, RL28.1, RL29.1, RL3.1, RL30.1, RL31.1, RL32.1, RL33.1, RL34.1, RL35.1, RL36.1, RL37.1, RL38.1, RL39.1, RL4.1, RL40.1, RL41.1, RL42.1, RL43.1, RL44.1, RL45.1, RL46.1, RL47.1, RL48.1, RL5.1, RL6.1, RL7.1, RL8.1, RL9.1, U2.3 (VI)
- new net BOOT0: CRST1.2, DRST.1 (K), RRST.1, U1.44 (BOOT0)
- new net NRST: CSRT2.1, QRST.2 (C), U1.7 (NRST)
- no-connect marks 12 -> 10
Other:
- note added: "Hard reset circuit"
- note added: "Power supply and protection circuit"
- note added: "Voltage regulation capacitor bank\n"
- moved on the sheet: C1, C2, C7, C9, DS1, F1, H1, H10, H11, H12, H2, H3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

Commit message: Began porting to STM32
Parts:
- removed QRST: Q_NPN_BCE, symbol Device:Q_NPN_BCE
- added QRST1: BC847, Package_TO_SOT_SMD:SOT-23, symbol Transistor_BJT:BC847
- added RGB1, RGB2, RGB3, RGB4, RGB5, RGB6, RGB7, RGB8: WS2812B, Keyboard_switches:LED_WS2812B, symbol LED:WS2812B
- CVBus1, CVBus2, CVBus3, CVBus4: footprint (none) -> Capacitor_SMD:C_0805_2012Metric_Pad1.15x1.40mm_HandSolder
- CVBus5: renamed from CVBus?; footprint (none) -> Capacitor_SMD:C_0805_2012Metric_Pad1.15x1.40mm_HandSolder
- DRST1: renamed from DRST; footprint Keyboard_switches:thtDiode -> Diode_SMD:D_0805_2012Metric_Pad1.15x1.40mm_HandSolder
- DS1: footprint Keyboard_switches:thtDiode -> Diode_SMD:D_0805_2012Metric_Pad1.15x1.40mm_HandSolder
- J1: footprint (none) -> USBconnector:TYPE-C-31-M-13
- RCC1: renamed from RCC; footprint (none) -> Resistor_SMD:R_1206_3216Metric_Pad1.42x1.75mm_HandSolder
- RD+1: renamed from RD+; footprint (none) -> Resistor_SMD:R_1206_3216Metric_Pad1.42x1.75mm_HandSolder
- RD+Up1: renamed from RD+Up; footprint (none) -> Resistor_SMD:R_1206_3216Metric_Pad1.42x1.75mm_HandSolder
- RD-1: renamed from RD-; footprint (none) -> Resistor_SMD:R_1206_3216Metric_Pad1.42x1.75mm_HandSolder
- RRST1: renamed from RRST; footprint (none) -> Resistor_SMD:R_1206_3216Metric_Pad1.42x1.75mm_HandSolder
- SWRST1: renamed from SW1; footprint (none) -> Button_Switch_SMD:SW_SPST_SKQG_WithoutStem
- U1: footprint (none) -> Package_QFP:LQFP-48_7x7mm_P0.5mm
- Y1: footprint (none) -> Crystal:Crystal_SMD_5032-4Pin_5.0x3.2mm
- renumbered CSin to CSin1, CSout to CSout1, DS1 to DF1, RPGate101 to RPGate1, RSGate101 to RSGate1
Connections:
- net VCC is gone; now on net 3.3V: SWRST1.1
- net 5V: now also RGB1.1 (VDD), RGB2.1 (VDD), RGB3.1 (VDD), RGB4.1 (VDD), RGB5.1 (VDD), RGB6.1 (VDD), RGB7.1 (VDD), RGB8.1 (VDD)
- net GND: now also QRST1.2 (E), RGB1.3 (VSS), RGB2.3 (VSS), RGB3.3 (VSS), RGB4.3 (VSS), RGB5.3 (VSS), RGB6.3 (VSS), RGB7.3 (VSS), RGB8.3 (VSS)
- net LED_PWM: now also U1.41 (PB5)
- net NRST: now also QRST1.3 (C)
- net RGB_PWM: now reaches U1.20 (PB2)
- net RGB_PWM: now also RGB1.4 (DIN), RGB5.4 (DIN)
- net at DRST1.2 (A), SWRST1.2: now also QRST1.1 (B)
- new net: RGB1.2 (DOUT), RGB2.4 (DIN)
- new net: RGB2.2 (DOUT), RGB3.4 (DIN)
- new net: RGB3.2 (DOUT), RGB4.4 (DIN)
- new net: RGB7.2 (DOUT), RGB8.4 (DIN)
- new net: RGB6.2 (DOUT), RGB7.4 (DIN)
- new net: RGB5.2 (DOUT), RGB6.4 (DIN)
Other:
- note added: "Shield\nnet"
- moved on the sheet: C7, CSin1, CSout1, CVBus1, CVBus2, CVBus3, CVBus4, CVBus5, DF1, DS1, F1, J1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

Commit message: Continued routing
Connections:
- net RGB_PWM: now also U1.19 (PB1); no longer U1.20 (PB2)
Changed lines of the file:
@@
 Wire Wire Line
 	2825 10050 2825 10100
-Text GLabel 15375 8075 2    50   Output ~ 0
+Text GLabel 15375 8175 2    50   Output ~ 0
 RGB_PWM
 Wire Wire Line
-	15375 8075 15300 8075
+	15375 8175 15300 8175
 Text GLabel 2475 9525 0    50   Input ~ 0
 RGB_PWM

Commit message: Continued routing
Connections:
- net Col10: now also U1.22 (PB11)
- net Col6: now also U1.15 (DAC1-OUT2/PA5)
- net Col7: now also U1.10 (PA0)
- net Col8: now also U1.21 (PB10)
- net LED_PWM: now also U1.46 (I2C1_SDA/PB9); no longer U1.41 (PB5)
- net Row2: now also U1.2 (PC13)
- net Row3: now also U1.14 (DAC1-OUT1/PA4)
- net Row4: now also U1.13 (PA3)
Changed lines of the file:
@@
 Wire Wire Line
 	3475 10800 4125 10800
-Text GLabel 15375 7775 2    50   Output ~ 0
+Text GLabel 15375 6875 2    50   Output ~ 0
 LED_PWM
 Wire Wire Line
-	15375 7775 15300 7775
+	15375 6875 15300 6875
 Text GLabel 2825 9100 1    50   Input ~ 0
 5V
@@
 Text GLabel 5875 8750 0    50   Input ~ 0
 3.3V
+Text GLabel 15375 9125 2    50   Input ~ 0
+Col7
+Wire Wire Line
+	15375 9125 15300 9125
+Text GLabel 15375 8725 2    50   Input ~ 0
+Row3
+Text GLabel 15375 9275 2    50   Input ~ 0
+Row2
+Wire Wire Line
+	15375 9275 15300 9275
+Text GLabel 15375 8825 2    50   Input ~ 0
+Row4
+Wire Wire Line
+	15375 8825 15300 8825
+Wire Wire Line
+	15375 8725 15300 8725
+Text GLabel 15375 9125 2    50   Input ~ 0
+Col7
+Text GLabel 15375 8625 2    50   Input ~ 0
+Col6
+Wire Wire Line
+	15375 8625 15300 8625
+Text GLabel 15375 6625 2    50   Input ~ 0
+Col10
+Wire Wire Line
+	15375 6625 15300 6625
+Text GLabel 15375 6725 2    50   Input ~ 0
+Col8
+Wire Wire Line
+	15375 6725 15300 6725
 $EndSCHEMATC

Commit message: Proceeded routing
Connections:
- net Col7: now also U1.2 (PC13); no longer U1.10 (PA0)
- net Row2: now also U1.39 (JTDO/TRACESWO/PB3); no longer U1.2 (PC13)
Changed lines of the file:
@@
 Text GLabel 5875 8750 0    50   Input ~ 0
 3.3V
-Text GLabel 15375 9125 2    50   Input ~ 0
+Text GLabel 15375 9275 2    50   Input ~ 0
 Col7
 Wire Wire Line
-	15375 9125 15300 9125
+	15375 9275 15300 9275
 Text GLabel 15375 8725 2    50   Input ~ 0
 Row3
-Text GLabel 15375 9275 2    50   Input ~ 0
+Text GLabel 15375 7975 2    50   Input ~ 0
 Row2
 Wire Wire Line
-	15375 9275 15300 9275
+	15375 7975 15300 7975
 Text GLabel 15375 8825 2    50   Input ~ 0
 Row4
@@
 Wire Wire Line
 	15375 8725 15300 8725
-Text GLabel 15375 9125 2    50   Input ~ 0
+Text GLabel 15375 9275 2    50   Input ~ 0
 Col7
 Text GLabel 15375 8625 2    50   Input ~ 0

Commit message: Changed to SMD changes
Parts:
- D1, D10, D11, D12, D13, D14, D15, D16, D17, D18, D19, D2, D20, D21, D22, D23, D24, D25, D26, D27, D28, D29, D3, D30, D31, D32, D33, D34, D35, D36, D37, D38, D39, D4, D40, D41, D42, D43, D44, D45, D46, D47, D48, D5, D6, D7, D8, D9: footprint Keyboard_switches:thtDiode -> Keyboard_switches:D_SOD-123
- RL1, RL10, RL11, RL12, RL13, RL14, RL15, RL16, RL17, RL18, RL19, RL2, RL20, RL21, RL22, RL23, RL24, RL25, RL26, RL27, RL28, RL29, RL3, RL30, RL31, RL32, RL33, RL34, RL35, RL36, RL37, RL38, RL39, RL4, RL40, RL41, RL42, RL43, RL44, RL45, RL46, RL47, RL48, RL5, RL6, RL7, RL8, RL9: footprint Keyboard_switches:Resistor_THT_5.08mm_Horizontal -> Resistor_SMD:R_1206_3216Metric
Connections:
- net Col10: now also U1.39 (JTDO/TRACESWO/PB3)
- net Col11: now also U1.38 (I2C1_SCL/JTDI/PA15)
- net Row2: now also U1.40 (JNTRST/PB4); no longer U1.39 (JTDO/TRACESWO/PB3)
