File: shark.sch (KiCad schematic (older format))
At the start: 252 parts, among them J1 USB_C_Receptacle, Q1 AO4406AL, SW1 MXSwitch, SW10 MXSwitch, SW11 MXSwitch, SW12 MXSwitch, SW13 MXSwitch, SW14 MXSwitch, SW15 MXSwitch, SW16 MXSwitch, SW17 MXSwitch, SW18 MXSwitch, SW19 MXSwitch, SW2 MXSwitch, SW20 MXSwitch, SW21 MXSwitch, SW22 MXSwitch, SW23 MXSwitch, SW24 MXSwitch, SW25 MXSwitch, SW26 MXSwitch, SW27 MXSwitch, SW28 MXSwitch, SW29 MXSwitch, SW3 MXSwitch, SW30 MXSwitch, SW31 MXSwitch, SW32 MXSwitch, SW33 MXSwitch, SW34 MXSwitch, SW35 MXSwitch, SW36 MXSwitch, SW37 MXSwitch, SW38 MXSwitch, SW39 MXSwitch, SW4 MXSwitch, SW40 MXSwitch, SW41 MXSwitch, SW42 MXSwitch, SW43 MXSwitch, SW44 MXSwitch, SW45 MXSwitch, SW46 MXSwitch, SW47 MXSwitch, SW48 MXSwitch, SW49 MXSwitch, SW5 MXSwitch, SW50 MXSwitch, SW51 MXSwitch, SW6 MXSwitch, SW7 MXSwitch, SW8 MXSwitch, SW9 MXSwitch, U1 STM32F303CCT7, U2 MCP1700-3302E_SOT23, Y1 8MHz

Commit message: Added photorealistic renders
Parts:
- added L2: LogoBack, sharkLogo:skark, symbol Mechanical:MountingHole
Other:
- moved on the sheet: L1
Changed lines of the file:
@@
 L Mechanical:MountingHole L1
 U 1 1 5C54F135
-P 14625 3700
-F 0 "L1" H 14725 3746 50  0000 L CNN
-F 1 "Logo" H 14725 3655 50  0000 L CNN
-F 2 "sharkLogo:sharkLogo" H 14625 3700 50  0001 C CNN
-F 3 "~" H 14625 3700 50  0001 C CNN
-	1    14625 3700
+P 14625 3525
+F 0 "L1" H 14725 3571 50  0000 L CNN
+F 1 "Logo" H 14725 3480 50  0000 L CNN
+F 2 "sharkLogo:sharkLogo" H 14625 3525 50  0001 C CNN
+F 3 "~" H 14625 3525 50  0001 C CNN
+	1    14625 3525
 	1    0    0    -1
 $EndComp
@@
 Wire Wire Line
 	15375 7975 15300 7975
+$Comp
+L Mechanical:MountingHole L2
+U 1 1 5C525928
+P 14625 3750
+F 0 "L2" H 14725 3796 50  0000 L CNN
+F 1 "LogoBack" H 14725 3705 50  0000 L CNN
+F 2 "sharkLogo:skark" H 14625 3750 50  0001 C CNN
+F 3 "~" H 14625 3750 50  0001 C CNN
+	1    14625 3750
+	1    0    0    -1
+$EndComp
 $EndSCHEMATC

Commit message: Added Pirulen font to the logo
Connections:
- net Col10: now also U1.10 (PA0); no longer U1.22 (PB11), U1.39 (JTDO/TRACESWO/PB3)
- net Col11: now also U1.25 (PB12); no longer U1.38 (I2C1_SCL/JTDI/PA15)
- net Col12: now also U1.31 (I2C2_SDA/PA10)
- net Row3: now also U1.22 (PB11); no longer U1.14 (DAC1-OUT1/PA4)
- net Row4: now also U1.20 (PB2); no longer U1.13 (PA3)
Changed lines of the file:
@@
 Wire Wire Line
 	15375 9275 15300 9275
-Text GLabel 15375 8725 2    50   Input ~ 0
+Text GLabel 15375 6625 2    50   Input ~ 0
 Row3
 Text GLabel 15375 7875 2    50   Input ~ 0
@@
 Wire Wire Line
 	15375 7875 15300 7875
-Text GLabel 15375 8825 2    50   Input ~ 0
+Text GLabel 15375 8075 2    50   Input ~ 0
 Row4
 Wire Wire Line
-	15375 8825 15300 8825
+	15375 8075 15300 8075
 Wire Wire Line
-	15375 8725 15300 8725
+	15375 6625 15300 6625
 Text GLabel 15375 9275 2    50   Input ~ 0
 Col7
@@
 Wire Wire Line
 	15375 8625 15300 8625
-Text GLabel 15375 6625 2    50   Input ~ 0
-Col10
-Wire Wire Line
-	15375 6625 15300 6625
 Text GLabel 15375 6725 2    50   Input ~ 0
 Col8
 Wire Wire Line
 	15375 6725 15300 6725
-Text GLabel 15375 7125 2    50   Input ~ 0
+Text GLabel 15375 6525 2    50   Input ~ 0
 Col11
 Wire Wire Line
-	15375 7125 15300 7125
-Text GLabel 15375 7975 2    50   Input ~ 0
+	15375 6525 15300 6525
+Text GLabel 15375 9125 2    50   Input ~ 0
 Col10
 Wire Wire Line
-	15375 7975 15300 7975
+	15375 9125 15300 9125
 $Comp
 L Mechanical:MountingHole L2
@@
 	1    0    0    -1
 $EndComp
+Text GLabel 15375 7225 2    50   Input ~ 0
+Col12
+Wire Wire Line
+	15375 7225 15300 7225
 $EndSCHEMATC

Commit message: Finished design. Thickening possible traces
Connections:
- net Col1: now also U1.2 (PC13)
- net Col2: now also U1.3 (PC14/OSC32_IN)
- net Col3: now also U1.4 (PC15/OSC32_OUT)
- net Col4: now also U1.11 (PA1)
- net Col5: now also U1.12 (PA2)
- net Col6: now also U1.13 (PA3); no longer U1.15 (DAC1-OUT2/PA5)
- net Col7: now also U1.15 (DAC1-OUT2/PA5); no longer U1.2 (PC13)
- net Col8: now also U1.14 (DAC1-OUT1/PA4); no longer U1.21 (PB10)
- net Col9: now also U1.16 (PA6)
- net LED_PWM: now also U1.22 (PB11); no longer U1.46 (I2C1_SDA/PB9)
- net RGB_PWM: now also U1.17 (PA7); no longer U1.19 (PB1)
- net Row1: now also U1.38 (I2C1_SCL/JTDI/PA15)
- net Row3: now also U1.21 (PB10); no longer U1.22 (PB11)
Changed lines of the file:
@@
 Wire Wire Line
 	3475 10800 4125 10800
-Text GLabel 15375 6875 2    50   Output ~ 0
+Text GLabel 15375 6625 2    50   Output ~ 0
 LED_PWM
 Wire Wire Line
-	15375 6875 15300 6875
+	15375 6625 15300 6625
 Text GLabel 2825 9100 1    50   Input ~ 0
 5V
@@
 Wire Wire Line
 	2825 10050 2825 10100
-Text GLabel 15375 8175 2    50   Output ~ 0
+Text GLabel 15400 8425 2    50   Output ~ 0
 RGB_PWM
-Wire Wire Line
-	15375 8175 15300 8175
 Text GLabel 2475 9525 0    50   Input ~ 0
 RGB_PWM
@@
 3.3V
 Text GLabel 15375 9275 2    50   Input ~ 0
-Col7
+Col1
 Wire Wire Line
 	15375 9275 15300 9275
-Text GLabel 15375 6625 2    50   Input ~ 0
+Text GLabel 15375 6725 2    50   Input ~ 0
 Row3
 Text GLabel 15375 7875 2    50   Input ~ 0
@@
 	15375 8075 15300 8075
 Wire Wire Line
-	15375 6625 15300 6625
-Text GLabel 15375 9275 2    50   Input ~ 0
+	15375 6725 15300 6725
+Text GLabel 15375 8625 2    50   Input ~ 0
 Col7
-Text GLabel 15375 8625 2    50   Input ~ 0
-Col6
 Wire Wire Line
 	15375 8625 15300 8625
-Text GLabel 15375 6725 2    50   Input ~ 0
-Col8
-Wire Wire Line
-	15375 6725 15300 6725
 Text GLabel 15375 6525 2    50   Input ~ 0
 Col11
@@
 Wire Wire Line
 	15375 7225 15300 7225
+Text GLabel 13050 7925 0    50   Input ~ 0
+Col2
+Wire Wire Line
+	13050 7925 13100 7925
+Text GLabel 13050 8025 0    50   Input ~ 0
+Col3
+Wire Wire Line
+	13050 8025 13100 8025
+Text GLabel 15375 9025 2    50   Input ~ 0
+Col4
+Wire Wire Line
+	15375 9025 15300 9025
+Text GLabel 15375 8925 2    50   Input ~ 0
+Col5
+Wire Wire Line
+	15375 8925 15300 8925
+Text GLabel 15375 8825 2    50   Input ~ 0
+Col6
+Wire Wire Line
+	15375 8825 15300 8825
+Text GLabel 15375 8725 2    50   Input ~ 0
+Col8
+Wire Wire Line
+	15375 8725 15300 8725
+Text GLabel 15375 8525 2    50   Input ~ 0
+Col9
+Wire Wire Line
+	15375 8525 15300 8525
+Text GLabel 15375 7125 2    50   Input ~ 0
+Row1
+Wire Wire Line
+	15375 7125 15300 7125
+Wire Wire Line
+	15400 8425 15300 8425
 $EndSCHEMATC

Commit message: Finished design and added BOM
Parts:
- H12: footprint Connector_Pin:Pin_D1.0mm_L10.0mm -> MountingHole:MountingHole_2.2mm_M2_Pad_Via
- RL1, RL10, RL11, RL12, RL13, RL14, RL15, RL16, RL17, RL18, RL19, RL2, RL20, RL21, RL22, RL23, RL24, RL25, RL26, RL27, RL28, RL29, RL3, RL30, RL31, RL32, RL33, RL34, RL35, RL36, RL37, RL38, RL39, RL40, RL41, RL42, RL43, RL44, RL45, RL46, RL47, RL48, RL5, RL6, RL7, RL8, RL9: value R_LED -> 360
- RSGate1: value 1k -> 100

Commit message: Change CVBus4 package to 0402
Parts:
- CVBus4: footprint Capacitor_SMD:C_0805_2012Metric_Pad1.15x1.40mm_HandSolder -> Capacitor_SMD:C_0402_1005Metric
Changed lines of the file:
@@
 F 0 "CVBus4" H 11642 8806 31  0000 L CNN
 F 1 "1u" H 11642 8744 31  0000 L CNN
-F 2 "Capacitor_SMD:C_0805_2012Metric_Pad1.15x1.40mm_HandSolder" H 11550 8775 50  0001 C CNN
+F 2 "Capacitor_SMD:C_0402_1005Metric" H 11550 8775 50  0001 C CNN
 F 3 "~" H 11550 8775 50  0001 C CNN
 	1    11550 8775

Commit message: Added OSH logo
Parts:
- added L3: OSHLogo, sharkLogo:osh-logo, symbol Mechanical:MountingHole
- added L4: BrazilianFlag, sharkLogo:brazilFlag, symbol Mechanical:MountingHole
Changed lines of the file:
@@
 Wire Wire Line
 	15400 8425 15300 8425
+$Comp
+L Mechanical:MountingHole L3
+U 1 1 5C66B5D5
+P 14625 3975
+F 0 "L3" H 14725 4021 50  0000 L CNN
+F 1 "OSHLogo" H 14725 3930 50  0000 L CNN
+F 2 "sharkLogo:osh-logo" H 14625 3975 50  0001 C CNN
+F 3 "~" H 14625 3975 50  0001 C CNN
+	1    14625 3975
+	1    0    0    -1
+$EndComp
+$Comp
+L Mechanical:MountingHole L4
+U 1 1 5C66D4A4
+P 14625 4200
+F 0 "L4" H 14725 4246 50  0000 L CNN
+F 1 "BrazilianFlag" H 14725 4155 50  0000 L CNN
+F 2 "sharkLogo:brazilFlag" H 14625 4200 50  0001 C CNN
+F 3 "~" H 14625 4200 50  0001 C CNN
+	1    14625 4200
+	1    0    0    -1
+$EndComp
 $EndSCHEMATC

Commit message: Added OSH logo
Parts:
- removed H10, H11, H7, H8, H9: MountingHole, MountingHole:MountingHole_2.5mm_Pad, symbol Mechanical:MountingHole
Changed lines of the file:
@@
 Wire Wire Line
 	14850 4950 15050 4950
-$Comp
-L Mechanical:MountingHole H7
-U 1 1 5D038FCF
-P 14625 2500
-F 0 "H7" H 14725 2546 50  0000 L CNN
-F 1 "MountingHole" H 14725 2455 50  0000 L CNN
-F 2 "MountingHole:MountingHole_2.5mm_Pad" H 14625 2500 50  0001 C CNN
-F 3 "~" H 14625 2500 50  0001 C CNN
-	1    14625 2500
-	1    0    0    -1
-$EndComp
-$Comp
-L Mechanical:MountingHole H8
-U 1 1 5D03B7BC
-P 14625 2700
-F 0 "H8" H 14725 2746 50  0000 L CNN
-F 1 "MountingHole" H 14725 2655 50  0000 L CNN
-F 2 "MountingHole:MountingHole_2.5mm_Pad" H 14625 2700 50  0001 C CNN
-F 3 "~" H 14625 2700 50  0001 C CNN
-	1    14625 2700
-	1    0    0    -1
-$EndComp
-$Comp
-L Mechanical:MountingHole H9
-U 1 1 5D03B8D6
-P 14625 2900
-F 0 "H9" H 14725 2946 50  0000 L CNN
-F 1 "MountingHole" H 14725 2855 50  0000 L CNN
-F 2 "MountingHole:MountingHole_2.5mm_Pad" H 14625 2900 50  0001 C CNN
-F 3 "~" H 14625 2900 50  0001 C CNN
-	1    14625 2900
-	1    0    0    -1
-$EndComp
-$Comp
-L Mechanical:MountingHole H10
-U 1 1 5C00FDC2
-P 14625 3100
-F 0 "H10" H 14725 3146 50  0000 L CNN
-F 1 "MountingHole" H 14725 3055 50  0000 L CNN
-F 2 "MountingHole:MountingHole_2.5mm_Pad" H 14625 3100 50  0001 C CNN
-F 3 "~" H 14625 3100 50  0001 C CNN
-	1    14625 3100
-	1    0    0    -1
-$EndComp
-$Comp
-L Mechanical:MountingHole H11
-U 1 1 5C00FEDC
-P 14625 3300
-F 0 "H11" H 14725 3346 50  0000 L CNN
-F 1 "MountingHole" H 14725 3255 50  0000 L CNN
-F 2 "MountingHole:MountingHole_2.5mm_Pad" H 14625 3300 50  0001 C CNN
-F 3 "~" H 14625 3300 50  0001 C CNN
-	1    14625 3300
-	1    0    0    -1
-$EndComp
 Wire Wire Line
 	5725 4325 6725 4325

Commit message: Added US and BR flags, rounded corners
Parts:
- added L5: usFlag, sharkLogo:usFlag, symbol Mechanical:MountingHole
- SWRST1: footprint Button_Switch_SMD:SW_SPST_SKQG_WithoutStem -> smdPushBtn:smdPushBtn
- Y1: footprint Crystal:Crystal_SMD_5032-4Pin_5.0x3.2mm -> crystal:Crystal_SMD_5032-4Pin_5.0x3.2mm
Changed lines of the file:
@@
 Sheet 1 1
 Title "SharkPCB"
-Date "2019-01-13"
-Rev "Rev 3.0.4"
+Date "2019-02-13"
+Rev "Rev 3.0.7"
 Comp "Gondolin Electronics"
 Comment1 ""
@@
 F 0 "SWRST1" H 6075 8950 31  0000 C CNN
 F 1 "SW_Push" H 6075 8929 31  0001 C CNN
-F 2 "Button_Switch_SMD:SW_SPST_SKQG_WithoutStem" H 6075 8950 50  0001 C CNN
+F 2 "smdPushBtn:smdPushBtn" H 6075 8950 50  0001 C CNN
 F 3 "" H 6075 8950 50  0001 C CNN
 	1    6075 8750
@@
 F 0 "Y1" H 14775 5225 50  0000 L CNN
 F 1 "8MHz" H 14750 5150 50  0000 L CNN
-F 2 "Crystal:Crystal_SMD_5032-4Pin_5.0x3.2mm" H 14700 4950 50  0001 C CNN
+F 2 "crystal:Crystal_SMD_5032-4Pin_5.0x3.2mm" H 14700 4950 50  0001 C CNN
 F 3 "~" H 14700 4950 50  0001 C CNN
 	1    14700 4950
@@
 	1    0    0    -1
 $EndComp
+$Comp
+L Mechanical:MountingHole L5
+U 1 1 5C6AAB95
+P 15375 4200
+F 0 "L5" H 15475 4246 50  0000 L CNN
+F 1 "usFlag" H 15475 4155 50  0000 L CNN
+F 2 "sharkLogo:usFlag" H 15375 4200 50  0001 C CNN
+F 3 "~" H 15375 4200 50  0001 C CNN
+	1    15375 4200
+	1    0    0    -1
+$EndComp
