File: shark.kicad_pcb (KiCad board)
At the start: 2 copper layers, 225.6 x 75.4 mm, 253 parts, among them J1 USB_C_Receptacle, Q1 AO4406AL, SW1 MXSwitch, SW10 MXSwitch, SW11 MXSwitch, SW12 MXSwitch, SW13 MXSwitch, SW14 MXSwitch, SW15 MXSwitch, SW16 MXSwitch, SW17 MXSwitch, SW18 MXSwitch, SW19 MXSwitch, SW2 MXSwitch, SW20 MXSwitch, SW21 MXSwitch, SW22 MXSwitch, SW23 MXSwitch, SW24 MXSwitch, SW25 MXSwitch, SW26 MXSwitch, SW27 MXSwitch, SW28 MXSwitch, SW29 MXSwitch, SW3 MXSwitch, SW30 MXSwitch, SW31 MXSwitch, SW32 MXSwitch, SW33 MXSwitch, SW34 MXSwitch, SW35 MXSwitch, SW36 MXSwitch, SW37 MXSwitch, SW38 MXSwitch, SW39 MXSwitch, SW4 MXSwitch, SW40 MXSwitch, SW41 MXSwitch, SW42 MXSwitch, SW43 MXSwitch, SW44 MXSwitch, SW45 MXSwitch, SW46 MXSwitch, SW47 MXSwitch, SW48 MXSwitch, SW49 MXSwitch, SW5 MXSwitch, SW50 MXSwitch, SW51 MXSwitch, SW6 MXSwitch, SW7 MXSwitch, SW8 MXSwitch, SW9 MXSwitch, U1 STM32F303CCT7, U2 MCP1700-3302E_SOT23, Y1 8MHz

Commit message: Started rounting
Parts:
- moved RL11 28.0 mm to (242.3, 74.2), turned to 90 degrees
- moved D33 12.6 mm to (204.3, 112.2), turned to 270 degrees
- moved RL34 11.9 mm to (206.7, 112.2), turned to 270 degrees
- moved RL43 9.08 mm to (168.1, 121.7), turned to 270 degrees
- moved D45 2.53 mm to (204.3, 131.2), turned to 270 degrees
- moved RL45 2.24 mm to (206.7, 131.2)
- moved D11 1.19 mm to (244.7, 74.2), turned to 270 degrees
- moved RL48 0.56 mm to (244.7, 131.2)
- moved RL24 0.55 mm to (244.7, 93.2)
- moved RL23 0.50 mm to (225.7, 93.2)
- moved LED48 0.29 mm to (253.0, 136.3)
- moved LED1 0.29 mm to (44.0, 79.3)
- moved LED37 0.29 mm to (44.0, 136.3)
- moved LED24 0.28 mm to (253.0, 98.3)
- moved LED13 0.28 mm to (44.0, 98.3)
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Routing:
- net Net-(LED1-PadK): track 0.00 -> 957.4 mm
- net Row1: track 0.00 -> 267.5 mm
- net Row2: track 0.00 -> 154.5 mm
- net Col2: track 0.00 -> 74.8 mm
- net Col1: track 0.00 -> 73.4 mm
- net Col12: track 0.00 -> 67.7 mm
- net Col11: track 0.00 -> 62.0 mm
- net Col6: track 0.00 -> 30.1 mm
- net Row3: track 0.00 -> 25.7 mm
- net Net-(LED43-PadA): track 0.00 -> 23.5 mm
- net Net-(LED20-PadA): track 0.00 -> 21.4 mm
- net Col9: track 0.00 -> 19.5 mm
- net Col4: track 0.00 -> 19.2 mm
- net Col3: track 0.00 -> 18.9 mm
- net Net-(LED13-PadA): track 0.00 -> 17.8 mm
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
Commit message: Continued routing
Parts:
- moved RL42 30.9 mm to (131.8, 121.7), turned to 270 degrees
- moved RL41 28.5 mm to (129.5, 121.7), turned to 270 degrees
- moved RL44 21.0 mm to (165.7, 120.0), turned to 270 degrees
- moved F1 1.27 mm to (226.2, 77.3)
- moved RD+Up1 1.19 mm to (226.2, 76.9)
- turned D32 to 90 degrees
- turned D33 to 90 degrees
- turned D34 to 90 degrees
- turned RGB4 to 180 degrees
Routing:
- net Row4: track 12.9 -> 248.7 mm
- net Row3: track 25.7 -> 256.0 mm
- net Net-(J1-PadA7): track 13.8 -> 170.2 mm, vias 0 -> 2
- net Net-(J1-PadA6): track 7.76 -> 157.0 mm, vias 0 -> 2
- net Net-(LED1-PadK): track 957.4 -> 1098.4 mm
- net Row2: track 154.5 -> 275.9 mm
- net Col8: track 0.00 -> 107.1 mm
- net Col7: track 9.99 -> 96.6 mm
- net Col5: track 10.1 -> 86.3 mm
- net LED_PWM: track 1.59 -> 59.1 mm
- net Col10: track 10.6 -> 60.2 mm
- net Col6: track 30.1 -> 75.0 mm
- net Col9: track 19.5 -> 58.8 mm
- net Col4: track 19.2 -> 58.5 mm
- net Col3: track 18.9 -> 57.5 mm
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