File: shark.kicad_pcb (KiCad board)
At the start: 2 copper layers, 225.6 x 75.4 mm, 253 parts, among them J1 USB_C_Receptacle, Q1 AO4406AL, SW1 MXSwitch, SW10 MXSwitch, SW11 MXSwitch, SW12 MXSwitch, SW13 MXSwitch, SW14 MXSwitch, SW15 MXSwitch, SW16 MXSwitch, SW17 MXSwitch, SW18 MXSwitch, SW19 MXSwitch, SW2 MXSwitch, SW20 MXSwitch, SW21 MXSwitch, SW22 MXSwitch, SW23 MXSwitch, SW24 MXSwitch, SW25 MXSwitch, SW26 MXSwitch, SW27 MXSwitch, SW28 MXSwitch, SW29 MXSwitch, SW3 MXSwitch, SW30 MXSwitch, SW31 MXSwitch, SW32 MXSwitch, SW33 MXSwitch, SW34 MXSwitch, SW35 MXSwitch, SW36 MXSwitch, SW37 MXSwitch, SW38 MXSwitch, SW39 MXSwitch, SW4 MXSwitch, SW40 MXSwitch, SW41 MXSwitch, SW42 MXSwitch, SW43 MXSwitch, SW44 MXSwitch, SW45 MXSwitch, SW46 MXSwitch, SW47 MXSwitch, SW48 MXSwitch, SW49 MXSwitch, SW5 MXSwitch, SW50 MXSwitch, SW51 MXSwitch, SW6 MXSwitch, SW7 MXSwitch, SW8 MXSwitch, SW9 MXSwitch, U1 STM32F303CCT7, U2 MCP1700-3302E_SOT23, Y1 8MHz

Commit message: Proceeded routing
Parts:
- SWRST1: moved to B.Cu
- moved SWRST1 19.0 mm to (224.5, 102.7), turned to 0 degrees
- moved CRST1 7.57 mm to (163.9, 86.7)
- moved L1 3.69 mm to (82.0, 105.7)
- moved RSGate1 3.28 mm to (130.9, 95.0)
- moved RPGate1 2.39 mm to (128.0, 95.0)
- moved C1 0.84 mm to (157.7, 104.5), turned to 180 degrees
- moved C2 0.74 mm to (157.7, 101.0)
- moved Y1 0.47 mm to (153.5, 102.7)
Connections:
- U1 pad 10: Col7 -> (no net)
- U1 pad 2: Row2 -> Col7
- U1 pad 39: (no net) -> Row2
Routing:
- net Col1: track 73.3 -> 201.8 mm
- net Col2: track 73.6 -> 117.9 mm
- net Col3: track 57.5 -> 83.5 mm
- net 3.3V: track 117.2 -> 135.6 mm, vias 6 -> 7
- net Net-(DRST1-Pad2): track 65.0 -> 83.4 mm, vias 0 -> 1
- net Row2: track 301.2 -> 284.7 mm
- net Col4: track 59.4 -> 67.2 mm
- net Col7: track 107.4 -> 114.1 mm
- net NRST: track 30.1 -> 24.8 mm
- net BOOT0: track 10.4 -> 14.2 mm
- net Col11: track 65.0 -> 63.7 mm
- net LED_PWM: track 57.0 -> 55.8 mm
- net Net-(Q1-PadG): track 6.63 -> 7.57 mm
- net Net-(LED1-PadK): track 1108.4 -> 1109.2 mm
- net Net-(J1-PadA7): track 189.6 -> 188.9 mm, vias 2 -> 0
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
Commit message: Changed to SMD changes
Parts:
- CRST1, CSRT2, DRST1, QRST1, RRST1: moved to B.Cu
- D1, D10, D11, D12, D13, D14, D15, D16, D17, D18, D19, D2, D20, D21, D22, D23, D24, D25, D26, D27, D28, D29, D3, D30, D31, D32, D33, D34, D35, D36, D37, D38, D39, D4, D40, D41, D42, D43, D44, D45, D46, D47, D48, D5, D6, D7, D8, D9: footprint Keyboard_switches:thtDiode -> Keyboard_switches:D_SOD-123
- RL1, RL10, RL11, RL12, RL13, RL14, RL15, RL16, RL17, RL18, RL19, RL2, RL20, RL21, RL22, RL23, RL24, RL25, RL26, RL27, RL28, RL29, RL3, RL30, RL31, RL32, RL33, RL34, RL35, RL36, RL37, RL38, RL39, RL4, RL40, RL45, RL46, RL47, RL48, RL5, RL6, RL7, RL8, RL9: footprint Keyboard_switches:Resistor_THT_5.08mm_Horizontal -> Resistor_SMD:R_1206_3216Metric; moved to B.Cu
- RL41, RL42, RL43, RL44: footprint Keyboard_switches:Resistor_THT_5.08mm_Horizontal -> Resistor_SMD:R_1206_3216Metric
- moved CRST1 63.6 mm to (227.4, 90.3)
- moved RRST1 58.8 mm to (224.8, 91.8)
- moved U1 57.0 mm to (224.5, 102.7)
- moved C1 53.7 mm to (211.4, 104.2), turned to 0 degrees
- moved C2 53.7 mm to (211.4, 100.7)
- moved Y1 53.7 mm to (207.2, 102.4)
- moved DRST1 53.4 mm to (222.1, 90.3)
- moved CVBus5 46.4 mm to (228.8, 99.3), turned to 90 degrees
- moved CVBus3 44.3 mm to (226.8, 99.3), turned to 90 degrees
- moved CVBus1 42.4 mm to (224.7, 99.3), turned to 90 degrees
- moved CVBus2 40.5 mm to (222.6, 99.3), turned to 90 degrees
- moved CVBus4 38.8 mm to (220.5, 99.3), turned to 90 degrees
- moved DS1 37.1 mm to (227.4, 103.3)
- moved U2 36.8 mm to (224.2, 103.6)
- moved CSin1 35.9 mm to (225.1, 106.9)
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Connections:
- U1 pad 38: (no net) -> Col11
- U1 pad 39: Row2 -> Col10
- U1 pad 40: (no net) -> Row2
Routing:
- net Net-(LED1-PadK): track 1109.2 -> 44.5 mm
- net Row3: track 268.4 -> 16.9 mm
- net Net-(J1-PadA7): track 188.9 -> 0.00 mm
- net RGB_PWM: track 189.6 -> 1.59 mm
- net Row1: track 262.5 -> 95.0 mm
- net Net-(J1-PadA6): track 156.8 -> 0.00 mm
- net Col1: track 201.8 -> 59.9 mm
- net Col11: track 63.7 -> 146.9 mm, vias 0 -> 1
- net Net-(RGB6-Pad2): track 77.5 -> 0.00 mm
- net 3.3V: track 135.6 -> 60.2 mm, vias 7 -> 5
- net Row4: track 288.3 -> 217.8 mm
- net Net-(RGB1-Pad2): track 69.7 -> 0.00 mm
- net Row2: track 284.7 -> 219.4 mm
- net Net-(RGB3-Pad2): track 65.2 -> 0.00 mm
- net Net-(RGB2-Pad2): track 57.3 -> 0.00 mm
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Other:
- board text added: "CSIn"
- board text removed: "CSI"

Commit message: Added photorealistic renders
Parts:
- removed the L1 at (174.6, 105.7)
- added L2: LogoBack, sharkLogo:skark, B.Cu at (152.6, 113.1)

Commit message: Added Pirulen font to the logo
Parts:
- Q1, RPGate1, RSGate1: moved to B.Cu
- moved RD+1 57.3 mm to (236.3, 101.6)
- moved RD-1 57.3 mm to (236.3, 103.9)
- moved RPGate1 10.1 mm to (131.8, 104.8), turned to 180 degrees
- moved RSGate1 10.1 mm to (131.8, 101.3), turned to 0 degrees
- moved Q1 5.37 mm to (124.1, 102.8), turned to 180 degrees
- moved C7 0.90 mm to (224.8, 66.5)
- moved R5 0.90 mm to (224.8, 68.9)
- moved J1 0.89 mm to (224.8, 72.5)
- moved DF1 0.26 mm to (222.7, 77.9), turned to 270 degrees
- turned RCC1 to 90 degrees
Connections:
- U1 pad 10: (no net) -> Col10
- U1 pad 13: Row4 -> (no net)
- U1 pad 14: Row3 -> (no net)
- U1 pad 20: (no net) -> Row4
- U1 pad 22: Col10 -> Row3
- U1 pad 25: (no net) -> Col11
- U1 pad 31: (no net) -> Col12
- U1 pad 38: Col11 -> (no net)
- U1 pad 39: Col10 -> (no net)
Routing:
- net Col1: track 59.9 -> 223.4 mm
- net Col2: track 101.4 -> 240.4 mm
- net Col3: track 81.2 -> 200.7 mm
- net Col4: track 101.4 -> 202.2 mm
- net Col5: track 90.5 -> 172.1 mm
- net Net-(J1-PadA6): track 0.00 -> 66.2 mm
- net Col6: track 96.8 -> 162.3 mm
- net Net-(J1-PadA7): track 0.00 -> 58.8 mm
- net Row4: track 217.8 -> 273.8 mm
- net Col12: track 92.2 -> 145.2 mm, vias 0 -> 1
- net Row3: track 16.9 -> 60.1 mm
- net Col7: track 86.0 -> 126.4 mm
- net GND: track 7.24 -> 32.6 mm, vias 6 -> 10
- net Net-(LED1-PadK): track 44.5 -> 66.3 mm
- net Col8: track 102.6 -> 123.4 mm
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Other:
- outline, holes or cut-outs redrawn

Commit message: Finished design. Thickening possible traces
Parts:
- added G***: LOGO, sharkLogo:brazilFlag, F.Cu at (167.5, 83.7)
- moved RGB1 151.9 mm to (224.4, 83.4)
- moved RGB4 151.9 mm to (72.5, 83.9), turned to 0 degrees
- moved RGB5 151.4 mm to (223.9, 121.7), turned to 0 degrees
- moved RGB8 151.4 mm to (72.5, 121.7)
- moved RGB2 76.0 mm to (186.5, 83.7)
- moved RGB3 76.0 mm to (110.5, 83.7)
- moved RGB6 76.0 mm to (186.5, 121.7), turned to 0 degrees
- moved RGB7 76.0 mm to (110.5, 121.7)
- moved RPGate1 3.98 mm to (131.5, 100.9), turned to 0 degrees
- moved RSGate1 3.17 mm to (131.5, 104.4), turned to 180 degrees
Connections:
- U1 pad 11: (no net) -> Col4
- U1 pad 12: (no net) -> Col5
- U1 pad 13: (no net) -> Col6
- U1 pad 14: (no net) -> Col8
- U1 pad 15: Col6 -> Col7
- U1 pad 16: (no net) -> Col9
- U1 pad 17: (no net) -> RGB_PWM
- U1 pad 19: RGB_PWM -> (no net)
- U1 pad 2: Col7 -> Col1
- U1 pad 21: Col8 -> Row3
- U1 pad 22: Row3 -> LED_PWM
- U1 pad 3: (no net) -> Col2
- U1 pad 38: (no net) -> Row1
- U1 pad 4: (no net) -> Col3
- U1 pad 46: LED_PWM -> (no net)
Routing:
- net Net-(LED1-PadK): track 66.3 -> 1120.0 mm, vias 0 -> 1
- net Row1: track 95.0 -> 256.4 mm, vias 0 -> 1
- net Row3: track 60.1 -> 212.6 mm, vias 1 -> 2
- net LED_PWM: track 2.48 -> 147.7 mm
- net GND: track 32.6 -> 155.4 mm, vias 10 -> 12
- net Net-(RGB6-Pad2): track 0.00 -> 81.9 mm
- net Net-(RGB2-Pad2): track 0.00 -> 72.5 mm
- net Col9: track 80.9 -> 130.5 mm, vias 0 -> 1
- net Net-(RGB7-Pad2): track 0.00 -> 47.6 mm
- net RGB_PWM: track 1.59 -> 45.6 mm
- net Col8: track 123.4 -> 159.9 mm, vias 1 -> 2
- net Net-(RGB3-Pad2): track 0.00 -> 36.6 mm
- net Net-(RGB1-Pad2): track 0.00 -> 36.3 mm
- net Net-(RGB5-Pad2): track 0.00 -> 35.5 mm
- net Col1: track 223.4 -> 258.6 mm, vias 0 -> 1
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
Commit message: Finished design and added BOM
Parts:
- H12: footprint Connector_Pin:Pin_D1.0mm_L10.0mm -> MountingHole:MountingHole_2.2mm_M2_Pad_Via
- moved H12 0.33 mm to (39.5, 103.6)
Routing:
- net Col1: track 258.6 -> 263.8 mm
- net Net-(LED1-PadK): track 1120.0 -> 1122.3 mm
- net Net-(LED35-PadA): track 16.3 -> 15.4 mm
- net Net-(RGB6-Pad2): track 81.9 -> 81.2 mm
- net Net-(LED12-PadA): track 9.76 -> 9.03 mm

Commit message: Change CVBus4 package to 0402
Parts:
- CVBus4: footprint Capacitor_SMD:C_0805_2012Metric_Pad1.15x1.40mm_HandSolder -> Capacitor_SMD:C_0402_1005Metric
- RL1, RL10, RL11, RL12, RL13, RL14, RL15, RL16, RL17, RL18, RL19, RL2, RL20, RL21, RL22, RL23, RL24, RL25, RL26, RL27, RL28, RL29, RL3, RL30, RL31, RL32, RL33, RL34, RL35, RL36, RL37, RL38, RL39, RL40, RL41, RL42, RL43, RL44, RL45, RL46, RL47, RL48, RL5, RL6, RL7, RL8, RL9: value R_LED -> 360
- RSGate1: value 1k -> 100
- moved CVBus4 0.38 mm to (220.9, 99.3)
Routing:
- net 3.3V: track 71.2 -> 72.0 mm
