File: shark.kicad_pcb (KiCad board)
At the start: 2 copper layers, 225.6 x 75.4 mm, 254 parts, among them J1 USB_C_Receptacle, Q1 AO4406AL, SW1 MXSwitch, SW10 MXSwitch, SW11 MXSwitch, SW12 MXSwitch, SW13 MXSwitch, SW14 MXSwitch, SW15 MXSwitch, SW16 MXSwitch, SW17 MXSwitch, SW18 MXSwitch, SW19 MXSwitch, SW2 MXSwitch, SW20 MXSwitch, SW21 MXSwitch, SW22 MXSwitch, SW23 MXSwitch, SW24 MXSwitch, SW25 MXSwitch, SW26 MXSwitch, SW27 MXSwitch, SW28 MXSwitch, SW29 MXSwitch, SW3 MXSwitch, SW30 MXSwitch, SW31 MXSwitch, SW32 MXSwitch, SW33 MXSwitch, SW34 MXSwitch, SW35 MXSwitch, SW36 MXSwitch, SW37 MXSwitch, SW38 MXSwitch, SW39 MXSwitch, SW4 MXSwitch, SW40 MXSwitch, SW41 MXSwitch, SW42 MXSwitch, SW43 MXSwitch, SW44 MXSwitch, SW45 MXSwitch, SW46 MXSwitch, SW47 MXSwitch, SW48 MXSwitch, SW49 MXSwitch, SW5 MXSwitch, SW50 MXSwitch, SW51 MXSwitch, SW6 MXSwitch, SW7 MXSwitch, SW8 MXSwitch, SW9 MXSwitch, U1 STM32F303CCT7, U2 MCP1700-3302E_SOT23, Y1 8MHz

Commit message: Added OSH logo
Parts:
- removed G***: LOGO, sharkLogo:brazilFlag
- added L3: OSHLogo, sharkLogo:osh-logo, F.Cu at (174.1, 102.9)
- added L4: BrazilianFlag, sharkLogo:brazilFlag, F.Cu at (167.5, 83.7)
- moved J1 0.30 mm to (224.5, 72.5)
- moved H10 0.25 mm to (243.5, 83.7)
- moved H5 0.25 mm to (243.5, 102.7)
Other:
- board size 225.6 x 75.4 mm -> 225.6 x 75.3 mm

Commit message: Added OSH logo
Parts:
- removed H10, H11, H7, H8, H9: MountingHole, MountingHole:MountingHole_2.5mm_Pad
- moved L4 2.13 mm to (165.5, 84.6)
Routing:
- net Col6: track 196.3 -> 193.5 mm
- net Col5: track 203.9 -> 204.4 mm
Other:
- outline, holes or cut-outs redrawn

Commit message: Added US and BR flags, rounded corners
Parts:
- removed the Y1 at (207.2, 102.4)
- added L5: usFlag, sharkLogo:usFlag, F.Cu at (166.3, 103.6)
- added Y1 (x2): 8MHz, crystal:Crystal_SMD_5032-4Pin_5.0x3.2mm, F.Cu at (207.2, 102.4)
- SWRST1: footprint Button_Switch_SMD:SW_SPST_SKQG_WithoutStem -> smdPushBtn:smdPushBtn
- moved L3 1.05 mm to (173.1, 103.0)
- moved L4 0.80 mm to (166.3, 84.9)
- moved RGB5 0.59 mm to (224.5, 121.7)
- moved C7 0.30 mm to (224.8, 66.8)
- moved J1 0.30 mm to (224.5, 72.8)
- moved R5 0.30 mm to (224.8, 69.2)
- turned RGB7 to 0 degrees
- turned RGB8 to 0 degrees
Routing:
- net Net-(RGB7-Pad2): track 47.6 -> 36.8 mm
- net Net-(RGB6-Pad2): track 81.2 -> 74.9 mm
- net Net-(LED1-PadK): track 1122.3 -> 1119.4 mm
- net Net-(J1-PadA6): track 65.6 -> 64.0 mm
- net XTAL1: track 17.8 -> 19.5 mm
- net 3.3V: track 72.0 -> 73.5 mm
- net RGB_PWM: track 45.6 -> 46.8 mm
- net Net-(J1-PadA7): track 58.9 -> 58.2 mm
- net Net-(DRST1-Pad2): track 56.3 -> 56.9 mm
Other:
- board size 225.6 x 75.3 mm -> 225.6 x 74.8 mm
- net class Default: clearance 0.13 -> 0.127
- net class Fine: clearance 0.13 -> 0.127
- rule trace_clearance: 0.13 -> 0.127
- board text added: "FG/1S"
- board text added: "GondolinElectronics UndecidedSharkPCB v3.0.7 "I like the nick 'Shark', but I'm so undecided" Shark illustration by Yohan Plantec at vectorportal.com"
- board text removed: "GondolinElectronics UndecidedSharkPCB v3.0 "I like the nick 'Shark', but I'm so undecided" Shark illustration by Yohan Plantec at vectorportal.com"

Commit message: Added rotary encoder support
Parts:
- removed the Y1 at (207.2, 102.4) (x2)
- added CA1: 10n, Capacitor_SMD:C_0805_2012Metric_Pad1.15x1.40mm_HandSolder, B.Cu at (87.3, 100.7)
- added CB1: 10n, Capacitor_SMD:C_0805_2012Metric_Pad1.15x1.40mm_HandSolder, B.Cu at (87.3, 103.9)
- added RA1: 10k, Resistor_SMD:R_1206_3216Metric_Pad1.42x1.75mm_HandSolder, B.Cu at (82.7, 103.9)
- added RA2: 10k, Resistor_SMD:R_1206_3216Metric_Pad1.42x1.75mm_HandSolder, B.Cu at (77.5, 103.9)
- added RB1: 10k, Resistor_SMD:R_1206_3216Metric_Pad1.42x1.75mm_HandSolder, B.Cu at (82.7, 100.9)
- added RB2: 10k, Resistor_SMD:R_1206_3216Metric_Pad1.42x1.75mm_HandSolder, B.Cu at (77.5, 100.9)
- added ROT1: Rotary_Encoder_Switch, encoders:ALPS_EC11E, F.Cu at (44.0, 131.2)
- added Y1 (x2): 8MHz, crystal:Crystal_SMD_5032-4Pin_5.0x3.2mm, F.Cu at (207.2, 102.4)
- moved D37 0.59 mm to (52.9, 131.2)
- moved D38 0.59 mm to (55.2, 131.2)
- moved RL37 0.59 mm to (52.9, 131.2)
- moved RL38 0.59 mm to (55.2, 131.2)
Connections:
- net Net-(D37-Pad2) renamed EncS1
- U1 pad 39: (no net) -> EncA
- U1 pad 41: (no net) -> EncB
Routing:
- net EncA: track 0.00 -> 314.2 mm, vias 0 -> 2
- net EncB: track 0.00 -> 313.1 mm, vias 0 -> 2
- net GND: track 155.4 -> 170.8 mm, vias 12 -> 13
- net Col1: track 264.2 -> 279.5 mm
- net Net-(LED1-PadK): track 1119.4 -> 1132.7 mm
- net EncS1: track 4.46 -> 16.5 mm
- net (no net): track 30.3 -> 26.9 mm, vias 15 -> 13
- net Net-(D48-Pad2): track 12.4 -> 14.8 mm
- net Net-(CB1-Pad2): track 0.00 -> 2.27 mm
- net Net-(CA1-Pad2): track 0.00 -> 2.01 mm
- net Col4: track 232.0 -> 233.7 mm
- net VBUS: track 9.64 -> 10.6 mm
Other:
- board text added: "GondolinElectronics UndecidedSharkPCB v3.1 "I like the nick 'Shark', but I'm so undecided" Shark illustration by Yohan Plantec at vectorportal.com"
- board text removed: "GondolinElectronics UndecidedSharkPCB v3.0.7 "I like the nick 'Shark', but I'm so undecided" Shark illustration by Yohan Plantec at vectorportal.com"

Commit message: Edited gerbers
Parts:
- removed the Y1 at (207.2, 102.4) (x2)
- added Y1 (x2): 8MHz, crystal:Crystal_SMD_5032-4Pin_5.0x3.2mm, F.Cu at (207.2, 102.4)
Routing:
- net Net-(LED1-PadK): track 1132.7 -> 1131.8 mm
Changed lines of the file:
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@@
     (thickness 1.6)
     (drawings 440)
-    (tracks 1809)
+    (tracks 1808)
     (zones 0)
     (modules 259)
@@
   (segment (start 64.1505 78.696125) (end 64.1505 78.993) (width 0.254) (layer F.Cu) (net 72) (status 30))
   (segment (start 197.1505 115.8055) (end 197.1505 116.696125) (width 0.5) (layer F.Cu) (net 72) (status 20))
-  (segment (start 216.233 117.323) (end 216.233 116.461) (width 0.5) (layer F.Cu) (net 72) (status 10))
   (segment (start 159.1505 116.993) (end 158.853625 116.993) (width 0.254) (layer F.Cu) (net 72) (status 30))
   (segment (start 235.233 117.323) (end 246.168 117.323) (width 1) (layer F.Cu) (net 72) (status 10))
@@
   (segment (start 121.12233 104.676825) (end 121.12233 100.990575) (width 1) (layer B.Cu) (net 72) (status 30))
   (via (at 121.39108 104.676825) (size 1) (drill 0.5) (layers F.Cu B.Cu) (net 72) (status 30))
-  (segment (start 216.233 117.323) (end 216.233 116.461) (width 0.254) (layer B.Cu) (net 72) (status 10))
   (segment (start 245.24425 131.243) (end 241.68175 131.243) (width 0.254) (layer F.Cu) (net 72))
   (segment (start 241.68175 131.243) (end 239.30675 133.618) (width 0.254) (layer F.Cu) (net 72))
@@
   (segment (start 135.4005 99.77425) (end 139.853625 99.77425) (width 0.7) (layer F.Cu) (net 72))
   (segment (start 133.94925 98.323) (end 135.4005 99.77425) (width 0.7) (layer F.Cu) (net 72))
-  (segment (start 216.233 116.461) (end 215.874375 116.102375) (width 0.5) (layer F.Cu) (net 72))
   (segment (start 159.1505 115.78125) (end 159.1505 117.289875) (width 0.5) (layer F.Cu) (net 72) (status 20))
   (segment (start 141.882 115.78125) (end 159.1505 115.78125) (width 0.5) (layer F.Cu) (net 72))
@@
   (segment (start 65.021073 137.111073) (end 65.021073 137.136198) (width 0.254) (layer F.Cu) (net 72))
   (segment (start 85.228625 100.071125) (end 102.125 100.071125) (width 0.7) (layer F.Cu) (net 72))
-  (segment (start 215.55325 115.78125) (end 215.874375 116.102375) (width 0.5) (layer F.Cu) (net 72))
   (segment (start 120.259875 100.071125) (end 121.1505 99.1805) (width 0.7) (layer F.Cu) (net 72))
   (segment (start 178.233 117.34747) (end 178.233 115.80572) (width 0.5) (layer F.Cu) (net 72))
   (segment (start 159.1505 115.78125) (end 178.233 115.78125) (width 0.5) (layer F.Cu) (net 72))
   (segment (start 178.233 115.78125) (end 215.55325 115.78125) (width 0.5) (layer F.Cu) (net 72))
+  (segment (start 215.55325 115.78125) (end 215.83029 115.78125) (width 0.5) (layer F.Cu) (net 72))
+  (segment (start 215.83029 115.78125) (end 216.44852 116.39948) (width 0.5) (layer F.Cu) (net 72))
+  (segment (start 216.44852 116.39948) (end 216.44852 116.99324) (width 0.5) (layer F.Cu) (net 72))
   (segment (start 55.24425 76.368) (end 58.463 79.58675) (width 1) (layer B.Cu) (net 73))
   (segment (start 55.24425 75.643) (end 55.24425 76.368) (width 1) (layer B.Cu) (net 73) (status 10))

Commit message: Fixed little problem with edge cuts
Parts:
- removed the Y1 at (207.2, 102.4) (x2)
- added Y1 (x2): 8MHz, crystal:Crystal_SMD_5032-4Pin_5.0x3.2mm, F.Cu at (207.2, 102.4)
Other:
- outline, holes or cut-outs redrawn
Changed lines of the file:
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@@
   (title_block
     (title SharkPCB)
-    (date 2019-02-20)
-    (rev V3.1)
+    (date 2019-02-27)
+    (rev V3.1.1)
     (company "Gondolin Electronics")
   )
@@
     )
   )
+  (gr_arc (start 255.27 72.263) (end 261.239 72.263) (angle -90) (layer Edge.Cuts) (width 0.15))
+  (gr_arc (start 230.124 65.659) (end 229.489 65.659) (angle -90) (layer Edge.Cuts) (width 0.15))
+  (gr_arc (start 228.854 65.151) (end 229.489 65.151) (angle -90) (layer Edge.Cuts) (width 0.15))
+  (gr_arc (start 220.091 65.151) (end 220.091 64.516) (angle -90) (layer Edge.Cuts) (width 0.15))
+  (gr_arc (start 218.821 65.659) (end 218.821 66.294) (angle -90) (layer Edge.Cuts) (width 0.15))
+  (gr_arc (start 41.656 72.263) (end 41.656 66.294) (angle -90) (layer Edge.Cuts) (width 0.15))
+  (gr_arc (start 41.656 133.35) (end 35.687 133.35) (angle -90) (layer Edge.Cuts) (width 0.15))
   (gr_text FG/1S (at 176.963 128.27425) (layer F.SilkS)
     (effects (font (size 0.75 0.75) (thickness 0.1875)))
@@
     (effects (font (size 0.8 0.8) (thickness 0.2)) (justify mirror))
   )
-  (gr_arc (start 41.588 72.164751) (end 41.588 66.227251) (angle -90) (layer Edge.Cuts) (width 0.15))
-  (gr_arc (start 41.588 133.321125) (end 35.6505 133.321125) (angle -90) (layer Edge.Cuts) (width 0.15))
-  (gr_arc (start 255.338 133.321125) (end 255.338 139.258625) (angle -90) (layer Edge.Cuts) (width 0.15))
-  (gr_arc (start 255.338 72.164875) (end 261.2755 72.164875) (angle -90) (layer Edge.Cuts) (width 0.15))
+  (gr_arc (start 255.27 133.35) (end 255.27 139.319) (angle -90) (layer Edge.Cuts) (width 0.15))
   (gr_circle (center 243.46332 121.743064) (end 246.330134 121.743064) (layer Edge.Cuts) (width 0.15))
   (gr_circle (center 243.46332 83.742936) (end 246.330134 83.742936) (layer Edge.Cuts) (width 0.15))
@@
   (gr_line (start 49.30675 67.118) (end 51.088 67.118) (layer F.SilkS) (width 0.15))
   (gr_line (start 51.088 67.118) (end 51.088 68.89925) (layer F.SilkS) (width 0.15))
-  (gr_line (start 220.009875 64.446125) (end 228.916396 64.445995) (layer Edge.Cuts) (width 0.15))
-  (gr_line (start 219.416125 65.633625) (end 219.416125 65.039875) (layer Edge.Cuts) (width 0.15))
-  (gr_arc (start 228.916398 65.039747) (end 229.510148 65.039747) (angle -90) (layer Edge.Cuts) (width 0.15))
-  (gr_arc (start 230.103623 65.633625) (end 229.509873 65.633625) (angle -90) (layer Edge.Cuts) (width 0.15))
-  (gr_arc (start 220.009875 65.039875) (end 220.009875 64.446125) (angle -90) (layer Edge.Cuts) (width 0.15))
-  (gr_arc (start 218.822612 65.633501) (end 218.822612 66.227251) (angle -90) (layer Edge.Cuts) (width 0.15))
+  (gr_line (start 220.091 64.516) (end 228.854 64.516) (layer Edge.Cuts) (width 0.15))
+  (gr_line (start 219.456 65.659) (end 219.456 65.151) (layer Edge.Cuts) (width 0.15))
   (gr_line (start 68.988926 93.118786) (end 68.988926 94.706286) (layer F.SilkS) (width 0.254))
   (gr_line (start 68.988926 94.706286) (end 67.401426 94.706286) (layer F.SilkS) (width 0.254))
-  (gr_line (start 229.509873 65.633625) (end 229.509873 65.039875) (layer Edge.Cuts) (width 0.15))
+  (gr_line (start 229.489 65.659) (end 229.489 65.151) (layer Edge.Cuts) (width 0.15))
   (gr_text "Surge\nprotection" (at 224.463 81.96175) (layer B.SilkS)
     (effects (font (size 0.508 0.508) (thickness 0.127)) (justify mirror))
@@
     (effects (font (size 0.508 0.508) (thickness 0.0762)))
   )
-  (gr_line (start 35.6505 133.321125) (end 35.6505 72.164875) (layer Edge.Cuts) (width 0.15))
-  (gr_line (start 255.338 139.258625) (end 41.588 139.258625) (layer Edge.Cuts) (width 0.15))
-  (gr_line (start 261.2755 72.164875) (end 261.2755 133.321125) (layer Edge.Cuts) (width 0.15))
+  (gr_line (start 35.687 133.35) (end 35.687 72.263) (layer Edge.Cuts) (width 0.15))
+  (gr_line (start 255.27 139.319) (end 41.656 139.319) (layer Edge.Cuts) (width 0.15))
+  (gr_line (start 261.239 72.263) (end 261.239 133.35) (layer Edge.Cuts) (width 0.15))
   (gr_text "GondolinElectronics UndecidedSharkPCB v3.1\n\"I like the nick 'Shark', but I'm so undecided\"\nShark illustration by Yohan Plantec at vectorportal.com" (at 109.2755 102.743) (layer F.SilkS)
     (effects (font (size 0.508 0.508) (thickness 0.0762)))
   )
-  (gr_line (start 230.103623 66.227375) (end 255.338 66.227375) (layer Edge.Cuts) (width 0.15))
-  (gr_line (start 41.588 66.227375) (end 218.822375 66.227375) (layer Edge.Cuts) (width 0.15))
+  (gr_line (start 230.124 66.294) (end 255.27 66.294) (layer Edge.Cuts) (width 0.15))
+  (gr_line (start 41.656 66.294) (end 218.821 66.294) (layer Edge.Cuts) (width 0.15))
   (segment (start 224.213 107.093) (end 224.213 109.571125) (width 0.13) (layer F.Cu) (net 0) (status 10))
   (segment (start 228.813 103.993) (end 231.291125 103.993) (width 0.13) (layer F.Cu) (net 0) (status 10))
