File: plate/fullGrid/fullGrid.kicad_pcb (KiCad board)
At the start: 2 copper layers, 233 x 81 mm, 48 parts

Commit message: Added encoder position and moved push button
Routing:
- net (no net): vias 6 -> 5
Changed lines of the file:
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@@
     (thickness 1.6)
     (drawings 8)
-    (tracks 6)
+    (tracks 5)
     (zones 0)
     (modules 48)
@@
   (via (at 53.4614 83.74268) (size 4) (drill 3) (layers F.Cu B.Cu) (net 0))
   (via (at 148.463 102.743) (size 4) (drill 3) (layers F.Cu B.Cu) (net 0))
-  (via (at 205.46396 102.743) (size 5) (drill 4) (layers F.Cu B.Cu) (net 0))
 )
