File: plate/universal/universal.kicad_pcb (KiCad board)
At the start: 2 copper layers, 233 x 81 mm, 45 parts

Commit message: Added encoder position and moved push button
Routing:
- net (no net): vias 6 -> 5
Changed lines of the file:
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@@
     (thickness 1.6)
     (drawings 8)
-    (tracks 6)
+    (tracks 5)
     (zones 0)
     (modules 45)
@@
   (gr_line (start 33.720426 62.219426) (end 263.205574 62.219426) (layer Edge.Cuts) (width 0.15))
   (via (at 243.4646 83.74268) (size 4) (drill 3) (layers F.Cu B.Cu) (net 0))
-  (via (at 205.46396 102.743) (size 5) (drill 4) (layers F.Cu B.Cu) (net 0))
   (via (at 243.4646 121.74332) (size 4) (drill 3) (layers F.Cu B.Cu) (net 0))
   (via (at 148.463 102.743) (size 4) (drill 3) (layers F.Cu B.Cu) (net 0))
