File: kicadFiles/shark.kicad_pcb (KiCad board)
At the start: 2 copper layers, 225.6 x 74.8 mm, 259 parts, among them J1 USB_C_Receptacle, Q1 AO4406AL, SW1 MXSwitch, SW10 MXSwitch, SW11 MXSwitch, SW12 MXSwitch, SW13 MXSwitch, SW14 MXSwitch, SW15 MXSwitch, SW16 MXSwitch, SW17 MXSwitch, SW18 MXSwitch, SW19 MXSwitch, SW2 MXSwitch, SW20 MXSwitch, SW21 MXSwitch, SW22 MXSwitch, SW23 MXSwitch, SW24 MXSwitch, SW25 MXSwitch, SW26 MXSwitch, SW27 MXSwitch, SW28 MXSwitch, SW29 MXSwitch, SW3 MXSwitch, SW30 MXSwitch, SW31 MXSwitch, SW32 MXSwitch, SW33 MXSwitch, SW34 MXSwitch, SW35 MXSwitch, SW36 MXSwitch, SW37 MXSwitch, SW38 MXSwitch, SW39 MXSwitch, SW4 MXSwitch, SW40 MXSwitch, SW41 MXSwitch, SW42 MXSwitch, SW43 MXSwitch, SW44 MXSwitch, SW45 MXSwitch, SW46 MXSwitch, SW47 MXSwitch, SW48 MXSwitch, SW49 MXSwitch, SW5 MXSwitch, SW50 MXSwitch, SW51 MXSwitch, SW6 MXSwitch, SW7 MXSwitch, SW8 MXSwitch, SW9 MXSwitch, U1 STM32F303CCT7, U2 MCP1700-3302E_SOT23, Y1 8MHz

Commit message: Reorganized folders
Parts:
- removed the Y1 at (207.2, 102.4) (x2)
- added Y1 (x2): 8MHz, acheronComponents:Crystal_SMD_5032-4Pin_5.0x3.2mm, F.Cu at (207.2, 102.4)
- D1, D10, D11, D12, D13, D14, D15, D16, D17, D18, D19, D2, D20, D21, D22, D23, D24, D25, D26, D27, D28, D29, D3, D30, D31, D32, D33, D34, D35, D36, D37, D38, D39, D4, D40, D41, D42, D43, D44, D45, D46, D47, D48, D5, D6, D7, D8, D9: footprint Keyboard_switches:D_SOD-123 -> acheronComponents:D_SOD-123
- J1: footprint USBconnector:TYPE-C-31-M-13 -> acheronConnectors:TYPE-C-31-M-12
- ROT1: footprint encoders:ALPS_EC11E -> acheronHardware:ALPS_EC11E
- SW1, SW10, SW11, SW12, SW13, SW14, SW15, SW16, SW17, SW18, SW19, SW2, SW20, SW21, SW22, SW23, SW24, SW25, SW26, SW27, SW28, SW29, SW3, SW30, SW31, SW32, SW33, SW34, SW35, SW36, SW37, SW38, SW39, SW4, SW40, SW41, SW42, SW43, SW44, SW45, SW46, SW47, SW48, SW5, SW6, SW7, SW8, SW9: footprint Keyboard_switches:MX100 -> acheronKeyboardSwitches:MX100
- SW49, SW50, SW51: footprint Keyboard_switches:MX200R -> acheronKeyboardSwitches:MX200R
Routing:
- net GND: track 170.8 -> 172.5 mm
Other:
- board text added: "GondolinElectronics UndecidedSharkPCB v3.1.2 "I like the nick 'Shark', but I'm so undecided""
- board text removed: "GondolinElectronics UndecidedSharkPCB v3.1 "I like the nick 'Shark', but I'm so undecided" Shark illustration by Yohan Plantec at vectorportal.com"

Commit message: Added encoder position and moved push button
Parts:
- removed the Y1 at (207.2, 102.4) (x2)
- added ROT2: Rotary_Encoder_Switch, acheronHardware:ALPS_EC11E, F.Cu at (253.0, 131.2)
- added Y1 (x2): 8MHz, acheronComponents:Crystal_SMD_5032-4Pin_5.0x3.2mm, F.Cu at (207.2, 102.4)
- CA1, CB1: value 10n -> 100n
- DF1: footprint Diode_SMD:D_SOD-123 -> acheronComponents:D_SOD-123
- LED1, LED10, LED11, LED12, LED13, LED14, LED15, LED16, LED17, LED18, LED19, LED2, LED20, LED21, LED22, LED23, LED24, LED25, LED26, LED27, LED28, LED29, LED3, LED30, LED31, LED32, LED33, LED34, LED35, LED36, LED37, LED38, LED39, LED4, LED40, LED41, LED42, LED43, LED44, LED45, LED46, LED47, LED48, LED49, LED5, LED50, LED51, LED6, LED7, LED8, LED9: footprint Keyboard_switches:thtLED -> acheronComponents:thtLED
- Q1: footprint Keyboard_switches:AO4406AL -> acheronComponents:AO4406AL
- RGB1, RGB2, RGB3, RGB4, RGB5, RGB6, RGB7, RGB8: footprint Keyboard_switches:LED_WS2812B -> acheronComponents:LED_WS2812B
- SWRST1: footprint smdPushBtn:smdPushBtn -> acheronHardware:smdPushBtn; moved to F.Cu
- U1: value STM32F303CCT7 -> STM32F303CCT6
- moved SWRST1 27.0 mm to (205.5, 75.7), turned to 270 degrees
- moved D10 10.4 mm to (212.9, 82.6), turned to 180 degrees
- moved RL10 10.4 mm to (212.9, 82.6), turned to 180 degrees
- moved D9 5.05 mm to (201.0, 78.1)
- moved RL9 1.51 mm to (204.6, 75.7)
- moved D47 0.59 mm to (241.7, 131.2)
- moved D48 0.59 mm to (244.1, 131.2)
- moved RL47 0.59 mm to (241.7, 131.2)
- moved RL48 0.59 mm to (244.1, 131.2)
- turned D36 to 270 degrees
- renumbered CSRT2 to CRST2, H12 to H7
Connections:
- net Net-(D48-Pad2) renamed EncS3
Routing:
- net EncA: track 314.2 -> 389.8 mm
- net EncB: track 313.1 -> 369.4 mm, vias 2 -> 3
- net 3.3V: track 73.5 -> 93.9 mm, vias 5 -> 7
- net Col12: track 141.8 -> 157.0 mm
- net Net-(DRST1-Pad2): track 56.9 -> 70.3 mm, vias 0 -> 1
- net Row2: track 260.4 -> 273.6 mm
- net Row1: track 256.2 -> 267.9 mm
- net EncS3: track 14.8 -> 23.1 mm
- net GND: track 172.5 -> 165.3 mm, vias 13 -> 12
- net Net-(LED10-PadA): track 11.7 -> 18.4 mm
- net Net-(LED1-PadK): track 1131.8 -> 1125.9 mm
- net Net-(D36-Pad2): track 20.3 -> 16.4 mm
- net Net-(LED35-PadA): track 15.4 -> 12.0 mm
- net Net-(RGB1-Pad2): track 36.5 -> 39.0 mm
- net Row3: track 212.9 -> 210.9 mm
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
Commit message: Added I2C pins and hi-pro compatible plates
Parts:
- removed the Y1 at (207.2, 102.4) (x2)
- added J2: Conn_01x04_Male, acheronConnectors:JSTBM04B-ASRS, F.Cu at (259.0, 83.7)
- added Y1 (x2): 8MHz, acheronComponents:Crystal_SMD_5032-4Pin_5.0x3.2mm, F.Cu at (207.2, 102.4)
Connections:
- U1 pad 30: (no net) -> SCL
- U1 pad 31: Col12 -> SDA
- U1 pad 34: (no net) -> Col12
Routing:
- net SCL: track 0.00 -> 55.4 mm, vias 0 -> 1
- net SDA: track 0.00 -> 52.6 mm, vias 0 -> 1
- net GND: track 165.3 -> 160.3 mm
- net (no net): track 26.9 -> 21.9 mm, vias 13 -> 11
- net Col11: track 138.2 -> 141.4 mm
- net Row1: track 267.9 -> 265.3 mm
- net 5V: track 15.1 -> 16.6 mm
- net Col12: track 157.0 -> 155.7 mm
- net Net-(RGB6-Pad2): track 74.9 -> 75.6 mm
- net Row2: track 273.6 -> 273.1 mm
Other:
- board text added: "5V"
- board text added: "GND"
- board text added: "I2C"
- board text added: "SCL"
- board text added: "SDA"

Commit message: [Feature] Changed the I2C pins to a common pin header
Parts:
- removed the Y1 at (207.2, 102.4) (x2)
- added Y1 (x2): 8MHz, acheronComponents:Crystal_SMD_5032-4Pin_5.0x3.2mm, F.Cu at (207.2, 102.4)
- J2: footprint acheronConnectors:JSTBM04B-ASRS -> acheronConnectors:4pinHeader
- moved J2 9.50 mm to (249.5, 83.7), turned to 0 degrees
Routing:
- net SCL: track 55.4 -> 53.1 mm
- net SDA: track 52.6 -> 50.3 mm
- net 5V: track 16.6 -> 15.1 mm
- net GND: track 160.3 -> 159.7 mm, vias 12 -> 11

Commit message: [Feature] Added header pins for the extra MCU pins
Parts:
- removed the Y1 at (207.2, 102.4) (x2)
- added J3: Conn_01x04_Male, acheronConnectors:4pinHeader, F.Cu at (249.5, 102.7)
- added J4: Conn_01x04_Male, acheronConnectors:4pinHeader, F.Cu at (186.5, 69.2)
- added Y1 (x2): 8MHz, acheronComponents:Crystal_SMD_5032-4Pin_5.0x3.2mm, F.Cu at (207.2, 102.4)
- moved RRST1 0.40 mm to (224.8, 91.4)
Connections:
- U1 pad 26: (no net) -> Extra4
- U1 pad 27: (no net) -> Extra3
- U1 pad 28: (no net) -> Extra2
- U1 pad 29: (no net) -> Extra1
- U1 pad 42: (no net) -> Extra8
- U1 pad 43: (no net) -> Extra7
- U1 pad 45: (no net) -> Extra6
- U1 pad 46: (no net) -> Extra5
Routing:
- net Extra5: track 0.00 -> 70.9 mm, vias 0 -> 2
- net Extra6: track 0.00 -> 64.4 mm, vias 0 -> 2
- net Row2: track 273.1 -> 210.6 mm, vias 1 -> 2
- net Extra7: track 0.00 -> 61.1 mm, vias 0 -> 2
- net Extra8: track 0.00 -> 55.0 mm, vias 0 -> 2
- net Extra4: track 0.00 -> 32.6 mm, vias 0 -> 1
- net Extra3: track 0.00 -> 29.7 mm, vias 0 -> 1
- net Extra2: track 0.00 -> 26.2 mm, vias 0 -> 1
- net Extra1: track 0.00 -> 23.7 mm, vias 0 -> 1
- net Net-(LED1-PadK): track 1125.6 -> 1146.8 mm
- net Row1: track 265.3 -> 286.0 mm
- net (no net): track 21.9 -> 5.65 mm, vias 11 -> 3
- net Col9: track 129.6 -> 138.6 mm
- net Net-(DRST1-Pad2): track 70.3 -> 63.1 mm
- net Col10: track 110.1 -> 115.8 mm, vias 1 -> 2
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Other:
- board text added: "EncA"
- board text added: "EncB"
- board text added: "P26"
- board text added: "P27"
- board text added: "P28"
- board text added: "P29"
- board text added: "P42"
- board text added: "P43"
- board text added: "P45"
- board text added: "P46"

Commit message: [Maintenance] Started adding dimensions and minimal values documentation
Parts:
- removed the Y1 at (207.2, 102.4) (x2)
- added Y1 (x2): 8MHz, acheronComponents:Crystal_SMD_5032-4Pin_5.0x3.2mm, F.Cu at (207.2, 102.4)
- moved J4 0.90 mm to (186.5, 70.1)
- moved F1 0.51 mm to (226.2, 78.3)
- moved RGB1 0.45 mm to (224.5, 83.8)
- moved DF1 0.29 mm to (222.7, 77.6)
- moved J2 0.18 mm to (249.6, 83.7)
- moved RGB4 0.14 mm to (72.5, 83.7)
- moved H7 0.09 mm to (39.6, 103.6)
Routing:
- net 5V: track 15.1 -> 147.0 mm, vias 14 -> 9
- net GND: track 159.9 -> 163.7 mm, vias 11 -> 10
- net Net-(RGB3-Pad2): track 36.6 -> 39.3 mm
- net 3.3V: track 93.4 -> 95.0 mm
- net Extra8: track 55.0 -> 56.4 mm
- net Extra6: track 64.4 -> 65.2 mm
- net Extra5: track 70.9 -> 70.2 mm
- net Net-(DRST1-Pad2): track 63.1 -> 62.4 mm
Other:
- board size 225.6 x 74.8 mm -> 225.6 x 74.6 mm
- board text added: "(1H) PCB HORIZONTAL DIMENSION"
- board text added: "(1R) EDGE CORNER RADIUS"
- board text added: "(1U) GRID UNIT"
- board text added: "(1V) PCB VERTICAL DIMENSION"
- board text added: "(2H) MOUNTING HOLES TO PCB EDGE HORIZONTAL DISTANCE"
- board text added: "(2V) MOUNTING HOLES TO PCB EDGE VERTICAL DISTANCE"
- board text added: "(3H) MCU HORIZONTAL DISTANCE TO PCB EDGE"
- board text added: "(3V) MCU VERTICAL DISTANCE TO PCB EDGE"
- board text added: "1.400 mm"
- board text added: "4.0 mm"
- board text added: "CLEARANCE: 0.13mm (approx. 5mil)"
- board text added: "MEASUREMENTS AND DISTANCES"
- board text added: "MINIMUM VALUES"
- board text added: "SILKSCREEN CHARACTER HEIGHT: 0.8mm"
- board text added: "SILKSCREEN CHARACTER WIDTH: 0.15mm"
- board text added: "TRACE WIDTH: 0.13mm (approx. 5mil)"
- board text added: "UndecidedSharkPCB v3.1.2 "I like the nick 'Shark', but I'm so undecided""
- board text added: "VIA DIAMETER: 0.5mm"
- board text added: "VIA HOLE SIZE: 0.2mm"
- board text added: "VIA-TO-VIA AND VIA-TO-TRACE CLEARANCE: 0.13mm (approx. 5mil)"
- board text removed: "GondolinElectronics UndecidedSharkPCB v3.1.2 "I like the nick 'Shark', but I'm so undecided""
