File: kicadFiles/shark.kicad_pcb (KiCad board)
At the start: 2 copper layers, 225.6 x 74.6 mm, 263 parts, among them J1 USB_C_Receptacle, J2 Conn_01x04_Male, J3 Conn_01x04_Male, J4 Conn_01x04_Male, Q1 AO4406AL, SW1 MXSwitch, SW10 MXSwitch, SW11 MXSwitch, SW12 MXSwitch, SW13 MXSwitch, SW14 MXSwitch, SW15 MXSwitch, SW16 MXSwitch, SW17 MXSwitch, SW18 MXSwitch, SW19 MXSwitch, SW2 MXSwitch, SW20 MXSwitch, SW21 MXSwitch, SW22 MXSwitch, SW23 MXSwitch, SW24 MXSwitch, SW25 MXSwitch, SW26 MXSwitch, SW27 MXSwitch, SW28 MXSwitch, SW29 MXSwitch, SW3 MXSwitch, SW30 MXSwitch, SW31 MXSwitch, SW32 MXSwitch, SW33 MXSwitch, SW34 MXSwitch, SW35 MXSwitch, SW36 MXSwitch, SW37 MXSwitch, SW38 MXSwitch, SW39 MXSwitch, SW4 MXSwitch, SW40 MXSwitch, SW41 MXSwitch, SW42 MXSwitch, SW43 MXSwitch, SW44 MXSwitch, SW45 MXSwitch, SW46 MXSwitch, SW47 MXSwitch, SW48 MXSwitch, SW49 MXSwitch, SW5 MXSwitch, SW50 MXSwitch, SW51 MXSwitch, SW6 MXSwitch, SW7 MXSwitch, SW8 MXSwitch, SW9 MXSwitch, U1 STM32F303CCT6, U2 MCP1700-3302E_SOT23, Y1 8MHz

Commit message: [Maintenance] Started adding dimensions and minimal values documentation
Parts:
- removed the Y1 at (207.2, 102.4) (x2)
- added Y1 (x2): 8MHz, acheronComponents:Crystal_SMD_5032-4Pin_5.0x3.2mm, F.Cu at (207.2, 102.4)
Routing:
- net GND: track 163.7 -> 156.8 mm, vias 10 -> 8
- net Col11: vias 1 -> 0
Other:
- outline, holes or cut-outs redrawn
- board text added: "(5H) USBC CONNECTOR PROTRUSION HORIZONTAL DIMENSION"
- board text added: "(5R) 0.7mm"
- board text added: "(5R) USBC CONNECTOR PROTRUSION RADIUS"
- board text added: "(5V) 1.4mm"
- board text added: "(5V) USBC CONNECTOR PROTRUSION VERTICAL DIMENSION"
- board text added: "CLEARANCE: 0.25mm"
- board text added: "ENCA"
- board text added: "ENCB"
- board text added: "MCU (LQFP 48)"
- board text added: "RECOMMENDED VALUES"
- board text added: "TRACE WIDTH: 0.25mm"
- board text added: "TRACE-TO-EDGE AND VIA-TO-EDGE DISTANCE: 0.2mm"
- board text added: "TRACE-TO-EDGE AND VIA-TO-EDGE DISTANCE: 0.5mm"
- board text added: "These values were the default values used when possible."
- board text added: "UndecidedSharkPCB v3.1.4 "I like the nick 'Shark', but I'm so undecided""
- board text added: "VIA DIAMETER: 1mm"
- board text added: "VIA HOLE SIZE: 0.5mm"
- board text added: "VIA-TO-VIA AND VIA-TO-TRACE CLEARANCE: 0.25mm"
- board text removed: "1.400 mm"
- board text removed: "EncA"
- board text removed: "EncB"
- board text removed: "STM32F303CCT6 (LQFP 48)"
- board text removed: "UndecidedSharkPCB v3.1.2 "I like the nick 'Shark', but I'm so undecided""

Commit message: [Maintenance] Started adding dimensions and minimal values documentation
Parts:
- removed the Y1 at (207.2, 102.4) (x2)
- added Y1 (x2): 8MHz, acheronComponents:Crystal_SMD_5032-4Pin_5.0x3.2mm, F.Cu at (207.2, 102.4)
Other:
- board text added: "(i) The grid unit value used was 19mm, as the Planck uses."
- board text added: "(ii) The PCB was designed to the standards of the JLCPCB (https://jlcpcb.com) manufacturer. Be aware that capabilities may vary, so check with your manufacturer if they support the minimum values listed above."
- board text added: "(iii) All parts were quoted on LCSC supplier (https://lcsc.com/). Also check if your supplier has all the parts listed on the Bill Of Materials and change the footprints and parts accordingly."
- board text added: "(iv) All measurements were done using the metric system, specially 0.1mm and 1mm grids."
- board text added: "(v) You can always contact Gondolindrim through SharkPCBs Github page (https://github.com/Gondolindrim/SharkPCB/)"
- board text added: "GENERAL OBSERVATIONS"
Changed lines of the file:
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@@
   (general
     (thickness 1.6)
-    (drawings 521)
+    (drawings 527)
     (tracks 2143)
     (zones 0)
@@
     )
   )
+  (gr_text "(v) You can always contact Gondolindrim through SharkPCBs Github page (https://github.com/Gondolindrim/SharkPCB/)" (at 44.463 281.743) (layer Dwgs.User)
+    (effects (font (size 1.5 1.5) (thickness 0.1)) (justify left))
+  )
+  (gr_text "(iii) All parts were quoted on LCSC supplier (https://lcsc.com/).\nAlso check if your supplier has all the parts listed on the Bill Of Materials and change the footprints and parts accordingly." (at 44.463 272.743) (layer Dwgs.User)
+    (effects (font (size 1.5 1.5) (thickness 0.1)) (justify left))
+  )
+  (gr_text "(iv) All measurements were done using the metric system, specially 0.1mm and 1mm grids." (at 44.463 277.743) (layer Dwgs.User)
+    (effects (font (size 1.5 1.5) (thickness 0.1)) (justify left))
+  )
+  (gr_text "(ii) The PCB was designed to the standards of the JLCPCB (https://jlcpcb.com) manufacturer.\nBe aware that capabilities may vary, so check with your manufacturer if they support the minimum values listed above." (at 44.463 266.743) (layer Dwgs.User)
+    (effects (font (size 1.5 1.5) (thickness 0.1)) (justify left))
+  )
+  (gr_text "GENERAL OBSERVATIONS" (at 44.463 256.743) (layer Dwgs.User)
+    (effects (font (size 2 2) (thickness 0.5)) (justify left))
+  )
+  (gr_text "(i) The grid unit value used was 19mm, as the Planck uses." (at 44.463 261.743) (layer Dwgs.User)
+    (effects (font (size 1.5 1.5) (thickness 0.1)) (justify left))
+  )
   (gr_text "TRACE-TO-EDGE AND VIA-TO-EDGE DISTANCE: 0.5mm" (at 149.463 209.743) (layer Dwgs.User)
     (effects (font (size 1.5 1.5) (thickness 0.1)) (justify left))
@@
   )
   (dimension 37.3 (width 0.15) (layer Dwgs.User)
-    (gr_text "37.300 mm" (at 14.209 84.993 90) (layer Dwgs.User)
+    (gr_text "(6) 37.3 mm" (at 14.209 84.993 90) (layer Dwgs.User)
       (effects (font (size 1.5 1.5) (thickness 0.15)))
     )
@@
   (segment (start 178.233 117.34747) (end 178.233 115.80572) (width 0.5) (layer F.Cu) (net 71))
   (segment (start 159.1505 115.78125) (end 178.233 115.78125) (width 0.5) (layer F.Cu) (net 71))
-  (segment (start 178.233 115.78125) (end 215.55325 115.78125) (width 0.5) (layer F.Cu) (net 71))
-  (segment (start 215.55325 115.78125) (end 215.83029 115.78125) (width 0.5) (layer F.Cu) (net 71))
-  (segment (start 215.83029 115.78125) (end 216.44852 116.39948) (width 0.5) (layer F.Cu) (net 71))
   (segment (start 216.44852 116.39948) (end 216.44852 116.99324) (width 0.5) (layer F.Cu) (net 71))
   (segment (start 241.68175 131.243) (end 244.35476 131.243) (width 0.254) (layer F.Cu) (net 71))
@@
   (via (at 218.5255 104.993) (size 0.5) (drill 0.2) (layers F.Cu B.Cu) (net 61))
   (via (at 217.634875 105.493) (size 0.5) (drill 0.2) (layers F.Cu B.Cu) (net 62))
+  (segment (start 178.233 115.78125) (end 215.55325 115.78125) (width 0.5) (layer F.Cu) (net 71))
+  (segment (start 215.83029 115.78125) (end 216.44852 116.39948) (width 0.5) (layer F.Cu) (net 71))
+  (segment (start 215.55325 115.78125) (end 215.83029 115.78125) (width 0.5) (layer F.Cu) (net 71))
   (via (at 227.263 111.343) (size 0.5) (drill 0.2) (layers F.Cu B.Cu) (net 138))
   (zone (net 48) (net_name "Net-(C7-Pad2)") (layer B.Cu) (hatch edge 0.508)

Commit message: [Maintenance] Started making silkscreen characters bigger for readability
Parts:
- removed the Y1 at (207.2, 102.4) (x2)
- added Y1 (x2): 8MHz, acheronComponents:Crystal_SMD_5032-4Pin_5.0x3.2mm, F.Cu at (220.2, 102.4)
- moved D12 13.0 mm to (257.7, 74.2)
- moved D24 13.0 mm to (257.7, 93.2)
- moved D36 13.0 mm to (257.7, 112.2)
- moved H5 13.0 mm to (256.5, 102.7)
- moved J3 13.0 mm to (262.5, 102.7)
- moved LED12 13.0 mm to (266.0, 79.2)
- moved LED24 13.0 mm to (266.0, 98.3)
- moved LED36 13.0 mm to (266.0, 117.3)
- moved LED48 13.0 mm to (266.0, 136.3)
- moved RL12 13.0 mm to (257.7, 74.2)
- moved RL24 13.0 mm to (257.7, 93.2)
- moved RL36 13.0 mm to (257.7, 112.2)
- moved SW12 13.0 mm to (266.0, 74.2)
- moved SW24 13.0 mm to (266.0, 93.2)
- moved SW36 13.0 mm to (266.0, 112.3)
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Other:
- board text added: "(4H) RGB UNDERGLOW RGB LEDS HORIZONTAL SPACING"
- board text added: "(4V) RGB UNDERGLOW RGB LEDS VERTICAL SPACING"
- board text added: "(6H) ESD CONNECTOR TO EDGE HORIZONTAL SPACING"
- board text added: "(6V) ESD CONNECTOR TO EDGE VERTICAL SPACING"
- board text added: "(I) If you want to check or reroute a specific trace, I recommend using the High Contrast mode. Turn it on by going in the View menu, "Contrast mode" and checking the "High contrast mode". Alternatively you can press H."
- board text added: "(II) All footprints are available either in KiCad's own native libraries or the Acheron Library (http://github.com/Gondolindrim/acheronLibrary). To facilitate the portability of this project, the project footprint libraries are addressed through a simbolic path, ${ACHERONLIB}$. So before modifying this PCB in any way, please download the Acheron Library. Then, in this KiCad file, go to "Preferenc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"
- board text added: "(v) You can always contact Gondolindrim through SharkPCBs Github page (https://github.com/Gondolindrim/SharkPCB/)."
- board text added: "(vi) JLCPCB states their minimum character width is 0.8mm, and anything below that will be undiscernable. In my opinion you can go down to 0.5mm without incurring in readability problems, although at that level you will need to look closely to the PCB to read the characters. The minimum character height at which there will certainly be easily redable to the naked eye is 0.8mm indeed."
- board text added: "SILKSCREEN CHARACTER HEIGHT: 0.5mm (see General Observation (x))"
- board text added: "STM32F303CCT6 (LQFP 48)"
- board text added: "These are general hints to use this PCB file. They are aimed specially at those new to KiCad or ECAD in general, and to whoever wishes to use this project."
- board text added: "USAGE GUIDE (PLEASE READ)"
- board text removed: "(v) You can always contact Gondolindrim through SharkPCBs Github page (https://github.com/Gondolindrim/SharkPCB/)"
- board text removed: "MCU (LQFP 48)"
- board text removed: "SILKSCREEN CHARACTER HEIGHT: 0.8mm"

Commit message: [Maintenance] Added documentation and notes on the design
Routing:
- net Extra6: track 65.2 -> 64.2 mm
Changed lines of the file:
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@@
     (thickness 1.6)
     (drawings 538)
-    (tracks 2143)
+    (tracks 2144)
     (zones 0)
     (modules 263)
@@
     (last_trace_width 0.254)
     (trace_clearance 0.127)
-    (zone_clearance 0.13)
+    (zone_clearance 0.127)
     (zone_45_only no)
     (trace_min 0.1)
@@
       (drillshape 0)
       (scaleselection 1)
-      (outputdirectory "../gerbers/pcb/"))
+      (outputdirectory "/home/alvaro/Desktop/output/FSilk"))
   )
   (net 0 "")
@@
     (attr smd)
     (fp_text reference D37 (at 0 0 180) (layer F.SilkS)
-      (effects (font (size 0.4 0.4) (thickness 0.1)))
+      (effects (font (size 0.6 0.6) (thickness 0.15)))
     )
     (fp_text value 1N4148 (at 0 2.1 90) (layer F.Fab)
@@
     (attr smd)
     (fp_text reference D38 (at 0 0 180) (layer F.SilkS)
-      (effects (font (size 0.4 0.4) (thickness 0.1)))
+      (effects (font (size 0.6 0.6) (thickness 0.15)))
     )
     (fp_text value 1N4148 (at 0 2.1 90) (layer F.Fab)
@@
     (attr smd)
     (fp_text reference D39 (at -0.075 -0.0125 unlocked) (layer F.SilkS)
-      (effects (font (size 0.5 0.5) (thickness 0.125)))
+      (effects (font (size 0.6 0.6) (thickness 0.15)))
     )
     (fp_text value 1N4148 (at 0 2.1 90) (layer F.Fab)
@@
     (attr smd)
     (fp_text reference D40 (at -0.075 0.0125 unlocked) (layer F.SilkS)
-      (effects (font (size 0.5 0.5) (thickness 0.125)))
+      (effects (font (size 0.6 0.6) (thickness 0.15)))
     )
     (fp_text value 1N4148 (at 0 2.1 90) (layer F.Fab)
@@
   (segment (start 209.863 90.643) (end 202.363 90.643) (width 0.13) (layer F.Cu) (net 150))
   (segment (start 198.126466 80.743) (end 197.963 80.579534) (width 0.13) (layer F.Cu) (net 150))
-  (segment (start 197.963 73.243) (end 199.463 71.743) (width 0.13) (layer F.Cu) (net 150))
-  (segment (start 197.963 80.579534) (end 197.963 73.243) (width 0.13) (layer F.Cu) (net 150))
   (segment (start 198.52001 86.80001) (end 198.52001 81.136543) (width 0.13) (layer F.Cu) (net 150))
   (segment (start 198.52001 81.136543) (end 198.126466 80.743) (width 0.13) (layer F.Cu) (net 150))
@@
   (segment (start 230.32001 96.28599) (end 225.10599 96.28599) (width 0.13) (layer B.Cu) (net 150))
   (via (at 236.213 96.8055) (size 0.5) (drill 0.2) (layers F.Cu B.Cu) (net 150))
+  (segment (start 197.963 74.718) (end 197.963 74.218) (width 0.13) (layer F.Cu) (net 150))
+  (segment (start 197.963 80.579534) (end 197.963 74.718) (width 0.13) (layer F.Cu) (net 150))
+  (segment (start 197.963 74.218) (end 199.463 72.718) (width 0.13) (layer F.Cu) (net 150))
   (segment (start 237.213 98.393) (end 237.213 96.8055) (width 0.13) (layer F.Cu) (net 151) (status 10))
   (segment (start 209.863 89.943) (end 209.863 89.943) (width 0.13) (layer B.Cu) (net 151))
@@
   (segment (start 200.463 80.243) (end 200.463 78.943) (width 0.13) (layer F.Cu) (net 152))
   (segment (start 200.463 78.743) (end 199.463 77.743) (width 0.13) (layer F.Cu) (net 152))
-  (zone (net 48) (net_name "Net-(C7-Pad2)") (layer B.Cu) (hatch edge 0.508)
-    (connect_pads yes (clearance 0.13))
-    (min_thickness 0.13)
-    (fill yes (arc_segments 16) (thermal_gap 0.254) (thermal_bridge_width 0.254))
-    (polygon
-      (pts
-        (xy 231.863 73.643) (xy 243.063 73.643) (xy 243.063 61.743) (xy 231.863 61.743)
-      )
-    )
-  )
   (zone (net 1) (net_name GND) (layer F.Cu) (hatch edge 0.508)
     (connect_pads yes (clearance 0.127))
@@
     )
   )
-  (zone (net 49) (net_name "Net-(C9-Pad2)") (layer F.Cu) (hatch edge 0.508)
-    (connect_pads yes (clearance 0.127))
-    (min_thickness 0.127)
-    (fill yes (arc_segments 16) (thermal_gap 0.5) (thermal_bridge_width 0.5))
+  (zone (net 48) (net_name "Net-(C7-Pad2)") (layer B.Cu) (hatch edge 0.508)
+    (connect_pads yes (clearance 0.13))
+    (min_thickness 0.13)
+    (fill yes (arc_segments 16) (thermal_gap 0.254) (thermal_bridge_width 0.254))
     (polygon
       (pts
-        (xy 45.359375 100.9375) (xy 57.53125 100.9375) (xy 57.53125 106.578125) (xy 45.359375 106.578125)
+        (xy 231.863 73.643) (xy 243.063 73.643) (xy 243.063 61.743) (xy 231.863 61.743)
       )
     )
@@
       )
     )
+  )
+  (zone (net 49) (net_name "Net-(C9-Pad2)") (layer F.Cu) (hatch edge 0.508)
+    (connect_pads yes (clearance 0.127))
+    (min_thickness 0.127)
+    (fill yes (arc_segments 16) (thermal_gap 0.5) (thermal_bridge_width 0.5))
+    (polygon
+      (pts
+        (xy 45.359375 100.9375) (xy 57.53125 100.9375) (xy 57.53125 106.578125) (xy 45.359375 106.578125)
+      )
+    )

Commit message: [Fix] Used 3.3V for encoder VCC instead of 5V
Parts:
- CA1, CB1, RA1, RA2, RB1, RB2: moved to F.Cu
- moved RB1 156.9 mm to (250.7, 125.1)
- moved RB2 155.8 mm to (244.7, 123.1)
- moved RA2 155.0 mm to (244.7, 120.1)
- moved RA1 155.0 mm to (249.9, 120.1)
- moved CB1 152.6 mm to (252.3, 117.7)
- moved CA1 152.3 mm to (251.0, 122.5), turned to 0 degrees
Connections:
- RA2 pad 2: 5V -> 3.3V
- RB2 pad 2: 5V -> 3.3V
Routing:
- net 5V: track 147.0 -> 26.0 mm, vias 9 -> 11
- net GND: track 156.8 -> 119.6 mm, vias 8 -> 6
- net EncB: track 369.4 -> 350.9 mm, vias 3 -> 4
- net 3.3V: track 95.0 -> 110.8 mm, vias 7 -> 8
- net Col10: track 115.8 -> 121.2 mm
- net Net-(DRST1-Pad2): track 62.4 -> 67.5 mm
- net Net-(LED1-PadK): track 1146.8 -> 1150.9 mm
- net Extra5: track 70.2 -> 66.7 mm
- net Extra6: track 64.2 -> 61.5 mm
- net Extra7: track 61.3 -> 58.8 mm
- net Net-(RGB3-Pad2): track 39.3 -> 37.6 mm
- net LED_PWM: track 147.7 -> 145.9 mm
- net Extra8: track 56.4 -> 54.8 mm
- net Net-(CA1-Pad2): track 2.01 -> 3.11 mm
- net EncA: track 391.4 -> 390.4 mm

Commit message: [Maintenance] Moved some SMD parts to the bottom layer to ensure no problems with switch mounting
Parts:
- CRST1, CSin1, CSout1, CVBus1, CVBus2, CVBus3, CVBus4, CVBus5, DRST1, DS1, RRST1, U2: moved to F.Cu
- moved DS1 38.3 mm to (206.9, 121.7)
- moved CSin1 36.7 mm to (204.5, 121.7), turned to 90 degrees
- moved U2 32.6 mm to (210.1, 121.7), turned to 180 degrees
- moved CSout1 27.5 mm to (213.5, 121.7)
- moved CVBus5 25.2 mm to (228.3, 120.5), turned to 270 degrees
- moved CVBus3 25.1 mm to (226.3, 120.5), turned to 270 degrees
- moved CVBus4 23.3 mm to (224.3, 120.5), turned to 270 degrees
- moved CVBus2 21.9 mm to (230.3, 120.5), turned to 270 degrees
- moved CVBus1 21.8 mm to (232.5, 120.5), turned to 270 degrees
- moved RRST1 1.87 mm to (239.2, 90.1), turned to 270 degrees
- moved CRST1 1.35 mm to (241.8, 90.1), turned to 90 degrees
- moved DRST1 1.31 mm to (236.4, 90.1), turned to 270 degrees
- moved L2 0.16 mm to (165.5, 113.1)
Connections:
- U1 pad 10: Col10 -> Col4
- U1 pad 11: Col4 -> Col10
Routing:
- net GND: track 119.6 -> 62.2 mm
- net 3.3V: track 110.8 -> 148.2 mm, vias 8 -> 9
- net 5V: track 26.0 -> 43.8 mm
- net EncB: track 350.9 -> 366.0 mm
- net EncA: track 390.4 -> 405.0 mm
- net Row2: track 210.4 -> 219.4 mm
- net Net-(J1-PadA6): track 64.6 -> 55.8 mm
- net Net-(RGB5-Pad2): track 35.3 -> 43.0 mm
- net RGB_PWM: track 46.7 -> 53.9 mm
- net Row1: track 286.0 -> 292.2 mm
- net Col1: track 278.7 -> 272.9 mm
- net Col2: track 274.5 -> 271.5 mm
- net Net-(DRST1-Pad2): track 67.5 -> 69.6 mm, vias 1 -> 2
- net Net-(RGB6-Pad2): track 75.6 -> 77.5 mm
- net LED_PWM: track 145.9 -> 147.6 mm
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Other:
- board text added: "CSI"
- board text added: "UndecidedSharkPCB v3.1.5 "I like the nick 'Shark', but I'm so undecided""
- board text removed: "UndecidedSharkPCB v3.1.4 "I like the nick 'Shark', but I'm so undecided""
