File: kicadFiles/shark.kicad_pcb (KiCad board)
At the start: 2 copper layers, 225.6 x 74.6 mm, 265 parts, among them J1 USB_C_Receptacle, J2 Conn_01x04_Male, J3 Conn_01x04_Male, J4 Conn_01x04_Male, J5 Conn_01x06_Male, Q1 AO4406AL, SW1 MXSwitch, SW10 MXSwitch, SW11 MXSwitch, SW12 MXSwitch, SW13 MXSwitch, SW14 MXSwitch, SW15 MXSwitch, SW16 MXSwitch, SW17 MXSwitch, SW18 MXSwitch, SW19 MXSwitch, SW2 MXSwitch, SW20 MXSwitch, SW21 MXSwitch, SW22 MXSwitch, SW23 MXSwitch, SW24 MXSwitch, SW25 MXSwitch, SW26 MXSwitch, SW27 MXSwitch, SW28 MXSwitch, SW29 MXSwitch, SW3 MXSwitch, SW30 MXSwitch, SW31 MXSwitch, SW32 MXSwitch, SW33 MXSwitch, SW34 MXSwitch, SW35 MXSwitch, SW36 MXSwitch, SW37 MXSwitch, SW38 MXSwitch, SW39 MXSwitch, SW4 MXSwitch, SW40 MXSwitch, SW41 MXSwitch, SW42 MXSwitch, SW43 MXSwitch, SW44 MXSwitch, SW45 MXSwitch, SW46 MXSwitch, SW47 MXSwitch, SW48 MXSwitch, SW49 MXSwitch, SW5 MXSwitch, SW50 MXSwitch, SW51 MXSwitch, SW6 MXSwitch, SW7 MXSwitch, SW8 MXSwitch, SW9 MXSwitch, U1 STM32F303CCT6, U2 MCP1700-3302E_SOT23, Y1 8MHz

Commit message: [Update] Pre-release of version 3.2.2
Parts:
- moved RGB5 1.00 mm to (237.5, 121.7)
- renumbered CESD1 to CESD, DESD1 to DESD, RESD1 to RESD
Routing:
- net RGB_PWM: track 44.3 -> 46.4 mm
- net Net-(RGB5-Pad2): track 46.0 -> 45.2 mm
- net 5V: track 44.2 -> 43.5 mm
Other:
- board text added: "SILKSCREEN CHARACTER HEIGHT: 0.6mm"
- board text added: "SILKSCREEN CHARACTER WIDTH: 0.125mm"
- board text added: "UndecidedSharkPCB v3.2.2 "I like the nick 'Shark', but I'm so undecided""
- board text removed: "UndecidedSharkPCB v3.2.0 "I like the nick 'Shark', but I'm so undecided""

Commit message: [Update] Made changes to routing
Routing:
- net BOOT0: track 61.8 -> 80.2 mm
- net EncA: track 382.0 -> 399.5 mm
- net Extra1: track 23.7 -> 27.4 mm
- net Extra5: track 63.0 -> 59.3 mm
- net SWCLK: track 62.4 -> 65.5 mm
- net SWDIO: track 61.9 -> 64.6 mm
- net Extra8: track 50.2 -> 52.3 mm
- net Col10: track 122.1 -> 124.2 mm
- net Extra2: track 26.2 -> 28.1 mm
- net Extra6: track 57.4 -> 55.8 mm
- net Net-(J1-PadA6): track 58.4 -> 59.7 mm
- net EncB: track 368.3 -> 369.6 mm
- net Col11: track 140.4 -> 141.6 mm
- net 3.3V: track 181.7 -> 182.9 mm
- net Col1: track 283.6 -> 284.6 mm
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Other:
- net class Super Thick added: clearance 0.13, trace_width 1, via_dia 0.45, via_drill 0.2
- board text added: "UndecidedSharkPCB v3.2.3 "I like the nick 'Shark', but I'm so undecided""
- board text removed: "UndecidedSharkPCB v3.2.2 "I like the nick 'Shark', but I'm so undecided""

Commit message: V3.2.4
Parts:
- added CUSB1: 4.7n, Capacitor_SMD:C_0805_2012Metric_Pad1.15x1.40mm_HandSolder, F.Cu at (253.1, 88.3)
- added CVA1: 1u, Capacitor_SMD:C_0805_2012Metric_Pad1.15x1.40mm_HandSolder, B.Cu at (236.5, 102.7)
- added CVA2: 10n, Capacitor_SMD:C_0805_2012Metric_Pad1.15x1.40mm_HandSolder, B.Cu at (238.5, 102.7)
- added U3: USBLC6-2SC6, Package_TO_SOT_SMD:SOT-23-6, F.Cu at (250.1, 83.9)
- moved RPGate1 9.38 mm to (153.7, 102.7), turned to 270 degrees
- moved RSGate1 6.91 mm to (151.2, 102.7), turned to 270 degrees
- moved Q1 5.37 mm to (142.5, 102.8)
- renumbered CV1 to CVB1, CV2 to CVB2, CV3 to CVB3, CV4 to CVB4, CV5 to CVB5, RD+Up1 to RDPUp1
Connections:
- J1 pad A6: Net-(J1-PadA6) -> D+Bus
- J1 pad A7: Net-(J1-PadA7) -> D-Bus
- J1 pad A8: (no net) -> Net-(J1-PadA8)
- J1 pad B6: Net-(J1-PadA6) -> D+Bus
- J1 pad B7: Net-(J1-PadA7) -> D-Bus
- J1 pad B8: (no net) -> Net-(J1-PadB8)
- RD+1 pad 2: Net-(J1-PadA6) -> Net-(RD+1-Pad2)
- RD-1 pad 2: Net-(J1-PadA7) -> Net-(RD-1-Pad2)
- RDPUp1 pad 1: 5V -> VBUS
- RDPUp1 pad 2: Net-(J1-PadA6) -> D+Bus
- RGB4 pad 2: (no net) -> Net-(RGB4-Pad2)
- RGB8 pad 2: (no net) -> Net-(RGB8-Pad2)
- U1 pad 18: (no net) -> Net-(U1-Pad18)
Routing:
- net Net-(J1-PadA7): track 61.8 -> 0.00 mm
- net Net-(J1-PadA6): track 59.7 -> 0.00 mm, vias 2 -> 0
- net Net-(RD-1-Pad2): track 0.00 -> 43.1 mm
- net Net-(RD+1-Pad2): track 0.00 -> 33.7 mm
- net D-Bus: track 0.00 -> 26.6 mm
- net D+Bus: track 0.00 -> 24.6 mm, vias 0 -> 2
- net LED_PWM: track 146.8 -> 155.0 mm
- net Net-(CUSB1-Pad2): track 0.00 -> 7.01 mm
- net GND: track 65.2 -> 59.4 mm
- net VBUS: track 13.5 -> 18.8 mm
- net Net-(U1-Pad18): track 0.00 -> 2.48 mm, vias 0 -> 1
- net (no net): track 2.48 -> 0.00 mm, vias 1 -> 0
- net Row1: track 311.6 -> 310.6 mm
- net Net-(LED1-PadK): track 1171.0 -> 1171.9 mm, vias 1 -> 0
- net 3.3V: track 182.9 -> 182.1 mm
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Other:
- board text added: "(III) For detailed information check the documentation: http://gondolindrim.io/AcheronDocs/shark/shark.html"
- board text added: "CVB1"
- board text added: "CVB2"
- board text added: "CVB3"
- board text added: "CVB4"
- board text added: "CVB5"
- board text added: "SharkPCB v3.2.4 "I like the nick 'Shark', but I'm so undecided""
- board text removed: "CV1"
- board text removed: "CV2"
- board text removed: "CV3"
- board text removed: "CV4"
- board text removed: "CV5"
- board text removed: "Surge protection"
- board text removed: "UndecidedSharkPCB v3.2.3 "I like the nick 'Shark', but I'm so undecided""

Commit message: Updated footprints according to Acheron Library changes
Parts:
- removed the Y1 at (220.2, 102.4) (x2)
- added Y1: 8MHz, acheronComponents:Crystal_SMD_5032-4Pin_5.0x3.2mm, F.Cu at (220.1, 102.2)
- J1: value USB_C_Receptacle -> TYPE-C-31-M12_13
- U1: value STM32F303CCT6 -> STM32F303-LQFP48; footprint Package_QFP:LQFP-48_7x7mm_P0.5mm -> acheronComponents:LQFP-48_7x7mm_P0.5mm
- U3: footprint Package_TO_SOT_SMD:SOT-23-6 -> acheronComponents:SOT-23-6
- moved L6 0.81 mm to (159.7, 84.1)
- renumbered CESD to CESD1, CUSB1 to CUSB, DESD to DESD1, RESD to RESD1
Connections:
- CUSB pad 2: Net-(CUSB1-Pad2) -> VBUS
- J1 pad A8: Net-(J1-PadA8) -> (no net)
- J1 pad B8: Net-(J1-PadB8) -> (no net)
- RD+1 pad 1: D+ -> (no net)
- RGB4 pad 2: Net-(RGB4-Pad2) -> (no net)
- RGB8 pad 2: Net-(RGB8-Pad2) -> (no net)
- U1 pad 18: Net-(U1-Pad18) -> (no net)
- U1 pad 32: D- -> (no net)
- U1 pad 33: D+ -> D-
- U3 pad 5: Net-(CUSB1-Pad2) -> VBUS
Routing:
- net VBUS: track 18.8 -> 38.2 mm, vias 2 -> 3
- net Net-(CUSB1-Pad2): track 7.01 -> 0.00 mm
- net Net-(RD-1-Pad2): track 43.1 -> 36.7 mm
- net D-: track 6.55 -> 12.8 mm, vias 1 -> 2
- net D+: track 6.28 -> 0.00 mm, vias 1 -> 0
- net D-Bus: track 26.6 -> 29.8 mm
- net Net-(U1-Pad18): track 2.48 -> 0.00 mm, vias 1 -> 0
- net (no net): track 0.00 -> 2.48 mm, vias 0 -> 1
- net GND: track 59.4 -> 57.9 mm
- net Row1: track 310.6 -> 311.2 mm
Other:
- board text added: "CESD"
- board text added: "DESD"
- board text added: "P45"
- board text added: "P46"
- board text added: "RESD"
- board text added: "SILKSCREEN CHARACTER HEIGHT: 0.5mm (see General Observation (vi))"
- board text added: "SILKSCREEN CHARACTER TRACE WIDTH: 0.125mm"
- board text added: "SharkPCB rev. Alpha "I like the nick 'Shark', but I'm so undecided""
- board text removed: "P42"
- board text removed: "P43"
- board text removed: "SILKSCREEN CHARACTER HEIGHT: 0.5mm (see General Observation (x))"
- board text removed: "SILKSCREEN CHARACTER WIDTH: 0.125mm"
- board text removed: "SharkPCB v3.2.4 "I like the nick 'Shark', but I'm so undecided""

Commit message: [Update] USB connector label and revisited BOM
Other:
- board text added: "SharkPCB V3.2.6 "I like the nick 'Shark', but I'm so undecided""
- board text removed: "SharkPCB rev. Alpha "I like the nick 'Shark', but I'm so undecided""
