File: kicadFiles/shark.sch (KiCad schematic (older format))
At the start: 262 parts, among them J1 USB_C_Receptacle, J2 Conn_01x04_Male, J3 Conn_01x04_Male, J4 Conn_01x04_Male, Q1 AO4406AL, SW1 MXSwitch, SW10 MXSwitch, SW11 MXSwitch, SW12 MXSwitch, SW13 MXSwitch, SW14 MXSwitch, SW15 MXSwitch, SW16 MXSwitch, SW17 MXSwitch, SW18 MXSwitch, SW19 MXSwitch, SW2 MXSwitch, SW20 MXSwitch, SW21 MXSwitch, SW22 MXSwitch, SW23 MXSwitch, SW24 MXSwitch, SW25 MXSwitch, SW26 MXSwitch, SW27 MXSwitch, SW28 MXSwitch, SW29 MXSwitch, SW3 MXSwitch, SW30 MXSwitch, SW31 MXSwitch, SW32 MXSwitch, SW33 MXSwitch, SW34 MXSwitch, SW35 MXSwitch, SW36 MXSwitch, SW37 MXSwitch, SW38 MXSwitch, SW39 MXSwitch, SW4 MXSwitch, SW40 MXSwitch, SW41 MXSwitch, SW42 MXSwitch, SW43 MXSwitch, SW44 MXSwitch, SW45 MXSwitch, SW46 MXSwitch, SW47 MXSwitch, SW48 MXSwitch, SW49 MXSwitch, SW5 MXSwitch, SW50 MXSwitch, SW51 MXSwitch, SW6 MXSwitch, SW7 MXSwitch, SW8 MXSwitch, SW9 MXSwitch, U1 STM32F303CCT6, U2 MCP1700-3302E_SOT23, Y1 8MHz

Commit message: [Feature] Adde the Acheron Project logo
Parts:
- added L6: usFlag, acheronLogos:acheronLogo, symbol Mechanical:MountingHole
Changed lines of the file:
@@
 Wire Wire Line
 	5900 12800 6175 12800
-Text Notes 14925 4425 0    100  Italic 20
+Text Notes 14925 4675 0    100  Italic 20
 Mounting holes
-Wire Notes Line width 20
-	16475 4475 16475 3000
-Text Notes 16550 4425 0    100  Italic 20
+Text Notes 16550 4675 0    100  Italic 20
 Logos and flags
 Wire Notes Line width 20
@@
 USB Connector
 Wire Notes Line width 20
-	14850 3000 14850 4500
-Wire Notes Line width 20
-	16150 3000 16150 4500
-Wire Notes Line width 20
-	14850 4500 16150 4500
+	14850 4750 16150 4750
 Wire Notes Line width 20 style dash_dot
 	14850 3000 16150 3000
@@
 	16475 3000 17900 3000
 Wire Notes Line width 20
-	17900 2975 17900 4475
-Wire Notes Line width 20
-	16475 4475 17900 4475
+	16475 4725 17900 4725
 Wire Notes Line width 20
 	15025 7125 17425 7125
@@
 Text GLabel 13400 10950 2    50   Input ~ 0
 Extra8
+Wire Notes Line width 20
+	14850 3000 14850 4750
+Wire Notes Line width 20
+	16150 3000 16150 4775
+$Comp
+L Mechanical:MountingHole L6
+U 1 1 5D02D130
+P 17025 4325
+F 0 "L6" H 17125 4371 50  0000 L CNN
+F 1 "usFlag" H 17125 4280 50  0000 L CNN
+F 2 "acheronLogos:acheronLogo" H 17025 4325 50  0001 C CNN
+F 3 "~" H 17025 4325 50  0001 C CNN
+	1    17025 4325
+	1    0    0    -1
+$EndComp
+Wire Notes Line width 20
+	16475 3000 16475 4725
+Wire Notes Line width 20
+	17900 2975 17900 4725
 $EndSCHEMATC

Commit message: [Update] Enlarged the plate pegs holes in the PCB
Parts:
- J1: symbol Connector:USB_C_Receptacle -> shark-rescue:USB_C_Receptacle-Connector
Changed lines of the file:
@@
 EESchema Schematic File Version 4
 LIBS:shark-cache
-EELAYER 26 0
+EELAYER 29 0
 EELAYER END
 $Descr A2 23386 16535
@@
 Title "SharkPCB"
 Date "2019-03-20"
-Rev "3.1.6"
+Rev "3.1.7"
 Comp "Gondolin Electronics"
 Comment1 ""
@@
 	16025 9850 16250 9850
 $Comp
-L Connector:USB_C_Receptacle J1
+L shark-rescue:USB_C_Receptacle-Connector J1
 U 1 1 5CC01BA3
 P 8625 10675

Commit message: [Update] Pre-release of version 3.2.0
Parts:
- removed H7: CASE, MountingHole:MountingHole_2.2mm_M2_Pad_Via, symbol Mechanical:MountingHole_Pad
- added DESD1: 1N4002, Diode_SMD:D_0805_2012Metric_Pad1.15x1.40mm_HandSolder, symbol Device:D
- added J5: Conn_01x06_Male, acheronConnectors:male6pinHeader, symbol Connector:Conn_01x06_Male
- H4: symbol Mechanical:MountingHole -> Mechanical:MountingHole_Pad
- renumbered C9 to CESD1, CVBus1 to CV1, CVBus2 to CV2, CVBus3 to CV3, CVBus4 to CV4, CVBus5 to CV5, C1 to CX1, C2 to CX2, R6 to RESD1
Connections:
- net labels added: CASE, SWCLK, SWDIO
- wire segments 648 -> 658
Other:
- note added: "Serial programming"
Changed lines of the file:
@@
 Sheet 1 1
 Title "SharkPCB"
-Date "2019-03-20"
-Rev "3.1.7"
+Date "2019-05-20"
+Rev "3.2.0"
 Comp "Gondolin Electronics"
 Comment1 ""
@@
 $EndDescr
 $Comp
-L Device:C_Small C1
+L Device:C_Small CX1
 U 1 1 5BEDBE98
 P 19950 7275
-F 0 "C1" H 20042 7321 50  0000 L CNN
+F 0 "CX1" H 20042 7321 50  0000 L CNN
 F 1 "22p" H 20042 7230 50  0000 L CNN
 F 2 "Capacitor_SMD:C_0805_2012Metric_Pad1.15x1.40mm_HandSolder" H 19950 7275 50  0001 C CNN
@@
 $EndComp
 $Comp
-L Device:C_Small C2
+L Device:C_Small CX2
 U 1 1 5BEDBF42
 P 20650 7275
-F 0 "C2" H 20742 7321 50  0000 L CNN
+F 0 "CX2" H 20742 7321 50  0000 L CNN
 F 1 "22p" H 20742 7230 50  0000 L CNN
 F 2 "Capacitor_SMD:C_0805_2012Metric_Pad1.15x1.40mm_HandSolder" H 20650 7275 50  0001 C CNN
@@
 $EndComp
 $Comp
-L Mechanical:MountingHole H4
+L Mechanical:MountingHole_Pad H4
 U 1 1 5BF2790A
-P 15225 3750
-F 0 "H4" H 15325 3796 50  0000 L CNN
-F 1 "MountingHole" H 15325 3705 50  0000 L CNN
-F 2 "MountingHole:MountingHole_2.5mm_Pad" H 15225 3750 50  0001 C CNN
-F 3 "~" H 15225 3750 50  0001 C CNN
-	1    15225 3750
-	1    0    0    -1
+P 15275 3750
+F 0 "H4" V 15325 3600 50  0000 L CNN
+F 1 "MountingHole" V 15200 3200 50  0000 L CNN
+F 2 "MountingHole:MountingHole_2.5mm_Pad" H 15275 3750 50  0001 C CNN
+F 3 "~" H 15275 3750 50  0001 C CNN
+	1    15275 3750
+	0    -1   -1   0
 $EndComp
 $Comp
@@
 U 1 1 5BF463E9
 P 15225 3350
-F 0 "H2" H 15325 3396 50  0000 L CNN
-F 1 "MountingHole" H 15325 3305 50  0000 L CNN
+F 0 "H2" V 15275 3150 50  0000 L CNN
+F 1 "MountingHole" V 15175 2750 50  0000 L CNN
 F 2 "MountingHole:MountingHole_2.5mm_Pad" H 15225 3350 50  0001 C CNN
 F 3 "~" H 15225 3350 50  0001 C CNN
 	1    15225 3350
-	1    0    0    -1
+	0    -1   -1   0
 $EndComp
 $Comp
@@
 	1    0    0    -1
 $EndComp
-Wire Wire Line
-	18275 12025 18275 12075
 $Comp
-L Device:C_Small C9
+L Device:C_Small CESD1
 U 1 1 5C391EB2
 P 18275 12225
-F 0 "C9" H 18350 12150 31  0000 R CNN
+F 0 "CESD1" V 18175 12275 31  0000 R CNN
 F 1 "4.7n" H 18400 12300 31  0000 R CNN
 F 2 "Capacitor_SMD:C_0805_2012Metric_Pad1.15x1.40mm_HandSolder" H 18275 12225 50  0001 C CNN
@@
 $EndComp
 $Comp
-L Device:R R6
+L Device:R RESD1
 U 1 1 5C391EB9
 P 18075 12225
-F 0 "R6" V 17975 12225 50  0000 C CNN
+F 0 "RESD1" V 17975 12225 50  0000 C CNN
 F 1 "1M" V 18075 12225 50  0000 C CNN
 F 2 "Resistor_SMD:R_1206_3216Metric_Pad1.42x1.75mm_HandSolder" V 18005 12225 50  0001 C CNN
@@
 	1    0    0    -1
 $EndComp
-$Comp
-L Mechanical:MountingHole_Pad H7
-U 1 1 5C3B52F4
-P 18275 11925
-F 0 "H7" H 18375 11976 50  0000 L CNN
-F 1 "CASE" H 18375 11885 50  0000 L CNN
-F 2 "MountingHole:MountingHole_2.2mm_M2_Pad_Via" H 18275 11925 50  0001 C CNN
-F 3 "~" H 18275 11925 50  0001 C CNN
-	1    18275 11925
-	1    0    0    -1
-$EndComp
 Connection ~ 2975 6025
 Wire Wire Line
@@
 Wire Wire Line
 	9300 10275 9300 10175
-Wire Wire Line
-	9225 10475 9300 10475
-Wire Wire Line
-	9300 10475 9300 10375
-Wire Wire Line
-	9300 10375 9225 10375
 Text GLabel 17250 9850 2    50   Output ~ 0
 3.3V
@@
 Wire Wire Line
 	9300 9875 9450 9875
-Connection ~ 9300 10375
 $Comp
-L Device:C_Small CVBus1
+L Device:C_Small CV1
 U 1 1 5ED231C7
 P 19400 10200
-F 0 "CVBus1" H 19492 10231 31  0000 L CNN
+F 0 "CV1" H 19492 10231 31  0000 L CNN
 F 1 "100n" H 19492 10169 31  0000 L CNN
 F 2 "Capacitor_SMD:C_0805_2012Metric_Pad1.15x1.40mm_HandSolder" H 19400 10200 50  0001 C CNN
@@
 $EndComp
 $Comp
-L Device:C_Small CVBus2
+L Device:C_Small CV2
 U 1 1 5ED24D83
 P 19750 10200
-F 0 "CVBus2" H 19842 10231 31  0000 L CNN
+F 0 "CV2" H 19842 10231 31  0000 L CNN
 F 1 "100n" H 19842 10169 31  0000 L CNN
 F 2 "Capacitor_SMD:C_0805_2012Metric_Pad1.15x1.40mm_HandSolder" H 19750 10200 50  0001 C CNN
@@
 $EndComp
 $Comp
-L Device:C_Small CVBus3
+L Device:C_Small CV3
 U 1 1 5ED24FA7
 P 20100 10200
-F 0 "CVBus3" H 20192 10231 31  0000 L CNN
+F 0 "CV3" H 20192 10231 31  0000 L CNN
 F 1 "100n" H 20192 10169 31  0000 L CNN
 F 2 "Capacitor_SMD:C_0805_2012Metric_Pad1.15x1.40mm_HandSolder" H 20100 10200 50  0001 C CNN
@@
 $EndComp
 $Comp
-L Device:C_Small CVBus4
+L Device:C_Small CV4
 U 1 1 5ED251CF
 P 20450 10200
-F 0 "CVBus4" H 20542 10231 31  0000 L CNN
+F 0 "CV4" H 20542 10231 31  0000 L CNN
 F 1 "1u" H 20542 10169 31  0000 L CNN
 F 2 "Capacitor_SMD:C_0805_2012Metric_Pad1.15x1.40mm_HandSolder" H 20450 10200 50  0001 C CNN
@@
 $EndComp
 $Comp
-L Device:C_Small CVBus5
+L Device:C_Small CV5
 U 1 1 5ED253F3
 P 20800 10200
-F 0 "CVBus5" H 20892 10231 31  0000 L CNN
+F 0 "CV5" H 20892 10231 31  0000 L CNN
 F 1 "4.7u" H 20892 10169 31  0000 L CNN
 F 2 "Capacitor_SMD:C_0805_2012Metric_Pad1.15x1.40mm_HandSolder" H 20800 10200 50  0001 C CNN
@@
 	9225 9675 9675 9675
 Wire Wire Line
-	9300 10375 9475 10375
-Wire Wire Line
 	9750 10475 9675 10475
-Wire Wire Line
-	9475 10475 9300 10475
-Connection ~ 9300 10475
 Text GLabel 9750 10475 2    50   Output ~ 0
 5V
@@
 Text GLabel 21450 3600 2    50   Input ~ 0
 Row3
-Text GLabel 21450 4750 2    50   Input ~ 0
+Text GLabel 21450 4000 2    50   Input ~ 0
 Row2
 Wire Wire Line
-	21450 4750 21375 4750
+	21450 4000 21375 4000
 Text GLabel 21450 4950 2    50   Input ~ 0
 Row4
@@
 Wire Wire Line
 	21450 3600 21375 3600
-Text GLabel 21450 5500 2    50   Input ~ 0
+Text GLabel 21450 5600 2    50   Input ~ 0
 Col7
 Wire Wire Line
@@
 	1    0    0    -1
 $EndComp
-Text GLabel 19100 4450 0    50   Input ~ 0
+Text GLabel 21450 5050 2    50   Input ~ 0
 Col12
 Text GLabel 19125 4800 0    50   Input ~ 0
@@
 Wire Wire Line
 	21450 5700 21375 5700
-Text GLabel 21450 5600 2    50   Input ~ 0
+Text GLabel 21450 5500 2    50   Input ~ 0
 Col8
 Wire Wire Line
@@
 Wire Wire Line
 	21450 5400 21375 5400
-Text GLabel 21450 4000 2    50   Input ~ 0
+Text GLabel 21450 4750 2    50   Input ~ 0
 Row1
 Wire Wire Line
-	21450 4000 21375 4000
+	21450 4750 21375 4750
 Wire Wire Line
 	21475 5300 21375 5300
@@
 Wire Wire Line
 	16325 6350 16400 6350
-Text GLabel 21450 4850 2    50   Input ~ 0
+Text GLabel 21450 4550 2    50   Input ~ 0
 EncA
-Text GLabel 21450 4650 2    50   Input ~ 0
+Text GLabel 21450 4450 2    50   Input ~ 0
 EncB
 Wire Wire Line
-	21450 4650 21375 4650
+	21450 4450 21375 4450
 Wire Wire Line
-	21375 4850 21450 4850
+	21375 4550 21450 4550
 $Comp
 L acheronSymbols:STM32F303CCT6 U1
@@
 	21375 4100 21450 4100
 Wire Wire Line
-	19100 4450 19175 4450
+	21450 5050 21375 5050
 Text GLabel 21450 4300 2    50   Input ~ 0
 Extra1
@@
 Text GLabel 21450 3850 2    50   Input ~ 0
 Extra7
-Text GLabel 21450 4450 2    50   Input ~ 0
+Text GLabel 21450 4650 2    50   Input ~ 0
 Extra6
-Text GLabel 21450 4550 2    50   Input ~ 0
+Text GLabel 21450 4850 2    50   Input ~ 0
 Extra5
 Wire Wire Line
-	21450 4550 21375 4550
+	21450 4850 21375 4850
 Wire Wire Line
-	21375 4450 21450 4450
+	21375 4650 21450 4650
 Wire Wire Line
 	21450 3750 21375 3750
@@
 Wire Notes Line width 20
 	17900 2975 17900 4725
+Text GLabel 18700 12075 2    50   Input ~ 0
+CASE
+Wire Wire Line
+	18375 12075 18275 12075
+Wire Wire Line
+	15375 3750 15500 3750
+Text GLabel 15500 3750 2    50   Input ~ 0
+CASE
+Text GLabel 19125 4450 0    50   Input ~ 0
+SWDIO
+Wire Wire Line
+	19125 4450 19175 4450
+Text GLabel 19125 4550 0    50   Input ~ 0
+SWCLK
+Wire Wire Line
+	19125 4550 19175 4550
+$Comp
+L Connector:Conn_01x06_Male J5
+U 1 1 5CF6EE3E
+P 13125 9600
+F 0 "J5" H 13225 10175 50  0000 C CNN
+F 1 "Conn_01x06_Male" H 13275 10000 50  0000 C CNN
+F 2 "acheronConnectors:male6pinHeader" H 13125 9600 50  0001 C CNN
+F 3 "~" H 13125 9600 50  0001 C CNN
+	1    13125 9600
+	1    0    0    -1
+$EndComp
+Wire Notes Line width 20
+	12675 9125 14550 9125
+Wire Notes Line width 20
+	14550 10200 12675 10200
+Text Notes 12725 10125 0    100  Italic 20
+Serial programming
+Wire Notes Line width 20
+	14550 10200 14550 9125
+Wire Notes Line width 20
+	12675 10200 12675 9125
+$Comp
+L Device:D DESD1
+U 1 1 5D0F26E7
+P 18525 12075
+F 0 "DESD1" V 18494 12154 31  0000 L CNN
+F 1 "1N4002" V 18556 12154 31  0000 L CNN
+F 2 "Diode_SMD:D_0805_2012Metric_Pad1.15x1.40mm_HandSolder" H 18525 12075 50  0001 C CNN
+F 3 "~" H 18525 12075 50  0001 C CNN
+	1    18525 12075
+	1    0    0    -1
+$EndComp
+Wire Wire Line
+	18700 12075 18675 12075
+Connection ~ 9300 10475
+Connection ~ 9300 10375
+Wire Wire Line
+	9300 10375 9475 10375
+Wire Wire Line
+	9300 10375 9225 10375
+Wire Wire Line
+	9475 10475 9300 10475
+Wire Wire Line
+	9225 10475 9300 10475
+Wire Wire Line
+	9300 10475 9300 10375
+$Comp
+L power:GND #PWR0103
+U 1 1 5CFDFC6D
+P 13400 9400
+F 0 "#PWR0103" H 13400 9150 50  0001 C CNN
+F 1 "GND" V 13405 9272 50  0000 R CNN
+F 2 "" H 13400 9400 50  0001 C CNN
+F 3 "" H 13400 9400 50  0001 C CNN
+	1    13400 9400
+	0    -1   -1   0
+$EndComp
+Wire Wire Line
+	13400 9800 13325 9800
+Text GLabel 13400 9800 2    50   Input ~ 0
+SWCLK
+Text GLabel 13400 9700 2    50   Input ~ 0
+SWDIO
+Wire Wire Line
+	13325 9700 13400 9700
+Wire Wire Line
+	13325 9400 13400 9400
+Text GLabel 13400 9900 2    50   Input ~ 0
+3.3V
+Wire Wire Line
+	13325 9900 13400 9900
+Wire Wire Line
+	13400 9600 13325 9600
+Text GLabel 13400 9600 2    50   Input ~ 0
+BOOT0
+Text GLabel 13400 9500 2    50   Input ~ 0
+NRST
+Wire Wire Line
+	13325 9500 13400 9500
 $EndSCHEMATC

Commit message: [Update] Pre-release of version 3.2.1
Parts:
- removed QRST1: BC847, Package_TO_SOT_SMD:SOT-23, symbol Transistor_BJT:BC847
- added QRST1: DTC123J, Package_TO_SOT_SMD:SOT-23, symbol Transistor_BJT:DTC123J
- CRST1: value 4.7n -> 10u
- DESD1: value 1N4002 -> 1N4007
Other:
- moved on the sheet: CRST1, DRST1, RRST1, SWRST1
Changed lines of the file:
@@
 L Switch:SW_Push SWRST1
 U 1 1 5E070BED
-P 15725 8050
-F 0 "SWRST1" H 15725 8250 31  0000 C CNN
-F 1 "SW_Push" H 15725 8229 31  0001 C CNN
-F 2 "smdPushBtn:smdPushBtn" H 15725 8250 50  0001 C CNN
-F 3 "" H 15725 8250 50  0001 C CNN
-	1    15725 8050
+P 15725 8275
+F 0 "SWRST1" H 15725 8475 31  0000 C CNN
+F 1 "SW_Push" H 15725 8454 31  0001 C CNN
+F 2 "smdPushBtn:smdPushBtn" H 15725 8475 50  0001 C CNN
+F 3 "" H 15725 8475 50  0001 C CNN
+	1    15725 8275
 	1    0    0    -1
 $EndComp
@@
 L Device:D DRST1
 U 1 1 5E071566
-P 16225 8050
-F 0 "DRST1" V 16194 8129 31  0000 L CNN
-F 1 "1N4148" V 16256 8129 31  0000 L CNN
-F 2 "Diode_SMD:D_0805_2012Metric_Pad1.15x1.40mm_HandSolder" H 16225 8050 50  0001 C CNN
-F 3 "~" H 16225 8050 50  0001 C CNN
-	1    16225 8050
+P 16225 8275
+F 0 "DRST1" V 16194 8354 31  0000 L CNN
+F 1 "1N4148" V 16256 8354 31  0000 L CNN
+F 2 "Diode_SMD:D_0805_2012Metric_Pad1.15x1.40mm_HandSolder" H 16225 8275 50  0001 C CNN
+F 3 "~" H 16225 8275 50  0001 C CNN
+	1    16225 8275
 	-1   0    0    1
 $EndComp
@@
 L Device:R_Small RRST1
 U 1 1 5E07225E
-P 16500 8250
-F 0 "RRST1" H 16350 8150 31  0000 L CNN
-F 1 "100k" V 16500 8200 31  0000 L CNN
-F 2 "Resistor_SMD:R_1206_3216Metric_Pad1.42x1.75mm_HandSolder" H 16500 8250 50  0001 C CNN
-F 3 "~" H 16500 8250 50  0001 C CNN
-	1    16500 8250
+P 16500 8475
+F 0 "RRST1" V 16425 8400 31  0000 L CNN
+F 1 "100k" V 16500 8425 31  0000 L CNN
+F 2 "Resistor_SMD:R_1206_3216Metric_Pad1.42x1.75mm_HandSolder" H 16500 8475 50  0001 C CNN
+F 3 "~" H 16500 8475 50  0001 C CNN
+	1    16500 8475
 	1    0    0    -1
 $EndComp
@@
 L Device:C_Small CRST1
 U 1 1 5E072855
-P 16650 8250
-F 0 "CRST1" H 16600 8175 31  0000 R CNN
-F 1 "4.7n" H 16625 8325 31  0000 R CNN
-F 2 "Capacitor_SMD:C_0805_2012Metric_Pad1.15x1.40mm_HandSolder" H 16650 8250 50  0001 C CNN
-F 3 "~" H 16650 8250 50  0001 C CNN
-	1    16650 8250
+P 16650 8475
+F 0 "CRST1" H 16600 8400 31  0000 R CNN
+F 1 "10u" H 16625 8550 31  0000 R CNN
+F 2 "Capacitor_SMD:C_0805_2012Metric_Pad1.15x1.40mm_HandSolder" H 16650 8475 50  0001 C CNN
+F 3 "~" H 16650 8475 50  0001 C CNN
+	1    16650 8475
 	-1   0    0    1
 $EndComp
@@
 L power:GND #PWR09
 U 1 1 5E65C8C3
-P 16500 8400
-F 0 "#PWR09" H 16500 8150 50  0001 C CNN
-F 1 "GND" H 16505 8241 31  0000 C CNN
-F 2 "" H 16500 8400 50  0001 C CNN
-F 3 "" H 16500 8400 50  0001 C CNN
-	1    16500 8400
+P 16500 8625
+F 0 "#PWR09" H 16500 8375 50  0001 C CNN
+F 1 "GND" H 16505 8466 31  0000 C CNN
+F 2 "" H 16500 8625 50  0001 C CNN
+F 3 "" H 16500 8625 50  0001 C CNN
+	1    16500 8625
 	1    0    0    -1
 $EndComp
@@
 L power:GND #PWR011
 U 1 1 5E65CDAB
-P 16650 8400
-F 0 "#PWR011" H 16650 8150 50  0001 C CNN
-F 1 "GND" H 16655 8241 31  0000 C CNN
-F 2 "" H 16650 8400 50  0001 C CNN
-F 3 "" H 16650 8400 50  0001 C CNN
-	1    16650 8400
-	1    0    0    -1
-$EndComp
-Wire Wire Line
-	16650 8400 16650 8350
-Wire Wire Line
-	16500 8400 16500 8350
-Wire Wire Line
-	15925 8050 16000 8050
-Wire Wire Line
-	16000 7975 16000 8050
-Connection ~ 16000 8050
-Wire Wire Line
-	16000 8050 16075 8050
+P 16650 8625
+F 0 "#PWR011" H 16650 8375 50  0001 C CNN
+F 1 "GND" H 16655 8466 31  0000 C CNN
+F 2 "" H 16650 8625 50  0001 C CNN
+F 3 "" H 16650 8625 50  0001 C CNN
+	1    16650 8625
+	1    0    0    -1
+$EndComp
+Wire Wire Line
+	16650 8625 16650 8575
+Wire Wire Line
+	16500 8625 16500 8575
 Wire Wire Line
 	15750 7675 15800 7675
 Wire Wire Line
-	16375 8050 16500 8050
-Wire Wire Line
-	16650 8050 16650 8150
-Connection ~ 16650 8050
-Wire Wire Line
-	16650 8050 16950 8050
-Wire Wire Line
-	16500 8050 16500 8150
-Connection ~ 16500 8050
-Wire Wire Line
-	16500 8050 16650 8050
+	16375 8275 16500 8275
+Wire Wire Line
+	16650 8275 16650 8375
+Connection ~ 16650 8275
+Wire Wire Line
+	16650 8275 16950 8275
+Wire Wire Line
+	16500 8275 16500 8375
+Connection ~ 16500 8275
+Wire Wire Line
+	16500 8275 16650 8275
 Wire Wire Line
 	16650 7625 16650 7675
@@
 Text GLabel 16950 7675 2    50   BiDi ~ 0
 NRST
-Text GLabel 16950 8050 2    50   BiDi ~ 0
+Text GLabel 16950 8275 2    50   BiDi ~ 0
 BOOT0
 Text GLabel 19125 5450 0    50   Input ~ 0
@@
 Wire Wire Line
 	19125 5600 19175 5600
-Wire Notes Line width 20
-	17425 7125 17425 8650
-Wire Notes Line width 20
-	15025 8650 15025 7125
 Text Notes 15100 7300 0    100  Italic 20
 Hard reset circuit
@@
 Wire Wire Line
 	11200 12225 11250 12225
-$Comp
-L Transistor_BJT:BC847 QRST1
-U 1 1 5D237915
-P 16000 7775
-F 0 "QRST1" V 16284 7775 31  0000 C CNN
-F 1 "BC847" V 16222 7775 31  0000 C CNN
-F 2 "Package_TO_SOT_SMD:SOT-23" H 16200 7700 50  0001 L CIN
-F 3 "http://www.infineon.com/dgdl/Infineon-BC847SERIES_BC848SERIES_BC849SERIES_BC850SERIES-DS-v01_01-en.pdf?fileId=db3a304314dca389011541d4630a1657" H 16000 7775 50  0001 L CNN
-	1    16000 7775
-	0    1    -1   0
-$EndComp
 Wire Notes Line
 	7975 12250 8525 12250
@@
 Wire Notes Line
 	7975 12250 7975 13225
-Text GLabel 15525 8050 0    50   Input ~ 0
+Text GLabel 15525 8275 0    50   Input ~ 0
 3.3V
 Text GLabel 21450 6150 2    50   Input ~ 0
@@
 Wire Notes Line width 20
 	15025 7125 17425 7125
-Wire Notes Line width 20
-	15025 8650 17425 8650
 Wire Notes Line width 20
 	15150 9050 18000 9050
@@
 P 18525 12075
 F 0 "DESD1" V 18494 12154 31  0000 L CNN
-F 1 "1N4002" V 18556 12154 31  0000 L CNN
+F 1 "1N4007" V 18556 12154 31  0000 L CNN
 F 2 "Diode_SMD:D_0805_2012Metric_Pad1.15x1.40mm_HandSolder" H 18525 12075 50  0001 C CNN
 F 3 "~" H 18525 12075 50  0001 C CNN
@@
 Wire Wire Line
 	13325 9500 13400 9500
+Wire Notes Line width 20
+	17425 7125 17425 8900
+Wire Notes Line width 20
+	15025 7125 15025 8900
+Wire Notes Line width 20
+	15025 8900 17450 8900
+$Comp
+L Transistor_BJT:DTC123J QRST1
+U 1 1 5D249555
+P 16000 7775
+F 0 "QRST1" V 16325 7775 50  0000 C CNN
+F 1 "DTC123J" V 16234 7775 50  0000 C CNN
+F 2 "Package_TO_SOT_SMD:SOT-23" H 16000 7775 50  0001 L CNN
+F 3 "" H 16000 7775 50  0001 L CNN
+	1    16000 7775
+	0    1    -1   0
+$EndComp
+Wire Wire Line
+	15925 8275 16000 8275
+Wire Wire Line
+	16000 8025 16000 8275
+Connection ~ 16000 8275
+Wire Wire Line
+	16000 8275 16075 8275
 $EndSCHEMATC

Commit message: [Update] Pre-release of version 3.2.2
Parts:
- J1: symbol shark-rescue:USB_C_Receptacle-Connector -> shark-rescue:USB_C_Receptacle-Connector-shark-rescue
Changed lines of the file:
@@
 Sheet 1 1
 Title "SharkPCB"
-Date "2019-05-20"
-Rev "3.2.0"
+Date "2019-05-21"
+Rev "3.2.2"
 Comp "Gondolin Electronics"
 Comment1 ""
@@
 	16025 9850 16250 9850
 $Comp
-L shark-rescue:USB_C_Receptacle-Connector J1
+L shark-rescue:USB_C_Receptacle-Connector-shark-rescue J1
 U 1 1 5CC01BA3
 P 8625 10675
@@
 U 1 1 5E5BA0B3
 P 9575 10175
-F 0 "RD-1" V 9500 10150 31  0000 L CNN
+F 0 "RD-1" V 9500 10110 31  0000 L CNN
 F 1 "22R" V 9575 10125 31  0000 L CNN
 F 2 "Resistor_SMD:R_1206_3216Metric_Pad1.42x1.75mm_HandSolder" H 9575 10175 50  0001 C CNN
@@
 U 1 1 5E5BB8E0
 P 9575 10375
-F 0 "RD+1" V 9500 10350 31  0000 L CNN
+F 0 "RD+1" V 9500 10310 31  0000 L CNN
 F 1 "22R" V 9575 10325 31  0000 L CNN
 F 2 "Resistor_SMD:R_1206_3216Metric_Pad1.42x1.75mm_HandSolder" H 9575 10375 50  0001 C CNN
@@
 U 1 1 5EA2CF13
 P 9550 9875
-F 0 "RCC1" V 9475 9850 31  0000 L CNN
+F 0 "RCC1" V 9475 9815 31  0000 L CNN
 F 1 "5.1k" V 9550 9825 31  0000 L CNN
 F 2 "Resistor_SMD:R_1206_3216Metric_Pad1.42x1.75mm_HandSolder" H 9550 9875 50  0001 C CNN
@@
 U 1 1 5EA80DA8
 P 9575 10475
-F 0 "RD+Up1" V 9650 10400 31  0000 L CNN
+F 0 "RD+Up1" V 9650 10380 31  0000 L CNN
 F 1 "1.5k" V 9575 10425 31  0000 L CNN
 F 2 "Resistor_SMD:R_1206_3216Metric_Pad1.42x1.75mm_HandSolder" H 9575 10475 50  0001 C CNN

Commit message: [Update] Made changes to routing
Parts:
- J1: symbol shark-rescue:USB_C_Receptacle-Connector-shark-rescue -> shark-rescue:USB_C_Receptacle-Connector-shark-rescue-shark-rescue
Changed lines of the file:
@@
 Title "SharkPCB"
 Date "2019-05-21"
-Rev "3.2.2"
+Rev "3.2.3"
 Comp "Gondolin Electronics"
 Comment1 ""
@@
 	16025 9850 16250 9850
 $Comp
-L shark-rescue:USB_C_Receptacle-Connector-shark-rescue J1
+L shark-rescue:USB_C_Receptacle-Connector-shark-rescue-shark-rescue J1
 U 1 1 5CC01BA3
 P 8625 10675
