File: kicadFiles/shark.kicad_sch (KiCad schematic)
At the start: 291 parts, among them J1 TYPE-C-31-M12_13, J2 ARM JTAG, Q1 DTC123JKAT146, Q2 AO3401A, Q3 DTC123JKAT146, SW1 ESC, SW10 O, SW11 P, SW12 BKSP, SW13 TAB, SW14 A, SW15 S, SW16 D, SW17 F, SW18 G, SW19 H, SW2 Q, SW20 J, SW21 K, SW22 L, SW23 COLON, SW24 QUOTE, SW25 SHIFT, SW26 Z, SW27 X, SW28 C, SW29 V, SW3 W, SW30 B, SW31 N, SW32 M, SW33 COMMA, SW34 DOT, SW35 SLSH, SW36 ENTER, SW37 CTRL, SW38 Q, SW39 WIN, SW4 E, SW40 ALT, SW41 F1, SW42 SPC_100, SW43 SPC_100, SW44 F2, SW45 LEFT, SW46 DOWN, SW47 UP, SW48 RIGHT, SW49 SPC_200, SW5 R, SW50 SPC_200, SW51 SPC_200, SW52 SPC_600, SW53 SPC_700, SW54 ALT_125, SW55 CTRL_125, SW56 ALT_125, SW57 CTRL_125, SW6 T, SW7 Y, SW8 U, SW9 I, U1 STM32F072CBT6, U2 USBLC6-2SC6, U3 MCP1700T-3302E/TT, U4 TXS0101

Commit message: Mounting holes, MCU, 3v3, grounding, LEDs
- Introduced Wurth SMD mounting standoffs and case grounding through a ferite bead on one of the standoffs
- Routed MCU with copper zones
- Routed 3V3 LDO circuit
- Routed first row with diodes and LEDs and LED resistors
- Added zone cutout on ground copper fill under USB connector
- Added USBC shield grounding through ferrite bead
Parts:
- removed SW52: SPC_600, acheron_MX_SolderMask:MX600R, symbol acheronSymbols:MXSwitch
- removed SW53: SPC_700, acheron_MX_SolderMask:MX700R, symbol acheronSymbols:MXSwitch
- removed SW54, SW56: ALT_125, acheron_MX_SolderMask:MX125, symbol acheronSymbols:MXSwitch
- removed SW55, SW57: CTRL_125, acheron_MX_SolderMask:MX125, symbol acheronSymbols:MXSwitch
- added H1: MountingHole_Pad, acheron_Hardware:9774030243R, symbol Mechanical:MountingHole_Pad
- added H2, H3, H4, H5, H6: MountingHole, acheron_Hardware:9774030243R, symbol Mechanical:MountingHole
- added L1, L2: 120R@100MHz, Inductor_SMD:L_1206_3216Metric_Pad1.42x1.75mm_HandSolder, symbol Device:L_Core_Ferrite
- added Q4: MMBFJ270, Package_TO_SOT_SMD:SOT-23, symbol Device:Q_PJFET_DSG
- added R77: 10k, acheron_Components:R_SMD_1206, symbol Device:R_Small
- C14: Specification MLCC 10V -> MLCC 5% 10V
- R10, R11: Specification (none) -> 1% 1/8W
Connections:
- net R1_S1 is gone; now on net C0: ROT1.S1
- net R2_S1 is gone; now on net C11: ROT2.S1
- net 3V3: now also C5.2, C6.2, U1.36 (VDDIO2)
- net BOOT0: now also R77.2
- net GND: now also L1.1, L2.1, Q4.2 (S)
- net R1: now also D13.1 (K), D14.1 (K), D15.1 (K), D16.1 (K), D17.1 (K), D18.1 (K), D19.1 (K), D20.1 (K), D21.1 (K), D22.1 (K), D23.1 (K), D24.1 (K)
- net R1_S2: now also D1.2 (A), SW1.2 (Row)
- net R2_S2: now also D12.2 (A), SW12.2 (Row)
- net R0: now reaches D1.1 (K), D10.1 (K), D11.1 (K), D12.1 (K), D2.1 (K), D3.1 (K), D4.1 (K), D5.1 (K), D6.1 (K), D7.1 (K), D8.1 (K), D9.1 (K)
- net C3: now reaches SW16.1 (Col), SW28.1 (Col), SW40.1 (Col)
- net C3: now also SW4.2 (Row); no longer SW4.1 (Col)
- net C10: now reaches SW11.1 (Col), SW23.1 (Col), SW35.1 (Col), SW47.1 (Col)
- net C4: now reaches SW17.1 (Col), SW29.1 (Col), SW41.1 (Col), SW5.1 (Col)
- net R2: now reaches D25.1 (K), D26.1 (K), D27.1 (K), D28.1 (K), D29.1 (K), D30.1 (K), D31.1 (K), D32.1 (K), D33.1 (K), D34.1 (K), D35.1 (K), D36.1 (K)
- net R3: now reaches D37.1 (K), D38.1 (K), D39.1 (K), D40.1 (K), D41.1 (K), D42.1 (K), D43.1 (K), D44.1 (K), D45.1 (K), D46.1 (K), D47.1 (K), D48.1 (K)
- net C9: now reaches SW10.1 (Col), SW22.1 (Col), SW34.1 (Col), SW46.1 (Col)
- net C2: now reaches SW15.1 (Col), SW27.1 (Col), SW3.1 (Col), SW39.1 (Col)
- net C8: now reaches SW21.1 (Col), SW33.1 (Col), SW45.1 (Col), SW9.1 (Col)
- net C11: now reaches SW12.1 (Col), SW24.1 (Col), SW36.1 (Col), SW48.1 (Col)
- net C5: now reaches SW18.1 (Col), SW30.1 (Col), SW42.1 (Col), SW50.1 (Col), SW6.1 (Col)
- net at D4.2 (A): now also SW4.1 (Col); no longer SW4.2 (Row)
- net C6: now reaches SW19.1 (Col), SW31.1 (Col), SW43.1 (Col), SW49.1 (Col), SW51.1 (Col), SW7.1 (Col)
- net GNDPWR: now reaches J1.S (SHIELD)
- net GNDPWR: now also L2.2
- net C7: now reaches SW20.1 (Col), SW32.1 (Col), SW44.1 (Col), SW8.1 (Col)
- net C0: now reaches SW1.1 (Col), SW13.1 (Col), SW25.1 (Col), SW37.1 (Col)
- net C1: now reaches SW14.1 (Col), SW2.1 (Col), SW26.1 (Col), SW38.1 (Col)
- net at D52.2 (A), Q1.1 (B), S1.2 (B): now also Q4.3 (G)
- new net: Q4.1 (D), R77.1
- new net: H1.1, L1.2
Other:
- moved on the sheet: C11, C14, D52, Q1, R10, R11, R7, S1, SW4

Commit message: Route 4th row, remove unusable LEDs, re-centered RGBs in 4th row
Parts:
- removed LED38, LED39, LED52, LED54: LED, acheron_Components:LED_THT_2.54mm, symbol acheronSymbols:LED
- removed R61, R63, R67, R69: 420R, acheron_Components:R_SMD_1206, symbol Device:R
- LED37: now in the parts list
Connections:
- net C0: now also SW37.2 (Row); no longer SW37.1 (Col)
- net C2: now also SW15.2 (Row); no longer SW15.1 (Col)
- net at LED48.A, R60.1: no longer LED37.A
- net at D15.2 (A): now also SW15.1 (Col); no longer SW15.2 (Row)
- net at LED43.A: now also LED42.A, R66.1
- net at LED47.A, R71.1: now also LED49.A
- net at R62.1: now also LED37.A
- net at D37.2 (A): now also SW37.1 (Col); no longer SW37.2 (Row)
- net at LED44.A, R68.1: now also LED45.A
Other:
- moved on the sheet: SW15, SW37
