File: kicadFiles/shark.kicad_sch (KiCad schematic)
At the start: 268 parts, among them J1 TYPE-C-31-M12_13, J2 Conn_01x04_Male, J3 Conn_01x04_Male, J4 Conn_01x04_Male, J5 Conn_01x06_Male, Q1 AO4406AL, SW1 MXSwitch, SW10 MXSwitch, SW11 MXSwitch, SW12 MXSwitch, SW13 MXSwitch, SW14 MXSwitch, SW15 MXSwitch, SW16 MXSwitch, SW17 MXSwitch, SW18 MXSwitch, SW19 MXSwitch, SW2 MXSwitch, SW20 MXSwitch, SW21 MXSwitch, SW22 MXSwitch, SW23 MXSwitch, SW24 MXSwitch, SW25 MXSwitch, SW26 MXSwitch, SW27 MXSwitch, SW28 MXSwitch, SW29 MXSwitch, SW3 MXSwitch, SW30 MXSwitch, SW31 MXSwitch, SW32 MXSwitch, SW33 MXSwitch, SW34 MXSwitch, SW35 MXSwitch, SW36 MXSwitch, SW37 MXSwitch, SW38 MXSwitch, SW39 MXSwitch, SW4 MXSwitch, SW40 MXSwitch, SW41 MXSwitch, SW42 MXSwitch, SW43 MXSwitch, SW44 MXSwitch, SW45 MXSwitch, SW46 MXSwitch, SW47 MXSwitch, SW48 MXSwitch, SW49 MXSwitch, SW5 MXSwitch, SW50 MXSwitch, SW51 MXSwitch, SW6 MXSwitch, SW7 MXSwitch, SW8 MXSwitch, SW9 MXSwitch, U1 STM32F303-LQFP48, U2 MCP1700-3302E_SOT23, U3 USBLC6-2SC6, Y1 8MHz

Commit message: Connect USB pullup to 3V3 on schematic
Parts:
- RPU1: value 5.1k -> 1.5k
Connections:
- net 3.3V: now also RPU1.1
- net VBUS: no longer RPU1.1
Changed lines of the file:
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@@
     )
   )
-  (global_label "VBUS" (shape output) (at 247.65 285.115 0) (fields_autoplaced)
+  (global_label "3.3V" (shape output) (at 247.65 285.115 0) (fields_autoplaced)
     (effects (font (size 1.27 1.27)) (justify left))
-    (property "Intersheet References" "${INTERSHEET_REFS}" (id 0) (at 0 0 0)
-      (effects (font (size 1.27 1.27)) hide)
+    (property "Intersheet References" "${INTERSHEET_REFS}" (id 0) (at 254.0866 285.0356 0)
+      (effects (font (size 1.27 1.27)) (justify left) hide)
     )
   )
@@
       (effects (font (size 0.7874 0.7874)) (justify left))
     )
-    (property "Value" "5.1k" (id 1) (at 241.935 285.115 90)
+    (property "Value" "1.5k" (id 1) (at 241.935 285.115 90)
       (effects (font (size 0.7874 0.7874)) (justify left))
     )
@@
     )
     (path "/00000000-0000-0000-0000-00005ea80da8"
-      (reference "RPU1") (unit 1) (value "5.1k") (footprint "acheronComponents:R_1026")
+      (reference "RPU1") (unit 1) (value "1.5k") (footprint "acheronComponents:R_1026")
     )
     (path "/00000000-0000-0000-0000-00005e07225e"
