File: plate/basePlate/basePlate.kicad_pcb (KiCad board)
At the start: 2 copper layers, 233 x 81 mm, 0 parts

Commit message: [Fix, Feature] Added frill file to PCB gerbers and added Shark logo to base plate
Parts:
- added G***: LOGO, sharkLogo:sharkPlated, F.Cu at (136.5, 111.3)
- added G***: LOGO, sharkLogo:sharkLogo, F.Cu at (41.5, 73.3)

Commit message: [Feature] Added Shark logo to base plate
Parts:
- removed the G*** at (41.5, 73.3)
