File: plate/hiPro/universal/universal.kicad_pcb (KiCad board)
At the start: 2 copper layers, 227.4 x 75.4 mm, 45 parts

Commit message: [Update] Updated universal hi-pro plate STEP file
Parts:
- turned REF** to 180 degrees (x15)
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Routing:
- net (no net): vias 7 -> 11
