File: plate/base/base.kicad_pcb (KiCad board)
At the start: 2 copper layers, 233 x 81 mm, 1 part

Commit message: [Fix] Adjusted base plate and made its shark logo plated
Parts:
- added G***: LOGO, sharkLogo:sharkLetters, F.Cu at (71.0, 100.0)
- moved G*** 38.2 mm to (170.0, 93.0), turned to 115 degrees
Routing:
- net (no net): vias 11 -> 5
Other:
- board size 233 x 81 mm -> 231.6 x 79.2 mm
