File: plate/lowProfile/lowProfile.kicad_pcb (KiCad board)
At the start: 2 copper layers, 231.6 x 79.2 mm, 45 parts

Commit message: [Fix] Adjusted base plate and made its shark logo plated
Routing:
- net (no net): vias 5 -> 11
Changed lines of the file:
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@@
     (thickness 1.6)
     (drawings 11)
-    (tracks 5)
+    (tracks 11)
     (zones 0)
     (modules 45)
@@
       (drillshape 0)
       (scaleselection 1)
-      (outputdirectory "../../../gerbers/plates/loPro/universal/"))
+      (outputdirectory "../../gerbers/plates/lopro/"))
   )
   (net 0 "")
@@
   (via (at 54.9914 119.05332) (size 4) (drill 2.5) (layers F.Cu B.Cu) (net 0))
   (via (at 54.9914 81.05268) (size 4) (drill 2.5) (layers F.Cu B.Cu) (net 0))
+  (via (at 54.9914 100) (size 6) (drill 4) (layers F.Cu B.Cu) (net 0))
+  (via (at 92.85 80.95) (size 6) (drill 4) (layers F.Cu B.Cu) (net 0))
+  (via (at 92.85 119.05) (size 6) (drill 4) (layers F.Cu B.Cu) (net 0))
+  (via (at 245.25 100) (size 6) (drill 4) (layers F.Cu B.Cu) (net 0))
+  (via (at 207.15 80.95) (size 6) (drill 4) (layers F.Cu B.Cu) (net 0))
+  (via (at 207.15 119.05) (size 6) (drill 4) (layers F.Cu B.Cu) (net 0))
 )
