File: kicad_files/shark.kicad_sch (KiCad schematic)
At the start: 454 parts, among them J1 TYPE-C-31-M12, J2 SM04B-SRSS-TB(LF)(SN), J3 SM04B-SRSS-TB(LF)(SN), Q1 2N7002, Q2 2N7002, Q3 AO3401A, Q4 2N7002, Q5 2N7002, SW1 K2-1187SQ-A4SW-06, SW10 MX Switch, SW11 MX Switch, SW12 MX Switch, SW13 MX Switch, SW14 MX Switch, SW15 MX Switch, SW16 MX Switch, SW17 MX Switch, SW18 MX Switch, SW19 MX Switch, SW2 MX Switch, SW20 MX Switch, SW21 MX Switch, SW22 MX Switch, SW23 MX Switch, SW24 MX Switch, SW25 MX Switch, SW26 MX Switch, SW27 MX Switch, SW28 MX Switch, SW29 MX Switch, SW3 MX Switch, SW30 MX Switch, SW31 MX Switch, SW32 MX Switch, SW33 MX Switch, SW34 MX Switch, SW35 MX Switch, SW36 MX Switch, SW37 MX Switch, SW38 MX Switch, SW39 MX Switch, SW4 MX Switch, SW40 MX Switch, SW41 MX Switch, SW42 MX Switch, SW43 MX Switch, SW44 MX Switch, SW45 MX Switch, SW46 MX Switch, SW47 MX Switch, SW48 MX Switch, SW49 MX Switch, SW5 MX Switch, SW6 MX Switch, SW7 MX Switch, SW8 MX Switch, SW9 MX Switch, U1 BL24C256A-SFRC, U2 STM32F411CEU6, U3 USBLC6-2SC6, U4 AT24C256C-SSHL-T, U5 SGM2007-3.3XN5/TR, U6 TXS0101DBVR, X1 ARM JTAG, X2 USB_EXPOSED_PINS, X3 MountingHole, X4 RGB_PINS, Y1 TAXM8M4RFDCET2T

Commit message: Start porting to Joker48 template
Parts:
- removed C21, C24, C25, C26, C27, C28, C29, C30, C31, C32, C33, C34, C35, C36, C37, C38, C39, C40, C41, C42, C43, C44, C45, C46, C47, C48, C49, C50, C51, C52, C53: 100n, Capacitor_SMD:C_0805_2012Metric, symbol Device:C_Small
- removed D28, D29, D30: WS2812C-2020, acheron_Components:LED_WS2812_2020_uparrow, symbol acheron_Symbols:WS2812B-2020
- removed D31, D32, D33, D34, D35, D36: WS2812C-2020, acheron_Components:LED_WS2812_2020, symbol acheron_Symbols:WS2812B-2020
- removed LED1, LED10, LED100, LED101, LED102, LED103, LED104, LED105, LED106, LED107, LED108, LED109, LED110, LED111, LED112, LED12, LED14, LED19, LED2, LED21, LED23, LED24, LED25, LED26, LED27, LED28, LED3, LED4, LED41, LED43, LED44, LED45, LED61, LED62, LED63, LED64, LED65, LED66, LED67, LED76, LED77, LED78, LED79, LED8, LED80, LED81, LED82, LED83, LED84, LED85, LED86, LED87, LED88, LED89, LED90, LED91, LED92, LED93, LED94, LED95, LED96, LED97, LED98, LED99: LED, acheron_Components:LED_THT_2.54mm, symbol acheron_Symbols:LED
- removed Q4: 2N7002, Package_TO_SOT_SMD:SOT-23, symbol Transistor_FET:2N7002
- removed R100, R101, R102, R103, R104, R105, R106, R107, R108, R109, R110, R111, R112, R113, R114, R115, R116, R117, R118, R119, R34, R36, R37, R38, R39, R52, R53, R54, R55, R56, R57, R72, R73, R74, R75, R83, R84, R85, R86, R87, R88, R89, R91, R92, R93, R95, R96, R97, R98, R99: 1k, Resistor_SMD:R_0805_2012Metric, symbol Device:R_Small
- removed R21: 100, Resistor_SMD:R_0402_1005Metric, symbol Device:R_Small
- removed R35: 10k, Resistor_SMD:R_0402_1005Metric, symbol Device:R_Small
- added C19: 100n, Capacitor_SMD:C_0402_1005Metric, symbol Device:C
- added LED49, LED50: LED, acheron_Components:LED_THT_2.54mm, symbol acheron_Symbols:LED
- added R20: 5.1R, Resistor_SMD:R_0402_1005Metric, symbol Device:R_Small
- added R63, R67, R68, R69: 1k, Resistor_SMD:R_0805_2012Metric, symbol Device:R_Small
- added U7: RS0102YH8, acheron_Components:SOT-23-8, symbol acheron_Symbols:RS0102YH8
- C22, C23: footprint Capacitor_SMD:C_0805_2012Metric -> Capacitor_SMD:C_0402_1005Metric; Manufacturer Part Number CL21B104KCFNNNE -> CL05B104KB54PNC; Package C0805 -> C0402; Specification 100V 100nF X7R ±10% 0805 MLCC -> 50V 100nF X7R ±10% 0402 MLCC; Vendor Part Number LCSC C28233 -> LCSC C307331
- D21, D22, D23, D24, D25, D26, D27: footprint acheron_Components:LED_WS2812_2020_uparrow -> acheron_Components:LED_WS2812_2020
- R19: value 10k -> 5.1R; Manufacturer Part Number 0402WGF1002TCE -> 0402WGJ033JTCE; Specification ±1% 1/16W Thick Film Resistors 50V 0402 -> ±1% 1/16W Thick Film Resistors 50V 0805; Vendor Part Number LCSC C25744 -> LCSC C25165
- renumbered C19 to C20, C20 to C21, D37 to D28, D38 to D29, D39 to D30, D40 to D31, D41 to D32, D42 to D33, D43 to D34, D44 to D35, D45 to D36, D46 to D37, D47 to D38, D48 to D39, D49 to D40, D50 to D41, D51 to D42, D52 to D43, D53 to D44, D54 to D45, D55 to D46, D56 to D47, D57 to D48, D58 to D49, D59 to D50, D60 to D51, D61 to D52, D62 to D53, D63 to D54, D64 to D55, D65 to D56, D66 to D57, D67 to D58, D68 to D59, D69 to D60, D70 to D61, D71 to D62, D72 to D63, D73 to D64, D74 to D65, D75 to D66, D76 to D67, D77 to D68, D78 to D69, D79 to D70, D80 to D71, D81 to D72, D82 to D73, D83 to D74, D84 to D75, LED5 to LED1, LED18 to LED10, LED20 to LED11, LED22 to LED12, LED29 to LED13, LED30 to LED14, LED31 to LED15, LED32 to LED16, LED33 to LED17, LED34 to LED18, LED35 to LED19, LED6 to LED2, LED36 to LED20, LED37 to LED21, LED38 to LED22, LED39 to LED23, LED40 to LED24, LED68 to LED25, LED69 to LED26, LED49 to LED27, LED50 to LED28, LED51 to LED29, LED7 to LED3, LED52 to LED30, LED53 to LED31, LED54 to LED32, LED55 to LED33, LED56 to LED34, LED57 to LED35, LED58 to LED36, LED59 to LED37, LED60 to LED38, LED70 to LED39, LED9 to LED4, LED71 to LED40, LED72 to LED41, LED73 to LED43, LED74 to LED44, LED75 to LED45, LED11 to LED5, LED13 to LED6, LED15 to LED7, LED16 to LED8, LED17 to LED9, Q5 to Q4, R2 to R1, R1 to R2, R20 to R21, R40 to R34, R41 to R35, R42 to R36, R43 to R37, R44 to R38, R45 to R39, R46 to R40, R47 to R41, R48 to R42, R49 to R43, R50 to R44, R51 to R45, R76 to R46, R58 to R47, R59 to R48, R60 to R49, R61 to R50, R62 to R51, R63 to R52, R64 to R53, R65 to R54, R66 to R55, R67 to R56, R68 to R57, R69 to R58, R90 to R59, R77 to R60, R78 to R61, R79 to R62, R80 to R64, R81 to R65, R82 to R66, R94 to R72
Connections:
- net 3V3: now also C19.2, U7.4 (OE), U7.8 (VCCA)
- net 5V: now also R20.2, U7.1 (VCCB); no longer C22.1, C23.1, D10.4 (VDD), D11.4 (VDD), D12.4 (VDD), D13.4 (VDD), D14.4 (VDD), D15.4 (VDD), D16.4 (VDD), D17.4 (VDD), D18.4 (VDD), D19.4 (VDD), D20.4 (VDD), D21.4 (VDD), D22.4 (VDD), D23.4 (VDD), D24.4 (VDD), D25.4 (VDD), D26.4 (VDD), D27.4 (VDD), D4.4 (VDD), D5.4 (VDD), D6.4 (VDD), D7.4 (VDD), D8.4 (VDD), D9.4 (VDD), U6.6 (VCCB)
- net D+: now also U3.1 (I/O1); no longer U3.3 (I/O2)
- net D-: now also U3.3 (I/O2); no longer U3.1 (I/O1)
- net DBUS+: now also U3.6 (I/O1); no longer U3.4 (I/O2)
- net DBUS-: now also U3.4 (I/O2); no longer U3.6 (I/O1)
- net GND: now also LED46.K, LED47.K, LED48.K, C19.1, LED49.K, LED50.K, U7.5 (GND); no longer U6.2 (GND)
- net RGB_3V3: now also U7.7 (A1); no longer U6.3 (A)
- net SCL: now also R2.1; no longer R1.1
- net SDA: now also R1.1; no longer R2.1
- net XTAL_IN: now also Y1.1; no longer Y1.3
- net XTAL_OUT: now also Y1.3; no longer Y1.1
- net at Q3.3 (D), R22.1, R23.1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: now also R63.1, R67.1, R68.1, R69.1; no longer LED46.A, LED47.A, LED48.A
- net at D21.1 (DOUT): no longer D22.3 (DIN)
- net at D21.3 (DIN): no longer D20.1 (DOUT)
- net at D12.1 (DOUT): no longer D13.3 (DIN)
- net at D12.3 (DIN): no longer D11.1 (DOUT)
- net at D26.3 (DIN): no longer D25.1 (DOUT)
- net at D25.3 (DIN): no longer D24.1 (DOUT)
- net at D26.1 (DOUT): no longer D27.3 (DIN)
- net at D18.1 (DOUT): no longer D19.3 (DIN)
- net at D18.3 (DIN): no longer D17.1 (DOUT)
- net at D9.1 (DOUT): no longer D10.3 (DIN)
- net at D9.3 (DIN): no longer D8.1 (DOUT)
- net at D14.1 (DOUT): no longer D15.3 (DIN)
- net at D14.3 (DIN): no longer D13.1 (DOUT)
- net at D5.1 (DOUT): no longer D6.3 (DIN)
- net at R19.1: now also C22.1, D4.4 (VDD); no longer R21.1
- net at D22.1 (DOUT): no longer D23.3 (DIN)
- net at LED42.A: now also R63.2
- net at D7.1 (DOUT): no longer D8.3 (DIN)
- net at D7.3 (DIN): no longer D6.1 (DOUT)
- net at D15.1 (DOUT): no longer D16.3 (DIN)
- net at D11.3 (DIN): no longer D10.1 (DOUT)
- net at R70.2: now also LED49.A
- net at D17.3 (DIN): no longer D16.1 (DOUT)
- net at R71.2: now also LED50.A
- net at D23.1 (DOUT): no longer D24.3 (DIN)
- net at D19.1 (DOUT): no longer D20.3 (DIN)
- net LED_PWM renamed BACKLIGHT_3V3
- net BACKLIGHT_3V3: now also U7.6 (A2)
- net RGB_5V_MAIN: no longer names the net of U6.4 (B)
- net RGB_5V_MAIN: no longer D4.3 (DIN)
- new net: C23.1, D5.4 (VDD), R20.1
- new net: LED47.A, R68.2
- new net: LED46.A, R67.2
- new net: LED48.A, R69.2
- new net BACKLIGHT_5V: R21.1, U7.3 (B2)
- new net RGB_5V: D4.3 (DIN), U7.2 (B1)
Other:
- title: Noxary X60 -> SharkPCB
- moved on the sheet: C20, LED1, LED10, LED11, LED12, LED13, LED14, LED15, LED16, LED17, LED18, LED19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

Commit message: Routing job
Parts:
- removed C1: 100n, Capacitor_SMD:C_0402_1005Metric, symbol Device:C_Small
- removed U1: BL24C256A-SFRC, acheron_Components:TSSOP-8_4.4x3mm_P0.65mm, symbol Memory_EEPROM:24LC256
- added C23, C24, C25, C26, C27, C28: 100n, Capacitor_SMD:C_0402_1005Metric, symbol Device:C_Small
- added R21, R22, R23, R24, R25, R26: 5.1R, Resistor_SMD:R_0402_1005Metric, symbol Device:R_Small
- renumbered C2 to C1, C11 to C10, C12 to C11, C13 to C12, C14 to C13, C15 to C14, C16 to C15, C17 to C16, C18 to C17, C19 to C18, C20 to C19, C3 to C2, C21 to C20, C22 to C21, C23 to C22, C4 to C3, C5 to C4, C6 to C5, C7 to C6, C8 to C7, C9 to C8, C10 to C9, R21 to R27, R22 to R28, R23 to R29, R24 to R30, R25 to R31, R26 to R32, R27 to R33, R28 to R34, R29 to R35, R30 to R36, R31 to R37, R32 to R38, R33 to R39, R34 to R40, R35 to R41, R36 to R42, R37 to R43, R38 to R44, R39 to R45, R40 to R46, R41 to R47, R42 to R48, R43 to R49, R44 to R50, R45 to R51, R46 to R52, R47 to R53, R48 to R54, R49 to R55, R50 to R56, R51 to R57, R52 to R58, R53 to R59, R54 to R60, R55 to R61, R56 to R62, R57 to R63, R58 to R64, R59 to R65, R60 to R66, R61 to R67, R62 to R68, R63 to R69, R64 to R70, R65 to R71, R66 to R72, R67 to R73, R68 to R74, R69 to R75, R70 to R76, R71 to R77, R72 to R78, U2 to U1, U3 to U2, U4 to U3, U5 to U4, U6 to U5, U7 to U6
Connections:
- net 5V: now also R21.2, R22.2, R23.2, R24.2, R25.2, R26.2
- net C0: now also U1.29 (PA8)
- net C1: now also U1.31 (PA10)
- net GND: now also C23.2, C24.2, C25.2, C26.2, C27.2, C28.2
- net at D9.1 (DOUT): now also D10.3 (DIN)
- net at D9.3 (DIN): now also D8.1 (DOUT)
- net at D9.4 (VDD): now also C26.1, R24.1
- net at D5.1 (DOUT): now also D6.3 (DIN)
- net at D7.1 (DOUT): now also D8.3 (DIN)
- net at D7.3 (DIN): now also D6.1 (DOUT)
- net at D7.4 (VDD): now also C24.1, R22.1
- net at D8.4 (VDD): now also C25.1, R23.1
- net at D6.4 (VDD): now also C23.1, R21.1
- net at D11.3 (DIN): now also D10.1 (DOUT)
- net at D11.4 (VDD): now also C28.1, R26.1
- net at D10.4 (VDD): now also C27.1, R25.1

Commit message: More routing
Parts:
- removed C17: 100n, Capacitor_SMD:C_0402_1005Metric, symbol Device:C
- removed C20: 1u, Capacitor_SMD:C_0805_2012Metric, symbol Device:C
- removed D3: SMF6.0A, acheron_Components:D_SOD-123, symbol Device:D_Schottky
- removed FB2: GZ2012D601TF, Inductor_SMD:L_0805_2012Metric, symbol Device:Ferrite_Bead_Small
- removed H1: DB_RGB_PASSTHROUGH_HOLE, athena_library:rgb_daughterboard_notch_plated_8x4mm, symbol Mechanical:MountingHole_Pad
- removed J2, J3: SM04B-SRSS-TB(LF)(SN), acheron_Connectors:SM04B-SRSS-TB(LF)(SN)_mounting-reliefs, symbol Connector_Generic_MountingPin:Conn_01x04_MountingPin
- removed LED25, LED26: LED, acheron_Components:LED_THT_2.54mm, symbol acheron_Symbols:LED
- removed Q4: 2N7002, Package_TO_SOT_SMD:SOT-23, symbol Transistor_FET:2N7002
- removed R17, R78: 10k, Resistor_SMD:R_0805_2012Metric, symbol Device:R_Small
- removed R18: 10k, Resistor_SMD:R_0402_1005Metric, symbol Device:R_Small
- removed R42, R43, R52, R54, R70, R71, R72, R73: 1k, Resistor_SMD:R_0805_2012Metric, symbol Device:R_Small
- removed R65: 100, Resistor_SMD:R_0805_2012Metric, symbol Device:R_Small
- removed U5: TXS0101DBVR, acheron_Components:SOT-23-6, symbol acheronSymbols:TXS0101
- removed X3: MountingHole, MountingHole:MountingHole_2.5mm_Pad, symbol Mechanical:MountingHole_Pad
- removed X4: RGB_PINS, acheron_Connectors:PinHeader_1x3_staggered_P2.54mm_Vertical, symbol Connector_Generic:Conn_01x03
- added C27, C28, C29, C30, C31, C32, C33, C34, C35, C36, C37, C38, C39, C40, C41, C42: 100n, Capacitor_SMD:C_0402_1005Metric, symbol Device:C_Small
- added LED44, LED46, LED48: LED, acheron_Components:LED_THT_2.54mm, symbol acheron_Symbols:LED
- added R25, R26, R27, R28, R29, R30, R31, R32, R33, R34, R35, R36, R37, R38, R39, R40: 5.1R, Resistor_SMD:R_0402_1005Metric, symbol Device:R_Small
- added R64, R66, R67, R79, R80, R81, R82, R90: 1k, Resistor_SMD:R_0402_1005Metric, symbol Device:R_Small
- added SW50, SW51, SW52: MX Switch, acheron_MX_soldermask:MX200R, symbol acheronSymbols:Mechanical_Switch
- R54: renamed from R41; footprint Resistor_SMD:R_0805_2012Metric -> Resistor_SMD:R_0402_1005Metric; Manufacturer Part Number 0805W8F1001T5E -> 0402WGF1001TCE; Package R0805 -> R0402; Specification ±1% 125mW Thick Film Resistors 150V 0805 -> 1% 125mW Thick Film Resistors 150V 0805; Vendor Part Number LCSC C17513 -> LCSC C11702
- R55: footprint Resistor_SMD:R_0805_2012Metric -> Resistor_SMD:R_0402_1005Metric; Manufacturer Part Number 0805W8F1001T5E -> 0402WGF1001TCE; Package R0805 -> R0402; Specification ±1% 125mW Thick Film Resistors 150V 0805 -> 1% 125mW Thick Film Resistors 150V 0805; Vendor Part Number LCSC C17513 -> LCSC C11702
- renumbered C18 to C17, C19 to C18, C21 to C19, C22 to C20, C23 to C21, C24 to C22, C25 to C23, C26 to C24, C27 to C25, C28 to C26, D11 to D10, D12 to D11, D13 to D12, D14 to D13, D15 to D14, D16 to D15, D17 to D16, D18 to D17, D19 to D18, D20 to D19, D21 to D20, D22 to D21, D23 to D22, D24 to D23, D25 to D24, D26 to D25, D27 to D26, D28 to D27, D29 to D28, D30 to D29, D4 to D3, D31 to D30, D32 to D31, D33 to D32, D34 to D33, D35 to D34, D36 to D35, D37 to D36, D38 to D37, D39 to D38, D40 to D39, D5 to D4, D41 to D40, D42 to D41, D43 to D42, D44 to D43, D45 to D44, D46 to D45, D47 to D46, D48 to D47, D49 to D48, D50 to D49, D6 to D5, D51 to D50, D52 to D51, D53 to D52, D54 to D53, D55 to D54, D56 to D55, D57 to D56, D58 to D57, D59 to D58, D60 to D59, D7 to D6, D61 to D60, D62 to D61, D63 to D62, D64 to D63, D65 to D64, D66 to D65, D67 to D66, D68 to D67, D69 to D68, D70 to D69, D8 to D7, D71 to D70, D72 to D71, D73 to D72, D74 to D73, D75 to D74, D9 to D8, D10 to D9, H2 to H1, H3 to H2, H4 to H3, H5 to H4, H6 to H5, LED9 to LED10, LED10 to LED11, LED11 to LED12, LED16 to LED14, LED24 to LED15, LED14 to LED16, LED15 to LED17, LED17 to LED18, LED18 to LED19, LED4 to LED2, LED19 to LED20, LED20 to LED21, LED21 to LED22, LED22 to LED23, LED23 to LED24, LED27 to LED25, LED30 to LED26, LED38 to LED27, LED12 to LED3, LED31 to LED30, LED32 to LED31, LED33 to LED32, LED34 to LED33, LED35 to LED34, LED36 to LED35, LED37 to LED36, LED39 to LED37, LED41 to LED38, LED42 to LED39, LED2 to LED4, LED50 to LED40, LED40 to LED41, LED43 to LED42, LED44 to LED43, LED46 to LED47, LED47 to LED49, LED3 to LED5, LED48 to LED50, LED49 to LED51, LED5 to LED6, LED6 to LED7, LED7 to LED8, LED8 to LED9, R19 to R17, R20 to R18, R21 to R19, R22 to R20, R23 to R21, R24 to R22, R25 to R23, R26 to R24, R27 to R41, R29 to R42, R30 to R43, R32 to R44, R33 to R45, R34 to R46, R35 to R47, R36 to R48, R37 to R49, R38 to R50, R28 to R51, R31 to R52, R39 to R53, R44 to R56, R45 to R57, R46 to R58, R47 to R59, R48 to R60, R49 to R61, R50 to R62, R40 to R63, R51 to R65, R57 to R68, R58 to R69, R59 to R70, R60 to R71, R61 to R72, R62 to R73, R63 to R74, R53 to R75, R56 to R76, R64 to R77, R67 to R78, R74 to R83, R75 to R84, R76 to R85, R66 to R86, R68 to R87, R69 to R88, R77 to R89, U6 to U5
Connections:
- net 3V3: now also C15.2, R14.2; no longer C15.1, R14.1
- net 5V: now also R25.2, R26.2, R27.2, R28.2, R29.2, R30.2, R31.2, R32.2, R33.2, R34.2, R35.2, R36.2, R37.2, R38.2, R39.2, R40.1
- net C0: now also SW14.1, U1.15 (PA5); no longer SW14.2, U1.29 (PA8)
- net C10: now also U1.11 (PA1)
- net C11: now also SW13.1, SW25.1, SW37.1, SW49.1, U1.12 (PA2); no longer SW13.2, SW25.2, SW37.2, SW49.2
- net C2: now also U1.2 (PC13)
- net C3: now also U1.46 (PB9)
- net C4: now also SW42.1, U1.45 (PB8); no longer SW42.2
- net C5: now also U1.41 (PB5), SW50.2
- net C6: now also U1.40 (PB4), SW51.2
- net C7: now also U1.39 (PB3), SW52.2
- net C8: now also U1.38 (PA15)
- net C9: now also U1.10 (PA0-WKUP)
- net GND: now also C15.1, R14.1, R51.2, R52.1, R53.2, R63.2, R65.2, R75.2, R76.2, R77.2, R86.2, R87.2, R88.2, R89.2, C27.2, C28.2, C29.2, C30.2, C31.2, C32.2, C33.2, C34.2, C35.2, C36.2, C37.2, C38.2, C39.2, C40.2, C41.2, C42.2, LED44.K, LED46.K, LED48.K, R64.2; no longer C15.2, LED1.K, LED13.K, LED14.K, LED15.K, LED2.K, LED25.K, LED26.K, LED27.K, LED3.K, LED37.K, LED38.K, LED39.K, LED40.K, R14.2
- net R0: now also U1.29 (PA8)
- net at D25.1 (DOUT): now also D26.3 (DIN)
- net at D25.3 (DIN): now also D24.1 (DOUT)
- net at D25.4 (VDD): now also C41.1, R39.1
- net at Q3.3 (D), R42.1, R43.1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: now also LED1.A, LED13.A, LED14.A, LED15.A, LED2.A, LED25.A, LED26.A, LED27.A, LED3.A, LED37.A, LED38.A, LED39.A, LED40.A, R66.1, R67.1, R79.1, R80.1, R81.1, R82.1; no longer R51.1, R52.2, R53.1, R63.1, R65.1, R75.1, R76.1, R77.1, R86.1, R87.1, R88.1, R89.1
- net at LED42.A: now also R79.2
- net R3: now reaches U1.13 (PA3)
- net R3: now also D63.1 (K), D64.1 (K), D65.1 (K), D66.1 (K), D67.1 (K), D68.1 (K), D69.1 (K), D70.1 (K), D71.1 (K), D72.1 (K), D73.1 (K), D74.1 (K)
- net R2: now reaches U1.14 (PA4)
- net R2: now also D51.1 (K), D52.1 (K), D53.1 (K), D54.1 (K), D55.1 (K), D56.1 (K), D57.1 (K), D58.1 (K), D59.1 (K), D60.1 (K), D61.1 (K), D62.1 (K)
- net R1: now reaches U1.27 (PB14)
- net R1: now also D39.1 (K), D40.1 (K), D41.1 (K), D42.1 (K), D43.1 (K), D44.1 (K), D45.1 (K), D46.1 (K), D47.1 (K), D48.1 (K), D49.1 (K), D50.1 (K)
- net at D20.1 (DOUT): now also D21.3 (DIN)
- net at D20.3 (DIN): now also D19.1 (DOUT)
- net at D20.4 (VDD): now also C36.1, R34.1
- net at D62.2 (A): now also SW37.2; no longer SW37.1
- net at D70.2 (A), SW45.1: now also SW52.1
- net at LED28.A: now also R66.2
- net at D11.1 (DOUT): now also D12.3 (DIN)
- net at D11.3 (DIN): now also D10.1 (DOUT)
- net at D11.4 (VDD): now also C27.1, R25.1
- net at D74.2 (A): now also SW49.2; no longer SW49.1
- net at LED17.A: now also R55.2
- net at LED45.A: now also LED46.A, R81.2
- net at D68.2 (A), SW43.1: now also SW50.1
- net at D50.2 (A): now also SW25.2; no longer SW25.1
- net at D38.2 (A): now also SW13.2; no longer SW13.1
- net at D17.1 (DOUT): now also D18.3 (DIN)
- net at D17.3 (DIN): now also D16.1 (DOUT)
- net at D17.4 (VDD): now also C33.1, R31.1
- net at LED43.A: now also LED44.A, R80.2
- net at D13.1 (DOUT): now also D14.3 (DIN)
- net at D13.3 (DIN): now also D12.1 (DOUT)
- net at D13.4 (VDD): now also C29.1, R27.1
- net at LED29.A: now also R67.2; no longer R55.2
- net at D12.4 (VDD): now also C28.1, R26.1
- net at D21.1 (DOUT): now also D22.3 (DIN)
- net at D21.4 (VDD): now also C37.1, R35.1
- net at D14.1 (DOUT): now also D15.3 (DIN)
- net at D14.4 (VDD): now also C30.1, R28.1
- net at D67.2 (A): now also SW42.2; no longer SW42.1
- net at LED47.A: now also LED48.A, R82.2
- net at D24.3 (DIN): now also D23.1 (DOUT)
- net at D24.4 (VDD): now also C40.1, R38.1
- net at D16.3 (DIN): now also D15.1 (DOUT)
- net at D16.4 (VDD): now also C32.1, R30.1
- net at D26.4 (VDD): now also C42.1, R40.2
- net at D22.1 (DOUT): now also D23.3 (DIN)
- net at D22.4 (VDD): now also C38.1, R36.1
- net at D39.2 (A): now also SW14.2; no longer SW14.1
- net at D23.4 (VDD): now also C39.1, R37.1
- net at D18.1 (DOUT): now also D19.3 (DIN)
- net at D18.4 (VDD): now also C34.1, R32.1
- net at D69.2 (A), SW44.1: now also SW51.1
- net at D19.4 (VDD): now also C35.1, R33.1
- net at D15.4 (VDD): now also C31.1, R29.1
- new net: LED1.K, R51.1
- new net: LED26.K, R76.1
- new net: LED39.K, R88.1
- new net: LED25.K, R75.1
- new net: LED38.K, R87.1
- new net: LED14.K, R64.1
- new net: LED40.K, R89.1
- new net: LED2.K, R52.2
- new net: LED15.K, R65.1
- new net: LED13.K, R63.1
- new net: LED37.K, R86.1
- new net: LED27.K, R77.1
- new net: LED3.K, R53.1
Other:
- note removed: "RGB STRIP"
- moved on the sheet: C15, LED1, LED13, LED14, LED15, LED2, LED25, LED26, LED27, LED3, LED37, LED38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

Commit message: Finish routing
Parts:
- removed GR2, GR4, GR6, GR9: Warning, acheron_Graphics:Warning_Sign_3.6x3.2mm, symbol Mechanical:MountingHole
- removed GR3: Grounding sign, acheron_Graphics:Grounding_Sign_3.6x3.2mm, symbol Mechanical:MountingHole
- removed X2: USB_EXPOSED_PINS, acheron_Connectors:PinHeader_1x4_P2.54mm_Vertical, symbol Connector_Generic:Conn_01x04
- added FB2: GZ2012D601TF, Inductor_SMD:L_0805_2012Metric, symbol Device:Ferrite_Bead_Small
- added MH1, MH2, MH3, MH4, MH5, MH6: MountingHole, shark_library:MountingHole_2.5mm_Pad, symbol Mechanical:MountingHole_Pad
- renumbered GR5 to GR2, GR7 to GR3, GR8 to GR4
Connections:
- net GND: now also FB2.1
- new net: FB2.2, MH2.1
- no-connect marks 3 -> 8

Commit message: Edit component metadata; prepare for releasee
Parts:
- removed R5: 0R, Resistor_SMD:R_0805_2012Metric, symbol Device:R_Small
- removed R76, R83, R84: 1k, Resistor_SMD:R_0805_2012Metric, symbol Device:R_Small
- removed R90: 1k, Resistor_SMD:R_0402_1005Metric, symbol Device:R_Small
- removed U5: RS0102YH8, acheron_Components:SOT-23-8, symbol acheron_Symbols:RS0102YH8
- added C2, C5: 100n, Capacitor_SMD:C_0402_1005Metric, symbol Device:C_Small
- added Q4: 2N7002, Package_TO_SOT_SMD:SOT-23, symbol Transistor_FET:2N7002
- added R40, R41, R44: 10k, Resistor_SMD:R_0402_1005Metric, symbol Device:R_Small
- added R43: 100, Resistor_SMD:R_0402_1005Metric, symbol Device:R_Small
- added R79, R86, R87: 1k, Resistor_SMD:R_0402_1005Metric, symbol Device:R_Small
- added SW1: EC11Ex, acheron_Hardware:ALPS_EC11E, symbol Device:RotaryEncoder_Switch
- added U5: TXS0101DRLR, acheron_Components:SOT-563, symbol acheronSymbols:TXS0101
- added X2: EXTRA_PINS, acheron_Connectors:PinHeader_2x5_P2.54mm_Vertical, symbol Connector_Generic:Conn_02x05_Odd_Even
- C6: renamed from C4; Specification 16V 1uF Tantallum -> 16V 10uF Tantallum
- GR3: value Athena Label -> Shark plated quote; footprint athena_library:athena_label_35x5.6 -> shark_library:sharkpcb_quote
- GR4: value Acheron Logo -> Shark label; footprint acheron_Logos:acheronLong -> shark_library:sharkpcb_label
- R3: Manufacturer (none) -> Uniroyal; Manufacturer Part Number (none) -> 0805W8F1002T5E; Specification (none) -> ±1% 1/8W Thick Film Resistors 150V 0805; Vendor Part Number (none) -> LCSC C17414
- SW10: renamed from SW9; Keycode ESC -> (none)
- SW11: renamed from SW10; Keycode ESC -> (none)
- SW12: renamed from SW11; Keycode ESC -> (none)
- SW13: renamed from SW12; Keycode ESC -> (none)
- SW14: renamed from SW13; Keycode ESC -> (none)
- SW15: renamed from SW14; Keycode ESC -> (none)
- SW16: renamed from SW15; Keycode ESC -> (none)
- SW17: renamed from SW16; Keycode ESC -> (none)
- SW18: renamed from SW17; Keycode ESC -> (none)
- SW19: renamed from SW18; Keycode ESC -> (none)
- SW20: renamed from SW19; Keycode ESC -> (none)
- SW21: renamed from SW20; Keycode ESC -> (none)
- SW22: renamed from SW21; Keycode ESC -> (none)
- SW23: renamed from SW22; Keycode ESC -> (none)
- SW24: renamed from SW23; Keycode ESC -> (none)
- SW25: renamed from SW24; Keycode ESC -> (none)
- SW26: renamed from SW25; Keycode ESC -> (none)
- SW27: renamed from SW26; Keycode ESC -> (none)
- SW28: renamed from SW27; Keycode ESC -> (none)
- SW29: renamed from SW28; Keycode ESC -> (none)
- SW3: renamed from SW2; Keycode ESC -> (none)
- SW30: renamed from SW29; Keycode ESC -> (none)
- SW31: renamed from SW30; Keycode ESC -> (none)
- SW32: renamed from SW31; Keycode ESC -> (none)
- SW33: renamed from SW32; Keycode ESC -> (none)
- SW34: renamed from SW33; Keycode ESC -> (none)
- SW35: renamed from SW34; Keycode ESC -> (none)
- SW36: renamed from SW35; Keycode ESC -> (none)
- SW37: renamed from SW36; Keycode ESC -> (none)
- SW38: renamed from SW37; Keycode ESC -> (none)
- SW39: renamed from SW38; Keycode ESC -> (none)
- SW4: renamed from SW3; Keycode ESC -> (none)
- SW40: renamed from SW39; Keycode ESC -> (none)
- SW41: renamed from SW40; Keycode ESC -> (none)
- SW42: renamed from SW41; Keycode ESC -> (none)
- SW43: renamed from SW42; Keycode ESC -> (none)
- SW44: renamed from SW43; Keycode ESC -> (none)
- SW45: renamed from SW44; Keycode ESC -> (none)
- SW46: renamed from SW45; Keycode ESC -> (none)
- SW47: renamed from SW46; Keycode ESC -> (none)
- SW48: renamed from SW47; Keycode ESC -> (none)
- SW49: renamed from SW48; Keycode ESC -> (none)
- SW5: renamed from SW4; Keycode ESC -> (none)
- SW50: renamed from SW49; Keycode ESC -> (none)
- SW51: renamed from SW50; Keycode ESC -> (none)
- SW52: renamed from SW51; Keycode ESC -> (none)
- SW53: renamed from SW52; Keycode ESC -> (none)
- SW6: renamed from SW5; Keycode ESC -> (none)
- SW7: renamed from SW6; Keycode ESC -> (none)
- SW8: renamed from SW7; Keycode ESC -> (none)
- SW9: renamed from SW8; Keycode ESC -> (none)
- renumbered C8 to C10, C9 to C11, C10 to C12, C11 to C13, C12 to C14, C13 to C15, C14 to C16, C15 to C17, C16 to C18, C17 to C19, C18 to C20, C19 to C21, C20 to C22, C21 to C23, C22 to C24, C23 to C25, C24 to C26, C25 to C27, C26 to C28, C27 to C29, C2 to C3, C28 to C30, C29 to C31, C30 to C32, C31 to C33, C32 to C34, C33 to C35, C34 to C36, C35 to C37, C36 to C38, C37 to C39, C3 to C4, C38 to C40, C39 to C41, C40 to C42, C41 to C43, C42 to C44, C5 to C7, C6 to C8, C7 to C9, R11 to R10, R12 to R11, R13 to R12, R14 to R13, R15 to R14, R16 to R15, R17 to R16, R18 to R17, R19 to R18, R20 to R19, R21 to R20, R22 to R21, R23 to R22, R24 to R23, R25 to R24, R26 to R25, R27 to R26, R28 to R27, R29 to R28, R30 to R29, R31 to R30, R32 to R31, R33 to R32, R34 to R33, R35 to R34, R36 to R35, R37 to R36, R38 to R37, R39 to R38, R40 to R39, R41 to R42, R42 to R45, R43 to R46, R44 to R47, R45 to R48, R46 to R49, R6 to R5, R47 to R50, R48 to R51, R49 to R52, R50 to R53, R51 to R54, R52 to R55, R53 to R56, R54 to R57, R55 to R58, R56 to R59, R7 to R6, R57 to R60, R58 to R61, R59 to R62, R60 to R63, R61 to R64, R62 to R65, R63 to R66, R64 to R67, R65 to R68, R66 to R69, R8 to R7, R67 to R70, R68 to R71, R69 to R72, R70 to R73, R71 to R74, R72 to R75, R73 to R76, R74 to R77, R75 to R78, R9 to R8, R77 to R80, R78 to R81, R79 to R82, R80 to R83, R81 to R84, R82 to R85, R85 to R88, R86 to R89, R10 to R9, R87 to R90, R88 to R91, R89 to R92, SW1 to SW2
Connections:
- net 3V3: now also R40.1, U5.1 (VCCA), X2.1 (Pin_1)
- net 5V: now also R41.2, U5.6 (VCCB), X2.4 (Pin_4)
- net BACKLIGHT_3V3: now also R43.1
- net C11: now also SW1.S1
- net GND: now also C2.1, C5.2, Q4.2 (S), R44.1, R79.2, SW1.C, U5.2 (GND), X2.6 (Pin_6)
- net RGB_3V3: now also U5.3 (A)
- net RGB_5V: now also U5.4 (B)
- net E_PA7: now reaches U1.17 (PA7)
- net E_PA7: now also X2.8 (Pin_8)
- net E_PB0: now reaches U1.18 (PB0)
- net E_PB0: now also X2.7 (Pin_7)
- net E_PB10: now reaches U1.21 (B10)
- net E_PB10: now also X2.9 (Pin_9)
- net E_PB12: now reaches U1.25 (PB12)
- net E_PB12: now also X2.3 (Pin_3)
- net E_PB13: now reaches U1.26 (PB13)
- net E_PB13: now also X2.2 (Pin_2)
- net E_B: now reaches U1.3 (PC14_OSC32IN)
- net E_B: now also C5.1, SW1.B
- net E_A: now reaches U1.4 (PC15_OSC32OUT)
- net E_A: now also C2.2, SW1.A
- net at LED1.A, LED13.A, LED14.A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: now also R86.1, R87.1
- net at LED26.K: now also R79.1
- net E_S2: now reaches D38.2 (A), SW14.2
- net E_S2: now also SW1.S2
- net at LED49.A: now also R86.2
- net at R42.2: now also Q4.3 (D), R41.1; no longer Q3.1 (G)
- net at LED50.A: now also R87.2
- net BACKLIGHT_5V: no longer names the net of R42.1
- net BACKLIGHT_5V: now also Q3.1 (G)
- net CAPS_INDICATOR renamed E_PB1
- net E_PB1: now also X2.10 (Pin_10)
- net PA9 renamed E_PA9
- net E_PA9: now also X2.5 (Pin_5)
- new net: Q4.1 (G), R43.2, R44.2
- new net: R40.2, U5.5 (OE)
- no-connect marks 8 -> 7
Other:
- note added: "ENCODER"
- note added: "MOUNTING"
- moved on the sheet: C1, C10, C11, C12, C13, C14, C15, C16, C17, C18, C19, C20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
